File: Yobi/Quectel-2560-v2.1.brd (EAGLE design)
At the start: 56.6 x 90.7 mm, 108 parts, among them IC1 LM2576S, IC2 LM2576S, J1 U.FL, T1 NPN, T2 PNP, T3 NPN, U1 ATMEGA1280AU, U2 Quectel M95, U3 QUECTEL-L80

Commit message: jkl
Parts:
- removed L3: 100uh, resistor:L5038P
- added JP11: Pogo Pin, pinhead:1X01
- added L4: 100uh, rcl:PIS2816
- added PAD1: Pad, wirepad:SMD1,27-2,54
- L1: value (none) -> Ferrite Bead
- L2: value 100uh -> 100uf; device resistor:L5038P -> rcl:PIS2816
- LED4: value (none) -> Charging
- R1: value 1k -> 0
- R10, R11, R47: value 50 -> 22
- R12, R6, R7, R8: value 220 -> 1k
- R14, R17, R18, R25, R27, R28: value 330 -> 1k
- R19, R22, R30, R35, R39, R42, R5: value 50 -> 35
- R23, R24, R4, R9: value 330 -> 2k
- R29: value 220 -> 2k
- R37: value 330 -> 3.6k
- R38: value 330 -> 11k
- R45: value 330 -> 2.4k
- R46: value 330 -> 5.6k
- moved L2 27.9 mm to (21.0, 19.5)
- moved DC16 7.60 mm to (2.60, 65.9), turned to 90 degrees
- moved C9 2.50 mm to (15.2, 31.4)
- moved R29 2.50 mm to (22.1, 55.4)
- moved D11 2.30 mm to (20.0, 44.5)
- moved T1 2.02 mm to (40.4, 43.1)
- moved R14 2.00 mm to (22.1, 57.6)
- moved R19 1.66 mm to (43.2, 57.9), turned to 90 degrees
- moved D3 1.60 mm to (9.11, 46.1)
- moved DC2 1.51 mm to (45.9, 77.4)
- moved R22 1.50 mm to (46.5, 57.2)
- moved LED5 1.41 mm to (53.8, 83.0)
- moved R21 1.39 mm to (47.1, 72.5)
- moved R38 1.30 mm to (32.6, 48.2), turned to 90 degrees
- moved C3 1.30 mm to (17.2, 60.3)
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Connections:
- new net N$69: PAD1.1, U1.90
- net +4.1V: now also JP11.1, L2.2; no longer L3.2
- net 5V: now also L4.2; no longer L2.2
- net N$65: now also L4.1; no longer L2.1
- net N$77: now also L2.1; no longer L3.1
Routing:
- net GND: track 703.0 -> 690.5 mm
- net 5V: track 184.0 -> 178.2 mm, vias 2 -> 3
- net +8V: track 47.6 -> 51.4 mm
- net N$69: track 0.00 -> 2.87 mm
- net N$78: track 8.43 -> 11.0 mm
- net N$65: track 11.4 -> 13.9 mm
- net N$15: track 11.0 -> 13.2 mm
- net 3.3V: track 101.7 -> 99.6 mm
- net N$47: track 12.9 -> 11.1 mm
- net N$46: track 12.3 -> 10.5 mm
- net N$22: track 15.2 -> 16.9 mm
- net N$72: track 5.37 -> 3.85 mm
- net N$40: track 8.74 -> 10.2 mm
- net +4.1V: track 118.3 -> 119.5 mm, vias 2 -> 1
- net N$66: track 3.36 -> 4.44 mm
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
Commit message: cbdg
Parts:
- removed PAD1: Pad, wirepad:SMD1,27-2,54
- added R48: 1k\, SparkFun-Resistors:0805
- added T4: NPN, semicon-smd-ipc:SOT23
- moved DC17 0.92 mm to (50.3, 69.9)
Connections:
- removed net N$69: PAD1.1, U1.90
- new net N$79: R44.1, T4.3
- new net N$80: R48.1, T4.1
- new net N$81: R48.2, U1.83
- net GND: now also T4.2; no longer R44.1
- net N$75: now also U1.84; no longer U1.83
Routing:
- net N$80: track 0.00 -> 25.9 mm, vias 0 -> 1
- net GND: track 690.5 -> 703.5 mm
- net N$81: track 0.00 -> 12.5 mm
- net N$79: track 0.00 -> 9.44 mm, vias 0 -> 1
- net N$69: track 2.87 -> 0.00 mm
- net N$47: track 11.1 -> 13.8 mm
- net N$75: track 12.1 -> 12.9 mm
