File: Yobi/Quectel-2560-v2.1.brd (EAGLE design)
At the start: 56.6 x 90.7 mm, 111 parts, among them IC1 LM2576S, IC2 LM2576S, J1 U.FL, T1 NPN, T2 PNP, T3 NPN, T4 NPN, U1 ATMEGA1280AU, U2 Quectel M95, U3 QUECTEL-L80

Commit message: dfbfd
Parts:
- removed DC8, DC9: pf, resistor:C0805
- removed J1: U.FL, SparkFun-Connectors:U.FL
- removed R1: 0, SparkFun-Resistors:0805
- removed R2: 1k, SparkFun-Resistors:0805
- removed R37: 3.6k, SparkFun-Resistors:0805
- removed R38: 11k, SparkFun-Resistors:0805
- removed T1: NPN, semicon-smd-ipc:SOT23
- added L3, L6: (no value), rcl:6000-XXXX-RC
- added R49: 2.4k, SparkFun-Resistors:0805
- added R50: 5.6k, SparkFun-Resistors:0805
- added U4: V_REG_317DPACK, SparkFun-IC-Power:V-REG_DPACK
- added X1: LTI-SASF54GT, con-coax:LTI-SASF54GT
- moved R41 2.26 mm to (49.4, 59.1)
- moved DC18 2.10 mm to (36.1, 69.6)
- moved L1 2.10 mm to (34.0, 69.6)
- moved D11 1.80 mm to (18.2, 44.5)
- moved L4 1.43 mm to (29.3, 46.1)
- moved R27 0.81 mm to (29.5, 58.7), turned to 90 degrees
- moved R8 0.70 mm to (19.7, 85.8)
- moved R23 0.60 mm to (19.7, 84.0)
- moved R6 0.50 mm to (19.7, 82.2)
- moved R9 0.30 mm to (19.7, 80.3)
- moved R24 0.20 mm to (19.7, 76.4)
- moved R7 0.10 mm to (19.7, 78.4)
- turned JP9 to 270 degrees
Connections:
- removed net N$14: R2.2, U1.76
- removed net N$15: R2.1, T1.1
- removed net N$46: T1.3, U2.20
- removed net N$5: DC9.1, J1.FEED, R1.2
- removed net N$72: IC1.4, R37.2, R38.1
- new net N$69: R49.1, R50.2, U4.1
- net +4.1V: now also L3.2, R50.1, U4.4
- net +8V: now also U4.3
- net 5V: now also IC1.4, L6.2; no longer R38.2
- net GND: now also R49.2, X1.2, X1.3, X1.4, X1.5; no longer DC8.1, DC9.2, J1.1, J1.2, R37.1, T1.2
- net N$21: now also X1.1; no longer DC8.2, R1.1
- net N$65: now also L6.1
- net N$77: now also L3.1
Routing:
- net GND: track 703.5 -> 670.8 mm
- net +4.1V: track 119.5 -> 146.9 mm
- net N$14: track 23.9 -> 0.00 mm, vias 1 -> 0
- net N$15: track 13.2 -> 0.00 mm, vias 1 -> 0
- net N$46: track 10.5 -> 0.00 mm
- net N$69: track 0.00 -> 7.89 mm
- net N$21: track 12.6 -> 6.27 mm
- net +8V: track 51.4 -> 57.7 mm
- net N$5: track 4.41 -> 0.00 mm
- net N$72: track 3.85 -> 0.00 mm
- net N$77: track 21.4 -> 24.8 mm
- net 5V: track 178.2 -> 180.6 mm
- net N$65: track 13.9 -> 15.6 mm
- net N$61: track 4.23 -> 2.61 mm
- net N$76: track 39.7 -> 38.2 mm
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- removed copper zone on layer 16, net 5V

Commit message: fdb
Parts:
- added JP12: IIC, pinhead:1X04
- added JP13: D, pinhead:1X03
Changed lines of the file:
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@@
 <layer number="14" name="Route14" color="1" fill="6" visible="no" active="no"/>
 <layer number="15" name="Route15" color="4" fill="6" visible="no" active="no"/>
-<layer number="16" name="Bottom" color="1" fill="1" visible="no" active="yes"/>
+<layer number="16" name="Bottom" color="1" fill="1" visible="yes" active="yes"/>
 <layer number="17" name="Pads" color="2" fill="1" visible="yes" active="yes"/>
 <layer number="18" name="Vias" color="2" fill="1" visible="yes" active="yes"/>
@@
 <layer number="43" name="vRestrict" color="2" fill="10" visible="no" active="yes"/>
 <layer number="44" name="Drills" color="7" fill="1" visible="no" active="yes"/>
-<layer number="45" name="Holes" color="7" fill="1" visible="no" active="yes"/>
+<layer number="45" name="Holes" color="7" fill="1" visible="yes" active="yes"/>
 <layer number="46" name="Milling" color="3" fill="1" visible="no" active="yes"/>
 <layer number="47" name="Measures" color="7" fill="1" visible="no" active="yes"/>
@@
 <circle x="51.1" y="53.8" radius="3.4" width="0.254" layer="22"/>
 <dimension x1="56.6" y1="90.7" x2="56.6" y2="0" x3="60.2" y3="45.35" textsize="1.778" layer="20" dtype="vertical"/>
-<dimension x1="0" y1="0" x2="56.6" y2="0" x3="28.3" y3="-3.8" textsize="1.778" layer="20" dtype="horizontal"/>
+<dimension x1="0" y1="0" x2="56.6" y2="0" x3="28.3" y3="-24.4" textsize="1.778" layer="20" dtype="horizontal"/>
+<wire x1="55.7" y1="-1" x2="55.7" y2="-16.6" width="0.4064" layer="21"/>
+<wire x1="55.7" y1="-1" x2="47.9" y2="-1" width="0.4064" layer="21"/>
+<wire x1="47.9" y1="-1" x2="47.9" y2="-16.6" width="0.4064" layer="21"/>
+<wire x1="47.9" y1="-16.6" x2="55.7" y2="-16.6" width="0.4064" layer="21"/>
 </plain>
 <attributes>
@@
 <attribute name="OC_NEWARK" value="unknown" x="46.2" y="4.9" size="1.778" layer="27" display="off"/>
 </element>
+<element name="JP12" library="pinhead" package="1X04" value="IIC" x="50.3" y="-8.7" rot="R270"/>
+<element name="JP13" library="pinhead" package="1X03" value="D" x="13.3" y="-8.4" rot="R90"/>
 </elements>
 <signals>

Commit message: tu
Parts:
- added DC8, DC9: 0.1uf, resistor:C0805
- added JP14, JP15, JP17: IIC, pinhead:1X04
- added JP16: D, pinhead:1X03
- added JP18: IN, pinhead:1X02
- added JP19: OUT, pinhead:1X02
- added Q1: CSM-7X-DU, crystal:CSM-7X-DU
- added R1, R37: 5.6k, SparkFun-Resistors:0805
- added R2: 2.4k, SparkFun-Resistors:0805
- added U5: V_REG_317DPACK, SparkFun-IC-Power:V-REG_DPACK
- moved JP13 25.4 mm to (38.7, -8.70), turned to 270 degrees
Connections:
- new net N$14: DC8.2, JP12.4, JP13.3, JP14.2
- new net N$15: JP13.2, JP14.3
- new net N$46: JP12.3, JP14.4
- new net N$5: DC8.1, JP12.1, JP13.1, JP14.1
- new net N$72: DC9.1, JP15.1, JP16.1, JP17.1
- new net N$82: DC9.2, JP15.4, JP16.3, JP17.2
- new net N$83: JP15.3, JP17.4
- new net N$84: JP16.2, JP17.3
- new net N$85: R1.2, R2.1, U5.1
- new net N$86: JP18.1, JP19.2, R2.2, R37.2
- new net N$87: JP18.2, U5.3
- new net N$88: JP19.1, Q1.2, R1.1, U5.4
- new net N$89: Q1.1, R37.1
Routing:
- net N$86: track 0.00 -> 35.4 mm
- net N$88: track 0.00 -> 31.4 mm
- net N$14: track 0.00 -> 23.3 mm
- net N$82: track 0.00 -> 22.8 mm
- net N$5: track 0.00 -> 17.3 mm
- net N$72: track 0.00 -> 17.2 mm
- net N$85: track 0.00 -> 10.9 mm, vias 0 -> 2
- net N$87: track 0.00 -> 9.20 mm
- net N$83: track 0.00 -> 6.85 mm
- net N$46: track 0.00 -> 6.85 mm
- net N$15: track 0.00 -> 6.33 mm
- net N$84: track 0.00 -> 6.23 mm
- net N$89: track 0.00 -> 2.32 mm
- net +4.1V: track 146.9 -> 148.2 mm
- added copper zone on layer 1, net N$5
- added copper zone on layer 16, net N$5
- added copper zone on layer 1, net N$72
- added copper zone on layer 16, net N$72
Other:
- board size 56.6 x 90.7 mm -> 56.6 x 108.4 mm
- board text added: "+5"
- board text added: "3.3"
- board text added: "A"
- board text added: "B"
- board text added: "C"
- board text added: "D"
- board text added: "DHT"
- board text added: "E"
- board text added: "F"
- board text added: "GND"
- board text added: "IIC"
- board text added: "L-80"
- board text added: "M"
- board text added: "MET"
- board text added: "OUT"
- board text added: "RI"
- board text added: "RST"
- board text added: "Rx"
- board text added: "S"
- board text added: "SCL"
- board text added: "SDA"
- board text added: "Tx"
- board text added: "VDD"

Commit message: tyj
Parts:
- removed R3: 330, SparkFun-Resistors:0805
- removed T2: PNP, semicon-smd-ipc:SOT23
- added DC19: 0.1uf, resistor:C0805
- added DC20: 1nf, resistor:C0805
- added IC3: ACS712, ACS712:SO08
- moved D3 5.56 mm to (3.71, 47.4), turned to 270 degrees
Connections:
- removed net N$18: R3.2, U2.26
- removed net N$28: R3.1, T2.1
- new net N$90: D3.K, IC3.1
- new net N$91: DC20.2, IC3.6
- net 5V: now also DC19.2, IC3.8
- net GND: now also DC19.1, DC20.1, IC3.5; no longer T2.3
- net N$13: no longer T2.2
- net N$19: now also IC3.4; no longer D3.K
Routing:
- net N$18: track 47.2 -> 0.00 mm, vias 1 -> 0
- net N$90: track 0.00 -> 9.96 mm
- net GND: track 670.8 -> 677.5 mm
- net 5V: track 180.6 -> 186.6 mm
- net N$13: track 112.8 -> 109.5 mm
- net N$91: track 0.00 -> 2.75 mm
- net N$28: track 2.12 -> 0.00 mm
- net N$19: track 10.5 -> 12.5 mm
- net N$25: track 13.3 -> 12.0 mm

Commit message: fhgjk
Parts:
- removed JP18: IN, pinhead:1X02
- removed JP19: OUT, pinhead:1X02
- removed Q1: CSM-7X-DU, crystal:CSM-7X-DU
- removed R2: 2.4k, SparkFun-Resistors:0805
- removed R37: 5.6k, SparkFun-Resistors:0805
- removed U5: V_REG_317DPACK, SparkFun-IC-Power:V-REG_DPACK
- added DC21: 1nf, resistor:C0805
- R1: value 5.6k -> 35
- moved R1 60.2 mm to (14.1, 53.8), flipped to the top, turned to 180 degrees
- moved DC9 15.0 mm to (17.7, -8.80)
- moved JP13 15.0 mm to (23.7, -8.70)
- moved JP17 15.0 mm to (8.60, -8.80)
- moved DC8 15.0 mm to (38.4, -8.80)
- moved JP12 15.0 mm to (35.3, -8.70)
- moved JP14 15.0 mm to (29.5, -8.70)
- moved JP15 15.0 mm to (14.4, -8.80)
- moved JP16 15.0 mm to (2.90, -8.80)
- moved R43 2.44 mm to (43.6, 45.5)
- moved R22 0.91 mm to (45.6, 57.1)
Connections:
- removed net N$85: R1.2, R2.1, U5.1
- removed net N$86: JP18.1, JP19.2, R2.2, R37.2
- removed net N$87: JP18.2, U5.3
- removed net N$88: JP19.1, Q1.2, R1.1, U5.4
- removed net N$89: Q1.1, R37.1
- new net N$18: DC21.1, R1.1, U1.82
- new net N$28: IC3.7, R1.2
- net GND: now also DC21.2
- net N$75: now also U1.85; no longer U1.84
- net N$76: now also U1.83; no longer U1.82
- net N$81: now also U1.84; no longer U1.83
Routing:
- net N$18: track 0.00 -> 71.0 mm, vias 0 -> 2
- net N$86: track 35.4 -> 0.00 mm
- net N$88: track 31.4 -> 0.00 mm
- net N$85: track 10.9 -> 0.00 mm, vias 2 -> 0
- net N$87: track 9.20 -> 0.00 mm
- net N$28: track 0.00 -> 7.26 mm, vias 0 -> 1
- net GND: track 677.5 -> 684.1 mm, vias 43 -> 45
- net N$89: track 2.32 -> 0.00 mm
- net N$76: track 38.2 -> 36.5 mm
- net +8V: track 57.7 -> 59.1 mm
- net N$22: track 17.7 -> 16.5 mm
Other:
- outline, holes or cut-outs redrawn
