File: Yobi/Quectel-2560-v2.1.sch (EAGLE design)
At the start: 108 parts, among them IC1 LM2576S, IC2 LM2576S, J1 U.FL, T1 NPN, T2 PNP, T3 NPN, U1 ATMEGA1280AU, U2 Quectel M95, U3 QUECTEL-L80

Commit message: jkl
Parts:
- removed L3: 100uh, resistor:L-USL5038P
- added JP11: Pogo Pin, pinhead:PINHD-1X1
- added L4: 100uh, rcl:L-USPIS2816
- added PAD1: Pad, wirepad:SMD2
- L1: value (none) -> Ferrite Bead
- L2: value 100uh -> 100uf; device resistor:L-USL5038P -> rcl:L-USPIS2816
- LED4: value (none) -> Charging
- R1: value 1k -> 0
- R10, R11, R47: value 50 -> 22
- R12, R6, R7, R8: value 220 -> 1k
- R14, R17, R18, R25, R27, R28: value 330 -> 1k
- R19, R22, R30, R35, R39, R42, R5: value 50 -> 35
- R23, R24, R4, R9: value 330 -> 2k
- R29: value 220 -> 2k
- R37: value 330 -> 3.6k
- R38: value 330 -> 11k
- R45: value 330 -> 2.4k
- R46: value 330 -> 5.6k
Connections:
- new net N$69: PAD1.P, U1.(ADC7/TDI)PF7
- net +4.1V: now also JP11.1, L2.2; no longer L3.2
- net 5V: now also L4.2; no longer L2.2
- net N$65: now also L4.1; no longer L2.1
- net N$77: now also L2.1; no longer L3.1
Other:
- moved on the sheet: L2

Commit message: cbdg
Parts:
- removed PAD1: Pad, wirepad:SMD2
- added R48: 1k\, SparkFun-Resistors:RESISTOR0805-RES
- added T4: NPN, semicon-smd-ipc:NPN-TRANSISTOR_SOT23
Connections:
- removed net N$69: PAD1.P, U1.(ADC7/TDI)PF7
- new net N$79: R44.1, T4.C
- new net N$80: R48.1, T4.B
- new net N$81: R48.2, U1.PK6(ADC14/PCINT22)
- net GND: now also T4.E; no longer R44.1
- net N$75: now also U1.PK5(ADC13/PCINT21); no longer U1.PK6(ADC14/PCINT22)
Changed lines of the file:
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@@
 <part name="DC16" library="resistor" deviceset="C-EU" device="C0805" value="0.1uf"/>
 <part name="JP11" library="pinhead" deviceset="PINHD-1X1" device="" value="Pogo Pin"/>
-<part name="PAD1" library="wirepad" deviceset="SMD2" device="" value="Pad"/>
 <part name="L4" library="rcl" deviceset="L-US" device="PIS2816" value="100uh"/>
 <part name="L2" library="rcl" deviceset="L-US" device="PIS2816" value="100uf"/>
+<part name="T4" library="semicon-smd-ipc" deviceset="NPN-TRANSISTOR_" device="SOT23" value="NPN"/>
+<part name="R48" library="SparkFun-Resistors" deviceset="RESISTOR" device="0805-RES" value="1k\"/>
 </parts>
 <sheets>
@@
 </instance>
 <instance part="SUPPLY54" gate="GND" x="104.14" y="71.12" rot="R270"/>
-<instance part="R43" gate="G$1" x="48.26" y="114.3" smashed="yes">
-<attribute name="VALUE" x="46.99" y="110.998" size="1.778" layer="96"/>
-</instance>
-<instance part="R44" gate="G$1" x="55.88" y="109.22" smashed="yes" rot="R90">
-<attribute name="VALUE" x="59.182" y="107.95" size="1.778" layer="96" rot="R90"/>
-</instance>
-<instance part="SUPPLY55" gate="+8V" x="35.56" y="114.3" rot="R90"/>
-<instance part="SUPPLY58" gate="GND" x="60.96" y="99.06"/>
+<instance part="R43" gate="G$1" x="50.8" y="116.84" smashed="yes">
+<attribute name="VALUE" x="49.53" y="113.538" size="1.778" layer="96"/>
+</instance>
+<instance part="R44" gate="G$1" x="58.42" y="116.84" smashed="yes" rot="R90">
+<attribute name="VALUE" x="61.722" y="115.57" size="1.778" layer="96" rot="R90"/>
+</instance>
+<instance part="SUPPLY55" gate="+8V" x="40.64" y="116.84" rot="R90"/>
+<instance part="SUPPLY58" gate="GND" x="58.42" y="99.06"/>
 <instance part="IC2" gate="A" x="142.24" y="292.1"/>
 <instance part="SUPPLY63" gate="+8V" x="119.38" y="297.18" rot="R90"/>
@@
 </instance>
 <instance part="JP11" gate="G$1" x="187.96" y="292.1"/>
-<instance part="PAD1" gate="1" x="142.24" y="93.98" rot="R90"/>
 <instance part="L4" gate="G$1" x="101.6" y="274.32" rot="R90"/>
 <instance part="L2" gate="G$1" x="165.1" y="292.1" rot="R90"/>
+<instance part="T4" gate="G$1" x="60.96" y="106.68" rot="MR0"/>
+<instance part="R48" gate="G$1" x="63.5" y="111.76" smashed="yes" rot="R90">
+<attribute name="VALUE" x="61.722" y="110.49" size="1.778" layer="96" rot="R90"/>
+</instance>
 </instances>
 <busses>
@@
 </segment>
 <segment>
+<pinref part="T4" gate="G$1" pin="E"/>
 <pinref part="SUPPLY58" gate="GND" pin="GND"/>
-<pinref part="R44" gate="G$1" pin="1"/>
-<wire x1="55.88" y1="104.14" x2="55.88" y2="101.6" width="0.1524" layer="91"/>
-<wire x1="55.88" y1="101.6" x2="60.96" y2="101.6" width="0.1524" layer="91"/>
 </segment>
 </net>
@@
 <segment>
 <pinref part="SUPPLY55" gate="+8V" pin="+8V"/>
-<wire x1="38.1" y1="114.3" x2="43.18" y2="114.3" width="0.1524" layer="91"/>
+<wire x1="43.18" y1="116.84" x2="45.72" y2="116.84" width="0.1524" layer="91"/>
 <pinref part="R43" gate="G$1" pin="1"/>
 </segment>
@@
 <wire x1="91.44" y1="86.36" x2="104.14" y2="86.36" width="0.1524" layer="91"/>
 <pinref part="R21" gate="G$1" pin="1"/>
-<wire x1="91.44" y1="127" x2="60.96" y2="127" width="0.1524" layer="91"/>
+<wire x1="91.44" y1="127" x2="58.42" y2="127" width="0.1524" layer="91"/>
 <pinref part="JP1" gate="A" pin="1"/>
-<wire x1="60.96" y1="127" x2="60.96" y2="124.46" width="0.1524" layer="91"/>
-<wire x1="60.96" y1="124.46" x2="48.26" y2="124.46" width="0.1524" layer="91"/>
+<wire x1="58.42" y1="127" x2="58.42" y2="124.46" width="0.1524" layer="91"/>
+<wire x1="58.42" y1="124.46" x2="48.26" y2="124.46" width="0.1524" layer="91"/>
 </segment>
 </net>
@@
 <wire x1="129.54" y1="71.12" x2="129.54" y2="114.3" width="0.1524" layer="91"/>
 <wire x1="129.54" y1="114.3" x2="99.06" y2="114.3" width="0.1524" layer="91"/>
-<pinref part="U1" gate="1" pin="PK6(ADC14/PCINT22)"/>
-<wire x1="99.06" y1="114.3" x2="99.06" y2="121.92" width="0.1524" layer="91"/>
-<wire x1="99.06" y1="121.92" x2="68.58" y2="121.92" width="0.1524" layer="91"/>
+<wire x1="99.06" y1="114.3" x2="99.06" y2="119.38" width="0.1524" layer="91"/>
+<pinref part="U1" gate="1" pin="PK5(ADC13/PCINT21)"/>
+<wire x1="68.58" y1="119.38" x2="99.06" y2="119.38" width="0.1524" layer="91"/>
 </segment>
 </net>
 <net name="N$76" class="0">
 <segment>
+<pinref part="R44" gate="G$1" pin="2"/>
+<wire x1="58.42" y1="121.92" x2="60.96" y2="121.92" width="0.1524" layer="91"/>
+<wire x1="60.96" y1="121.92" x2="60.96" y2="124.46" width="0.1524" layer="91"/>
+<pinref part="U1" gate="1" pin="PK7(ADC15/PCINT23)"/>
+<wire x1="60.96" y1="124.46" x2="68.58" y2="124.46" width="0.1524" layer="91"/>
 <pinref part="R43" gate="G$1" pin="2"/>
-<pinref part="R44" gate="G$1" pin="2"/>
-<wire x1="53.34" y1="114.3" x2="55.88" y2="114.3" width="0.1524" layer="91"/>
-<wire x1="55.88" y1="114.3" x2="55.88" y2="121.92" width="0.1524" layer="91"/>
-<wire x1="55.88" y1="121.92" x2="63.5" y2="121.92" width="0.1524" layer="91"/>
-<wire x1="63.5" y1="121.92" x2="63.5" y2="124.46" width="0.1524" layer="91"/>
-<pinref part="U1" gate="1" pin="PK7(ADC15/PCINT23)"/>
-<wire x1="63.5" y1="124.46" x2="68.58" y2="124.46" width="0.1524" layer="91"/>
-<junction x="55.88" y="114.3"/>
+<wire x1="58.42" y1="121.92" x2="55.88" y2="121.92" width="0.1524" layer="91"/>
+<wire x1="55.88" y1="121.92" x2="55.88" y2="116.84" width="0.1524" layer="91"/>
+<junction x="58.42" y="121.92"/>
 </segment>
 </net>
@@
 </segment>
 </net>
-<net name="N$69" class="0">
-<segment>
-<pinref part="PAD1" gate="1" pin="P"/>
-<pinref part="U1" gate="1" pin="(ADC7/TDI)PF7"/>
-<wire x1="142.24" y1="96.52" x2="139.7" y2="96.52" width="0.1524" layer="91"/>
-</segment>
-</net>
+<net name="N$79" class="0">
+<segment>
+<pinref part="R44" gate="G$1" pin="1"/>
+<pinref part="T4" gate="G$1" pin="C"/>
+</segment>
+</net>
+<net name="N$80" class="0">
+<segment>
+<pinref part="T4" gate="G$1" pin="B"/>
+<pinref part="R48" gate="G$1" pin="1"/>
+</segment>
+</net>
+<net name="N$81" class="0">
+<segment>
+<pinref part="R48" gate="G$1" pin="2"/>
+<wire x1="63.5" y1="116.84" x2="63.5" y2="121.92" width="0.1524" layer="91"/>
+<pinref part="U1" gate="1" pin="PK6(ADC14/PCINT22)"/>
+<wire x1="63.5" y1="121.92" x2="68.58" y2="121.92" width="0.1524" layer="91"/>
+</segment>
+</net>

Commit message: dfbfd
Parts:
- removed DC8, DC9: pf, resistor:C-EUC0805
- removed J1: U.FL, SparkFun-Connectors:U.FL2PIN
- removed R1: 0, SparkFun-Resistors:RESISTOR0805-RES
- removed R2: 1k, SparkFun-Resistors:RESISTOR0805-RES
- removed R37: 3.6k, SparkFun-Resistors:RESISTOR0805-RES
- removed R38: 11k, SparkFun-Resistors:RESISTOR0805-RES
- removed T1: NPN, semicon-smd-ipc:NPN-TRANSISTOR_SOT23
- added L3, L6: (no value), rcl:L-US6000-XXX-RC
- added R49: 2.4k, SparkFun-Resistors:RESISTOR0805-RES
- added R50: 5.6k, SparkFun-Resistors:RESISTOR0805-RES
- added U4: V_REG_317DPACK, SparkFun-IC-Power:V_REG_317DPACK
- added X1: LTI-SASF54GT, con-coax:LTI-SASF54GT
Connections:
- removed net N$14: R2.2, U1.(AD2)PA2
- removed net N$15: R2.1, T1.B
- removed net N$46: T1.C, U2.DTR
- removed net N$5: DC9.1, J1.SIGNAL, R1.2
- removed net N$72: IC1.FB, R37.2, R38.1
- new net N$69: R49.1, R50.2, U4.ADJ
- net +4.1V: now also L3.2, R50.1, U4.OUT
- net +8V: now also U4.IN
- net 5V: now also IC1.FB, L6.2; no longer R38.2
- net GND: now also R49.2, X1.2; no longer DC8.1, DC9.2, J1.GND, R37.1, T1.E
- net N$21: now also X1.1; no longer DC8.2, R1.1
- net N$65: now also L6.1
- net N$77: now also L3.1
Other:
- moved on the sheet: C1, C10, JP11

Commit message: fdb
Parts:
- added JP12: IIC, pinhead:PINHD-1X4
- added JP13: D, pinhead:PINHD-1X3
Changed lines of the file:
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@@
 <part name="X1" library="con-coax" deviceset="LTI-SASF54GT" device=""/>
 <part name="SUPPLY46" library="supply2" deviceset="GND" device=""/>
+<part name="JP12" library="pinhead" deviceset="PINHD-1X4" device="" value="IIC"/>
+<part name="JP13" library="pinhead" deviceset="PINHD-1X3" device="" value="D"/>
 </parts>
 <sheets>
@@
 <instance part="X1" gate="G$1" x="160.02" y="104.14"/>
 <instance part="SUPPLY46" gate="GND" x="162.56" y="99.06"/>
+<instance part="JP12" gate="A" x="228.6" y="246.38" rot="R90"/>
+<instance part="JP13" gate="A" x="226.06" y="233.68" rot="R90"/>
 </instances>
 <busses>

Commit message: tu
Parts:
- added DC8, DC9: 0.1uf, resistor:C-EUC0805
- added JP14, JP15, JP17: IIC, pinhead:PINHD-1X4
- added JP16: D, pinhead:PINHD-1X3
- added JP18: IN, pinhead:PINHD-1X2
- added JP19: OUT, pinhead:PINHD-1X2
- added Q1: CSM-7X-DU, crystal:CSM-7X-DU
- added R1, R37: 5.6k, SparkFun-Resistors:RESISTOR0805-RES
- added R2: 2.4k, SparkFun-Resistors:RESISTOR0805-RES
- added U5: V_REG_317DPACK, SparkFun-IC-Power:V_REG_317DPACK
Connections:
- new net N$14: DC8.2, JP12.4, JP13.3, JP14.2
- new net N$15: JP13.2, JP14.3
- new net N$46: JP12.3, JP14.4
- new net N$5: DC8.1, JP12.1, JP13.1, JP14.1
- new net N$72: DC9.1, JP15.1, JP16.1, JP17.1
- new net N$82: DC9.2, JP15.4, JP16.3, JP17.2
- new net N$83: JP15.3, JP17.4
- new net N$84: JP16.2, JP17.3
- new net N$85: R1.2, R2.1, U5.ADJ
- new net N$86: JP18.1, JP19.2, R2.2, R37.2
- new net N$87: JP18.2, U5.IN
- new net N$88: JP19.1, Q1.2, R1.1, U5.OUT
- new net N$89: Q1.1, R37.1
Changed lines of the file:
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@@
 <part name="JP12" library="pinhead" deviceset="PINHD-1X4" device="" value="IIC"/>
 <part name="JP13" library="pinhead" deviceset="PINHD-1X3" device="" value="D"/>
+<part name="JP14" library="pinhead" deviceset="PINHD-1X4" device="" value="IIC"/>
+<part name="DC8" library="resistor" deviceset="C-EU" device="C0805" value="0.1uf"/>
+<part name="JP15" library="pinhead" deviceset="PINHD-1X4" device="" value="IIC"/>
+<part name="JP16" library="pinhead" deviceset="PINHD-1X3" device="" value="D"/>
+<part name="JP17" library="pinhead" deviceset="PINHD-1X4" device="" value="IIC"/>
+<part name="DC9" library="resistor" deviceset="C-EU" device="C0805" value="0.1uf"/>
+<part name="U5" library="SparkFun-IC-Power" deviceset="V_REG_317" device="DPACK"/>
+<part name="R1" library="SparkFun-Resistors" deviceset="RESISTOR" device="0805-RES" value="5.6k"/>
+<part name="R2" library="SparkFun-Resistors" deviceset="RESISTOR" device="0805-RES" value="2.4k"/>
+<part name="JP18" library="pinhead" deviceset="PINHD-1X2" device="" value="IN"/>
+<part name="JP19" library="pinhead" deviceset="PINHD-1X2" device="" value="OUT"/>
+<part name="Q1" library="crystal" deviceset="CSM-7X-DU" device=""/>
+<part name="R37" library="SparkFun-Resistors" deviceset="RESISTOR" device="0805-RES" value="5.6k"/>
 </parts>
 <sheets>
@@
 <instance part="JP12" gate="A" x="228.6" y="246.38" rot="R90"/>
 <instance part="JP13" gate="A" x="226.06" y="233.68" rot="R90"/>
+<instance part="JP14" gate="A" x="243.84" y="236.22" rot="R90"/>
+<instance part="DC8" gate="G$1" x="238.76" y="243.84" smashed="yes" rot="R90">
+<attribute name="VALUE" x="243.459" y="245.364" size="1.778" layer="96" rot="R90"/>
+</instance>
+<instance part="JP15" gate="A" x="248.92" y="281.94" rot="R90"/>
+<instance part="JP16" gate="A" x="246.38" y="269.24" rot="R90"/>
+<instance part="JP17" gate="A" x="264.16" y="271.78" rot="R90"/>
+<instance part="DC9" gate="G$1" x="259.08" y="279.4" smashed="yes" rot="R90">
+<attribute name="VALUE" x="263.779" y="280.924" size="1.778" layer="96" rot="R90"/>
+</instance>
+<instance part="U5" gate="G$1" x="238.76" y="312.42"/>
+<instance part="R1" gate="G$1" x="243.84" y="297.18" smashed="yes" rot="R180">
+<attribute name="VALUE" x="245.11" y="295.402" size="1.778" layer="96" rot="R180"/>
+</instance>
+<instance part="R2" gate="G$1" x="233.68" y="297.18" smashed="yes" rot="R180">
+<attribute name="VALUE" x="234.95" y="300.482" size="1.778" layer="96" rot="R180"/>
+</instance>
+<instance part="JP18" gate="G$1" x="220.98" y="312.42" rot="R180"/>
+<instance part="JP19" gate="G$1" x="259.08" y="309.88"/>
+<instance part="Q1" gate="P" x="246.38" y="320.04"/>
+<instance part="R37" gate="G$1" x="238.76" y="320.04" smashed="yes" rot="R180">
+<attribute name="VALUE" x="240.03" y="318.262" size="1.778" layer="96" rot="R180"/>
+</instance>
 </instances>
 <busses>
@@
 </segment>
 </net>
+<net name="N$5" class="0">
+<segment>
+<pinref part="JP12" gate="A" pin="1"/>
+<pinref part="JP13" gate="A" pin="1"/>
+<wire x1="223.52" y1="243.84" x2="223.52" y2="231.14" width="0.1524" layer="91"/>
+<wire x1="223.52" y1="231.14" x2="223.52" y2="223.52" width="0.1524" layer="91"/>
+<pinref part="JP14" gate="A" pin="1"/>
+<wire x1="223.52" y1="223.52" x2="238.76" y2="223.52" width="0.1524" layer="91"/>
+<wire x1="238.76" y1="223.52" x2="238.76" y2="233.68" width="0.1524" layer="91"/>
+<pinref part="DC8" gate="G$1" pin="1"/>
+<wire x1="236.22" y1="243.84" x2="236.22" y2="238.76" width="0.1524" layer="91"/>
+<wire x1="236.22" y1="238.76" x2="238.76" y2="238.76" width="0.1524" layer="91"/>
+<wire x1="238.76" y1="238.76" x2="238.76" y2="233.68" width="0.1524" layer="91"/>
+</segment>
+</net>
+<net name="N$14" class="0">
+<segment>
+<pinref part="JP12" gate="A" pin="4"/>
+<wire x1="231.14" y1="243.84" x2="231.14" y2="231.14" width="0.1524" layer="91"/>
+<pinref part="JP13" gate="A" pin="3"/>
+<wire x1="231.14" y1="231.14" x2="228.6" y2="231.14" width="0.1524" layer="91"/>
+<pinref part="JP14" gate="A" pin="2"/>
+<wire x1="231.14" y1="231.14" x2="241.3" y2="231.14" width="0.1524" layer="91"/>
+<wire x1="241.3" y1="231.14" x2="241.3" y2="233.68" width="0.1524" layer="91"/>
+<pinref part="DC8" gate="G$1" pin="2"/>
+<wire x1="243.84" y1="243.84" x2="243.84" y2="238.76" width="0.1524" layer="91"/>
+<wire x1="243.84" y1="238.76" x2="241.3" y2="238.76" width="0.1524" layer="91"/>
+<wire x1="241.3" y1="238.76" x2="241.3" y2="233.68" width="0.1524" layer="91"/>
+</segment>
+</net>
+<net name="N$46" class="0">
+<segment>
+<pinref part="JP12" gate="A" pin="3"/>
+<wire x1="228.6" y1="243.84" x2="228.6" y2="236.22" width="0.1524" layer="91"/>
+<wire x1="228.6" y1="236.22" x2="246.38" y2="236.22" width="0.1524" layer="91"/>
+<pinref part="JP14" gate="A" pin="4"/>
+<wire x1="246.38" y1="236.22" x2="246.38" y2="233.68" width="0.1524" layer="91"/>
+</segment>
+</net>
+<net name="N$15" class="0">
+<segment>
+<pinref part="JP13" gate="A" pin="2"/>
+<wire x1="226.06" y1="231.14" x2="226.06" y2="226.06" width="0.1524" layer="91"/>
+<wire x1="226.06" y1="226.06" x2="243.84" y2="226.06" width="0.1524" layer="91"/>
+<pinref part="JP14" gate="A" pin="3"/>
+<wire x1="243.84" y1="233.68" x2="243.84" y2="226.06" width="0.1524" layer="91"/>
+</segment>
+</net>
+<net name="N$72" class="0">
+<segment>
+<pinref part="JP15" gate="A" pin="1"/>
+<pinref part="JP16" gate="A" pin="1"/>
+<wire x1="243.84" y1="279.4" x2="243.84" y2="266.7" width="0.1524" layer="91"/>
+<wire x1="243.84" y1="266.7" x2="243.84" y2="259.08" width="0.1524" layer="91"/>
+<pinref part="JP17" gate="A" pin="1"/>
+<wire x1="243.84" y1="259.08" x2="259.08" y2="259.08" width="0.1524" layer="91"/>
+<wire x1="259.08" y1="259.08" x2="259.08" y2="269.24" width="0.1524" layer="91"/>
+<pinref part="DC9" gate="G$1" pin="1"/>
+<wire x1="256.54" y1="279.4" x2="256.54" y2="274.32" width="0.1524" layer="91"/>
+<wire x1="256.54" y1="274.32" x2="259.08" y2="274.32" width="0.1524" layer="91"/>
+<wire x1="259.08" y1="274.32" x2="259.08" y2="269.24" width="0.1524" layer="91"/>
+</segment>
+</net>
+<net name="N$82" class="0">
+<segment>
+<pinref part="JP15" gate="A" pin="4"/>
+<wire x1="251.46" y1="279.4" x2="251.46" y2="266.7" width="0.1524" layer="91"/>
+<pinref part="JP16" gate="A" pin="3"/>
+<wire x1="251.46" y1="266.7" x2="248.92" y2="266.7" width="0.1524" layer="91"/>
+<pinref part="JP17" gate="A" pin="2"/>
+<wire x1="251.46" y1="266.7" x2="261.62" y2="266.7" width="0.1524" layer="91"/>
+<wire x1="261.62" y1="266.7" x2="261.62" y2="269.24" width="0.1524" layer="91"/>
+<pinref part="DC9" gate="G$1" pin="2"/>
+<wire x1="264.16" y1="279.4" x2="264.16" y2="274.32" width="0.1524" layer="91"/>
+<wire x1="264.16" y1="274.32" x2="261.62" y2="274.32" width="0.1524" layer="91"/>
+<wire x1="261.62" y1="274.32" x2="261.62" y2="269.24" width="0.1524" layer="91"/>
+</segment>
+</net>
+<net name="N$83" class="0">
+<segment>
+<pinref part="JP15" gate="A" pin="3"/>
+<wire x1="248.92" y1="279.4" x2="248.92" y2="271.78" width="0.1524" layer="91"/>
+<wire x1="248.92" y1="271.78" x2="266.7" y2="271.78" width="0.1524" layer="91"/>
+<pinref part="JP17" gate="A" pin="4"/>
+<wire x1="266.7" y1="271.78" x2="266.7" y2="269.24" width="0.1524" layer="91"/>
+</segment>
+</net>
+<net name="N$84" class="0">
+<segment>
+<pinref part="JP16" gate="A" pin="2"/>
+<wire x1="246.38" y1="266.7" x2="246.38" y2="261.62" width="0.1524" layer="91"/>
+<wire x1="246.38" y1="261.62" x2="264.16" y2="261.62" width="0.1524" layer="91"/>
+<pinref part="JP17" gate="A" pin="3"/>
+<wire x1="264.16" y1="269.24" x2="264.16" y2="261.62" width="0.1524" layer="91"/>
+</segment>
+</net>
+<net name="N$85" class="0">
+<segment>
+<pinref part="R1" gate="G$1" pin="2"/>
+<pinref part="R2" gate="G$1" pin="1"/>
+<pinref part="U5" gate="G$1" pin="ADJ"/>
+<wire x1="238.76" y1="304.8" x2="238.76" y2="297.18" width="0.1524" layer="91"/>
+</segment>
+</net>
+<net name="N$86" class="0">
+<segment>
+<pinref part="JP18" gate="G$1" pin="1"/>
+<wire x1="223.52" y1="309.88" x2="226.06" y2="309.88" width="0.1524" layer="91"/>
+<wire x1="226.06" y1="309.88" x2="226.06" y2="307.34" width="0.1524" layer="91"/>
+<pinref part="R2" gate="G$1" pin="2"/>
+<wire x1="226.06" y1="307.34" x2="226.06" y2="302.26" width="0.1524" layer="91"/>
+<wire x1="226.06" y1="302.26" x2="226.06" y2="297.18" width="0.1524" layer="91"/>
+<wire x1="226.06" y1="297.18" x2="228.6" y2="297.18" width="0.1524" layer="91"/>
+<pinref part="JP19" gate="G$1" pin="2"/>
+<wire x1="226.06" y1="302.26" x2="256.54" y2="302.26" width="0.1524" layer="91"/>
+<wire x1="256.54" y1="302.26" x2="256.54" y2="309.88" width="0.1524" layer="91"/>
+<pinref part="R37" gate="G$1" pin="2"/>
+<wire x1="233.68" y1="320.04" x2="231.14" y2="320.04" width="0.1524" layer="91"/>
+<wire x1="231.14" y1="320.04" x2="231.14" y2="307.34" width="0.1524" layer="91"/>
+<wire x1="231.14" y1="307.34" x2="226.06" y2="307.34" width="0.1524" layer="91"/>
+</segment>
+</net>
+<net name="N$87" class="0">
+<segment>
+<pinref part="JP18" gate="G$1" pin="2"/>
+<pinref part="U5" gate="G$1" pin="IN"/>
+<wire x1="223.52" y1="312.42" x2="231.14" y2="312.42" width="0.1524" layer="91"/>
+</segment>
+</net>
+<net name="N$88" class="0">
+<segment>
+<pinref part="JP19" gate="G$1" pin="1"/>
+<pinref part="U5" gate="G$1" pin="OUT"/>
+<wire x1="256.54" y1="312.42" x2="248.92" y2="312.42" width="0.1524" layer="91"/>
+<pinref part="R1" gate="G$1" pin="1"/>
+<wire x1="248.92" y1="312.42" x2="246.38" y2="312.42" width="0.1524" layer="91"/>
+<wire x1="248.92" y1="312.42" x2="248.92" y2="297.18" width="0.1524" layer="91"/>
+<pinref part="Q1" gate="P" pin="2"/>
+<wire x1="248.92" y1="320.04" x2="248.92" y2="312.42" width="0.1524" layer="91"/>
+</segment>
+</net>
+<net name="N$89" class="0">
+<segment>
+<pinref part="Q1" gate="P" pin="1"/>
+<pinref part="R37" gate="G$1" pin="1"/>
+</segment>
+</net>

Commit message: tyj
Parts:
- removed R3: 330, SparkFun-Resistors:RESISTOR0805-RES
- removed T2: PNP, semicon-smd-ipc:PNP-TRANSISTOR_SOT23
- added DC19: 0.1uf, resistor:C-EUC0805
- added DC20: 1nf, resistor:C-EUC0805
- added IC3: ACS712, ACS712:ACS712
Connections:
- removed net N$18: R3.2, U2.RI
- removed net N$28: R3.1, T2.B
- new net N$90: D3.K, IC3.I+_0
- new net N$91: DC20.2, IC3.FILTER
- net 5V: now also DC19.2, IC3.VCC
- net GND: now also DC19.1, DC20.1, IC3.GND; no longer T2.C
- net N$13: no longer T2.E
- net N$19: now also IC3.I-_1; no longer D3.K
Other:
- moved on the sheet: D3, JP9, LED4
