File: Yobi/Quectel-2560-v2.1.sch (EAGLE design)
At the start: 125 parts, among them IC1 LM2576S, IC2 LM2576S, IC3 ACS712, Q1 CSM-7X-DU, T3 NPN, T4 NPN, U1 ATMEGA1280AU, U2 Quectel M95, U3 QUECTEL-L80, U4 V_REG_317DPACK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

Commit message: fhgjk
Parts:
- removed JP18: IN, pinhead:PINHD-1X2
- removed JP19: OUT, pinhead:PINHD-1X2
- removed Q1: CSM-7X-DU, crystal:CSM-7X-DU
- removed R2: 2.4k, SparkFun-Resistors:RESISTOR0805-RES
- removed R37: 5.6k, SparkFun-Resistors:RESISTOR0805-RES
- removed U5: V_REG_317DPACK, SparkFun-IC-Power:V_REG_317DPACK
- added DC21: 1nf, resistor:C-EUC0805
- R1: value 5.6k -> 35
Connections:
- removed net N$85: R1.2, R2.1, U5.ADJ
- removed net N$86: JP18.1, JP19.2, R2.2, R37.2
- removed net N$87: JP18.2, U5.IN
- removed net N$88: JP19.1, Q1.2, R1.1, U5.OUT
- removed net N$89: Q1.1, R37.1
- new net N$18: DC21.1, R1.1, U1.PK7(ADC15/PCINT23)
- new net N$28: IC3.VOUT, R1.2
- net GND: now also DC21.2
- net N$75: now also U1.PK4(ADC12/PCINT20); no longer U1.PK5(ADC13/PCINT21)
- net N$76: now also U1.PK6(ADC14/PCINT22); no longer U1.PK7(ADC15/PCINT23)
- net N$81: now also U1.PK5(ADC13/PCINT21); no longer U1.PK6(ADC14/PCINT22)
Changed lines of the file:
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@@
 <part name="JP17" library="pinhead" deviceset="PINHD-1X4" device="" value="IIC"/>
 <part name="DC9" library="resistor" deviceset="C-EU" device="C0805" value="0.1uf"/>
-<part name="U5" library="SparkFun-IC-Power" deviceset="V_REG_317" device="DPACK"/>
-<part name="R1" library="SparkFun-Resistors" deviceset="RESISTOR" device="0805-RES" value="5.6k"/>
-<part name="R2" library="SparkFun-Resistors" deviceset="RESISTOR" device="0805-RES" value="2.4k"/>
-<part name="JP18" library="pinhead" deviceset="PINHD-1X2" device="" value="IN"/>
-<part name="JP19" library="pinhead" deviceset="PINHD-1X2" device="" value="OUT"/>
-<part name="Q1" library="crystal" deviceset="CSM-7X-DU" device=""/>
-<part name="R37" library="SparkFun-Resistors" deviceset="RESISTOR" device="0805-RES" value="5.6k"/>
 <part name="IC3" library="ACS712" deviceset="ACS712" device=""/>
 <part name="SUPPLY44" library="SparkFun-Aesthetics" deviceset="5V" device=""/>
@@
 <part name="DC20" library="resistor" deviceset="C-EU" device="C0805" value="1nf"/>
 <part name="SUPPLY62" library="supply2" deviceset="GND" device=""/>
+<part name="R1" library="SparkFun-Resistors" deviceset="RESISTOR" device="0805-RES" value="35"/>
+<part name="DC21" library="resistor" deviceset="C-EU" device="C0805" value="1nf"/>
+<part name="SUPPLY13" library="supply2" deviceset="GND" device=""/>
 </parts>
 <sheets>
@@
 <attribute name="VALUE" x="263.779" y="280.924" size="1.778" layer="96" rot="R90"/>
 </instance>
-<instance part="U5" gate="G$1" x="238.76" y="312.42"/>
-<instance part="R1" gate="G$1" x="243.84" y="297.18" smashed="yes" rot="R180">
-<attribute name="VALUE" x="245.11" y="295.402" size="1.778" layer="96" rot="R180"/>
-</instance>
-<instance part="R2" gate="G$1" x="233.68" y="297.18" smashed="yes" rot="R180">
-<attribute name="VALUE" x="234.95" y="300.482" size="1.778" layer="96" rot="R180"/>
-</instance>
-<instance part="JP18" gate="G$1" x="220.98" y="312.42" rot="R180"/>
-<instance part="JP19" gate="G$1" x="259.08" y="309.88"/>
-<instance part="Q1" gate="P" x="246.38" y="320.04"/>
-<instance part="R37" gate="G$1" x="238.76" y="320.04" smashed="yes" rot="R180">
-<attribute name="VALUE" x="240.03" y="318.262" size="1.778" layer="96" rot="R180"/>
-</instance>
 <instance part="IC3" gate="A" x="43.18" y="223.52" rot="MR270"/>
 <instance part="SUPPLY44" gate="G$1" x="33.02" y="208.28" rot="R90"/>
@@
 </instance>
 <instance part="SUPPLY62" gate="GND" x="33.02" y="198.12"/>
+<instance part="R1" gate="G$1" x="40.64" y="195.58" smashed="yes" rot="R90">
+<attribute name="VALUE" x="43.942" y="194.31" size="1.778" layer="96" rot="R90"/>
+</instance>
+<instance part="DC21" gate="G$1" x="38.1" y="190.5" smashed="yes" rot="R270">
+<attribute name="VALUE" x="33.401" y="188.976" size="1.778" layer="96" rot="R270"/>
+</instance>
+<instance part="SUPPLY13" gate="GND" x="30.48" y="190.5" rot="R270"/>
 </instances>
 <busses>
@@
 <pinref part="DC19" gate="G$1" pin="1"/>
 <pinref part="SUPPLY62" gate="GND" pin="GND"/>
+</segment>
+<segment>
+<pinref part="DC21" gate="G$1" pin="2"/>
+<pinref part="SUPPLY13" gate="GND" pin="GND"/>
 </segment>
 </net>
@@
 <wire x1="129.54" y1="71.12" x2="129.54" y2="114.3" width="0.1524" layer="91"/>
 <wire x1="129.54" y1="114.3" x2="99.06" y2="114.3" width="0.1524" layer="91"/>
-<wire x1="99.06" y1="114.3" x2="99.06" y2="119.38" width="0.1524" layer="91"/>
-<pinref part="U1" gate="1" pin="PK5(ADC13/PCINT21)"/>
-<wire x1="68.58" y1="119.38" x2="99.06" y2="119.38" width="0.1524" layer="91"/>
+<wire x1="99.06" y1="114.3" x2="99.06" y2="116.84" width="0.1524" layer="91"/>
+<pinref part="U1" gate="1" pin="PK4(ADC12/PCINT20)"/>
+<wire x1="68.58" y1="116.84" x2="99.06" y2="116.84" width="0.1524" layer="91"/>
 </segment>
 </net>
@@
 <segment>
 <pinref part="R44" gate="G$1" pin="2"/>
-<wire x1="58.42" y1="121.92" x2="60.96" y2="121.92" width="0.1524" layer="91"/>
-<wire x1="60.96" y1="121.92" x2="60.96" y2="124.46" width="0.1524" layer="91"/>
-<pinref part="U1" gate="1" pin="PK7(ADC15/PCINT23)"/>
-<wire x1="60.96" y1="124.46" x2="68.58" y2="124.46" width="0.1524" layer="91"/>
 <pinref part="R43" gate="G$1" pin="2"/>
 <wire x1="58.42" y1="121.92" x2="55.88" y2="121.92" width="0.1524" layer="91"/>
 <wire x1="55.88" y1="121.92" x2="55.88" y2="116.84" width="0.1524" layer="91"/>
 <junction x="58.42" y="121.92"/>
+<pinref part="U1" gate="1" pin="PK6(ADC14/PCINT22)"/>
+<wire x1="68.58" y1="121.92" x2="58.42" y2="121.92" width="0.1524" layer="91"/>
 </segment>
 </net>
@@
 <segment>
 <pinref part="R48" gate="G$1" pin="2"/>
-<wire x1="63.5" y1="116.84" x2="63.5" y2="121.92" width="0.1524" layer="91"/>
-<pinref part="U1" gate="1" pin="PK6(ADC14/PCINT22)"/>
-<wire x1="63.5" y1="121.92" x2="68.58" y2="121.92" width="0.1524" layer="91"/>
+<wire x1="63.5" y1="116.84" x2="63.5" y2="119.38" width="0.1524" layer="91"/>
+<pinref part="U1" gate="1" pin="PK5(ADC13/PCINT21)"/>
+<wire x1="68.58" y1="119.38" x2="63.5" y2="119.38" width="0.1524" layer="91"/>
 </segment>
 </net>
@@
 </segment>
 </net>
-<net name="N$85" class="0">
-<segment>
-<pinref part="R1" gate="G$1" pin="2"/>
-<pinref part="R2" gate="G$1" pin="1"/>
-<pinref part="U5" gate="G$1" pin="ADJ"/>
-<wire x1="238.76" y1="304.8" x2="238.76" y2="297.18" width="0.1524" layer="91"/>
-</segment>
-</net>
-<net name="N$86" class="0">
-<segment>
-<pinref part="JP18" gate="G$1" pin="1"/>
-<wire x1="223.52" y1="309.88" x2="226.06" y2="309.88" width="0.1524" layer="91"/>
-<wire x1="226.06" y1="309.88" x2="226.06" y2="307.34" width="0.1524" layer="91"/>
-<pinref part="R2" gate="G$1" pin="2"/>
-<wire x1="226.06" y1="307.34" x2="226.06" y2="302.26" width="0.1524" layer="91"/>
-<wire x1="226.06" y1="302.26" x2="226.06" y2="297.18" width="0.1524" layer="91"/>
-<wire x1="226.06" y1="297.18" x2="228.6" y2="297.18" width="0.1524" layer="91"/>
-<pinref part="JP19" gate="G$1" pin="2"/>
-<wire x1="226.06" y1="302.26" x2="256.54" y2="302.26" width="0.1524" layer="91"/>
-<wire x1="256.54" y1="302.26" x2="256.54" y2="309.88" width="0.1524" layer="91"/>
-<pinref part="R37" gate="G$1" pin="2"/>
-<wire x1="233.68" y1="320.04" x2="231.14" y2="320.04" width="0.1524" layer="91"/>
-<wire x1="231.14" y1="320.04" x2="231.14" y2="307.34" width="0.1524" layer="91"/>
-<wire x1="231.14" y1="307.34" x2="226.06" y2="307.34" width="0.1524" layer="91"/>
-</segment>
-</net>
-<net name="N$87" class="0">
-<segment>
-<pinref part="JP18" gate="G$1" pin="2"/>
-<pinref part="U5" gate="G$1" pin="IN"/>
-<wire x1="223.52" y1="312.42" x2="231.14" y2="312.42" width="0.1524" layer="91"/>
-</segment>
-</net>
-<net name="N$88" class="0">
-<segment>
-<pinref part="JP19" gate="G$1" pin="1"/>
-<pinref part="U5" gate="G$1" pin="OUT"/>
-<wire x1="256.54" y1="312.42" x2="248.92" y2="312.42" width="0.1524" layer="91"/>
-<pinref part="R1" gate="G$1" pin="1"/>
-<wire x1="248.92" y1="312.42" x2="246.38" y2="312.42" width="0.1524" layer="91"/>
-<wire x1="248.92" y1="312.42" x2="248.92" y2="297.18" width="0.1524" layer="91"/>
-<pinref part="Q1" gate="P" pin="2"/>
-<wire x1="248.92" y1="320.04" x2="248.92" y2="312.42" width="0.1524" layer="91"/>
-</segment>
-</net>
-<net name="N$89" class="0">
-<segment>
-<pinref part="Q1" gate="P" pin="1"/>
-<pinref part="R37" gate="G$1" pin="1"/>
-</segment>
-</net>
 <net name="N$90" class="0">
 <segment>
@@
 </segment>
 </net>
+<net name="N$18" class="0">
+<segment>
+<wire x1="40.64" y1="185.42" x2="30.48" y2="185.42" width="0.1524" layer="91"/>
+<wire x1="30.48" y1="185.42" x2="30.48" y2="162.56" width="0.1524" layer="91"/>
+<wire x1="30.48" y1="162.56" x2="81.28" y2="162.56" width="0.1524" layer="91"/>
+<pinref part="U1" gate="1" pin="PK7(ADC15/PCINT23)"/>
+<wire x1="68.58" y1="124.46" x2="81.28" y2="124.46" width="0.1524" layer="91"/>
+<wire x1="81.28" y1="124.46" x2="81.28" y2="162.56" width="0.1524" layer="91"/>
+<pinref part="R1" gate="G$1" pin="1"/>
+<wire x1="40.64" y1="190.5" x2="40.64" y2="185.42" width="0.1524" layer="91"/>
+<pinref part="DC21" gate="G$1" pin="1"/>
+<junction x="40.64" y="190.5"/>
+</segment>
+</net>
+<net name="N$28" class="0">
+<segment>
+<pinref part="IC3" gate="A" pin="VOUT"/>
+<pinref part="R1" gate="G$1" pin="2"/>
+<wire x1="40.64" y1="208.28" x2="40.64" y2="200.66" width="0.1524" layer="91"/>
+</segment>
+</net>
