File: Yobi/Quectel-2560-v2.3.brd (EAGLE design)
At the start: 60.4 x 116.3 mm, 158 parts, among them IC1 LM2576S, IC2 LM2576S, IC3 ACS712, T1 NPN, T2 NPN, U1 ATMEGA2560, U2 Quectel M95, X1 LTI-SASF54GT

Commit message: a
Parts:
- moved R62 6.52 mm to (-7.20, 57.6), turned to 270 degrees
