File: POVBase.brd (EAGLE design)
At the start: 19 parts, among them IC1 LM2576S, Q5 IRF540, Q6 IRF540

Commit message: xgns
Parts:
- removed D2: (no value), semicon-smd-ipc:MELF-MLL41
- removed IC1: LM2576S, lm2576:TO263-5
- removed L1: (no value), rcl:6000-XXXX-RC
- added C3: (no value), resistor:C0805
- added IC2: PIC16F876SO, microchip:SO28W
- added JP3: (no value), pinhead:1X06
- added JP4: (no value), pinhead:1X03
- added Q8: (no value), special:QS
- added R5, R6, R7, R8: (no value), resistor:R0805
- C1: device rcl:CT7343 -> resistor:C0805
- C2: device rcl:153CLV-1014 -> resistor:C0805
- moved C1 23.6 mm to (-20.8, -11.7), flipped to the bottom, turned to 270 degrees
- moved C2 21.8 mm to (-20.8, -7.40), flipped to the bottom
- moved R4 16.9 mm to (-39.5, -7.80), flipped to the bottom, turned to 0 degrees
- moved Q2 14.9 mm to (-41.3, -1.80), flipped to the bottom, turned to 0 degrees
- moved R1 14.2 mm to (-24.9, -4.10), flipped to the bottom, turned to 90 degrees
- moved Q1 11.7 mm to (-29.0, -1.80), flipped to the bottom, turned to 0 degrees
- moved Q3 11.7 mm to (-33.1, -1.80), flipped to the bottom, turned to 0 degrees
- moved Q6 11.1 mm to (-45.4, -9.30)
- moved R2 9.36 mm to (-31.9, -6.70), flipped to the bottom, turned to 90 degrees
- moved Q5 8.70 mm to (-26.6, -9.30)
- moved Q4 8.50 mm to (-37.1, -1.80), flipped to the bottom, turned to 0 degrees
- moved Q9 7.40 mm to (-45.4, 12.1)
- moved JP1 6.94 mm to (-36.2, 23.6)
- moved JP2 6.74 mm to (-4.60, 23.6)
- moved R3 5.09 mm to (-36.0, -6.80), flipped to the bottom
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Connections:
- new net N$12: IC2.1, JP3.1, R5.1
- new net N$13: IC2.28, JP3.4
- new net N$14: IC2.27, JP3.5
- new net N$15: IC2.11, R6.1
- new net N$16: C1.2, IC2.10, Q8.1
- new net N$17: C2.2, IC2.9, Q8.2
- new net N$20: R7.1, R8.2
- net +12V: no longer C1.+, IC1.1
- net +5V: now also C3.2, IC2.20, JP3.2, JP4.2, R5.2, R8.1; no longer C2.+, IC1.4, L1.2
- net GND: now also C1.1, C2.1, C3.1, IC2.19, IC2.8, JP3.3, JP4.1, R7.2; no longer C1.-, C2.-, D2.2, IC1.3, IC1.5
- net N$9: now also JP4.3, R6.2; no longer D2.1, IC1.2, L1.1
Routing:
- net GND: track 106.4 -> 252.0 mm, vias 2 -> 1
- net +5V: track 19.4 -> 85.5 mm, vias 1 -> 2
- net N$15: track 0.00 -> 54.4 mm, vias 0 -> 1
- net N$17: track 0.00 -> 18.2 mm
- net N$16: track 0.00 -> 14.0 mm
- net N$11: track 24.9 -> 38.9 mm
- net N$10: track 24.9 -> 38.7 mm
- net N$12: track 0.00 -> 9.54 mm
- net N$14: track 0.00 -> 9.35 mm
- net +12V: track 100.4 -> 107.8 mm, vias 2 -> 1
- net N$13: track 0.00 -> 6.92 mm
- net N$5: track 9.76 -> 2.95 mm
- net N$4: track 36.7 -> 43.5 mm, vias 0 -> 1
- net N$1: track 42.6 -> 47.4 mm, vias 2 -> 1
- net N$9: track 11.7 -> 16.1 mm
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