File: POVBase.brd (EAGLE design)
At the start: 55.5 x 51.2 mm, 25 parts, among them IC2 PIC16F876SO, Q5 IRF540, Q6 IRF540

Commit message: sdgs
Connections:
- net N$1: now also Q5.G; no longer Q6.G
- net N$4: now also Q6.G; no longer Q5.G
- net N$7: now also R1.1; no longer R4.1
- net N$8: now also R4.1; no longer R1.1
Routing:
- net N$4: track 53.7 -> 43.0 mm
- net N$8: track 53.1 -> 43.0 mm
- net N$1: track 50.3 -> 44.5 mm
- net N$3: track 4.94 -> 0.00 mm
- net N$2: track 3.25 -> 0.00 mm
- net N$7: track 37.9 -> 35.2 mm
Changed lines of the file:
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@@
 <grid distance="0.1" unitdist="mm" unit="mm" style="lines" multiple="1" display="yes" altdistance="0.025" altunitdist="inch" altunit="inch"/>
 <layers>
-<layer number="1" name="Top" color="4" fill="1" visible="no" active="yes"/>
+<layer number="1" name="Top" color="4" fill="1" visible="yes" active="yes"/>
 <layer number="2" name="Route2" color="1" fill="3" visible="no" active="no"/>
 <layer number="3" name="Route3" color="4" fill="3" visible="no" active="no"/>
@@
 <layer number="18" name="Vias" color="2" fill="1" visible="yes" active="yes"/>
 <layer number="19" name="Unrouted" color="6" fill="1" visible="yes" active="yes"/>
-<layer number="20" name="Dimension" color="15" fill="1" visible="no" active="yes"/>
-<layer number="21" name="tPlace" color="7" fill="1" visible="no" active="yes"/>
-<layer number="22" name="bPlace" color="7" fill="1" visible="no" active="yes"/>
-<layer number="23" name="tOrigins" color="15" fill="1" visible="no" active="yes"/>
-<layer number="24" name="bOrigins" color="15" fill="1" visible="no" active="yes"/>
+<layer number="20" name="Dimension" color="15" fill="1" visible="yes" active="yes"/>
+<layer number="21" name="tPlace" color="7" fill="1" visible="yes" active="yes"/>
+<layer number="22" name="bPlace" color="7" fill="1" visible="yes" active="yes"/>
+<layer number="23" name="tOrigins" color="15" fill="1" visible="yes" active="yes"/>
+<layer number="24" name="bOrigins" color="15" fill="1" visible="yes" active="yes"/>
 <layer number="25" name="tNames" color="7" fill="1" visible="no" active="yes"/>
 <layer number="26" name="bNames" color="7" fill="1" visible="no" active="yes"/>
@@
 <contactref element="Q1" pad="3"/>
 <contactref element="Q3" pad="3"/>
-<contactref element="Q6" pad="G"/>
 <contactref element="Q7" pad="G"/>
 <wire x1="-37.8" y1="4" x2="-33.7" y2="4" width="0.4064" layer="16"/>
@@
 <wire x1="-48" y1="6.6" x2="-45.3" y2="6.6" width="0.4064" layer="16"/>
 <via x="-45.3" y="6.6" extent="1-16" drill="0.8"/>
-<wire x1="-57.14" y1="-2.54" x2="-57.14" y2="-8.34" width="0.4064" layer="16"/>
 <wire x1="-29.24" y1="9.46" x2="-42.44" y2="9.46" width="0.4064" layer="1"/>
 <wire x1="-42.44" y1="9.46" x2="-45.3" y2="6.6" width="0.4064" layer="1"/>
 <wire x1="-29.24" y1="9.46" x2="-33.7" y2="5" width="0.4064" layer="16"/>
 <wire x1="-33.7" y1="5" x2="-33.7" y2="4" width="0.4064" layer="16"/>
+<contactref element="Q5" pad="G"/>
+<wire x1="-33.7" y1="4" x2="-29.24" y2="-8.34" width="0" layer="19" extent="16-16"/>
 </signal>
 <signal name="N$4">
 <contactref element="Q2" pad="3"/>
 <contactref element="Q4" pad="3"/>
-<contactref element="Q5" pad="G"/>
 <contactref element="Q9" pad="G"/>
 <wire x1="-46" y1="4" x2="-41.8" y2="4" width="0.4064" layer="16"/>
@@
 <wire x1="-48.4" y1="8.8" x2="-44.6" y2="8.8" width="0.4064" layer="16"/>
 <wire x1="-44.6" y1="8.8" x2="-41.8" y2="6" width="0.4064" layer="16"/>
-<wire x1="-39.86" y1="-8.34" x2="-29.24" y2="-8.34" width="0.4064" layer="1"/>
+<contactref element="Q6" pad="G"/>
+<wire x1="-56.2" y1="5.9" x2="-57.14" y2="-8.34" width="0" layer="19" extent="16-16"/>
 </signal>
 <signal name="N$5">
@@
 <wire x1="-40.7" y1="1.65" x2="-40.7" y2="-1.15" width="0.4064" layer="16"/>
 </signal>
-<signal name="N$2">
-<contactref element="Q1" pad="1"/>
-<contactref element="R1" pad="2"/>
-<wire x1="-32.75" y1="1.8" x2="-32.5" y2="1.55" width="0.4064" layer="16"/>
-<wire x1="-32.5" y1="1.55" x2="-29.6" y2="1.55" width="0.4064" layer="16"/>
-</signal>
-<signal name="N$3">
-<contactref element="Q2" pad="1"/>
-<contactref element="R4" pad="2"/>
-<wire x1="-45.05" y1="1.8" x2="-45.15" y2="1.7" width="0.4064" layer="16"/>
-<wire x1="-45.15" y1="1.7" x2="-45.15" y2="-3.1" width="0.4064" layer="16"/>
-</signal>
 <signal name="N$7">
 <contactref element="R2" pad="1"/>
-<contactref element="R4" pad="1"/>
-<wire x1="-43.25" y1="-3.1" x2="-43.25" y2="-5.85" width="0.4064" layer="16"/>
 <wire x1="-43.25" y1="-5.85" x2="-42" y2="-7.1" width="0.4064" layer="16"/>
 <wire x1="-42" y1="-7.1" x2="-38.2" y2="-7.1" width="0.4064" layer="16"/>
@@
 <wire x1="-28.1" y1="-17.2" x2="-38.2" y2="-7.1" width="0.4064" layer="16"/>
 <wire x1="-28.1" y1="-17.2" x2="-22.5" y2="-17.2" width="0.4064" layer="16"/>
+<contactref element="R1" pad="1"/>
+<wire x1="-29.6" y1="-0.35" x2="-36.6" y2="-2.95" width="0" layer="19" extent="16-16"/>
 </signal>
 <signal name="N$8">
-<contactref element="R1" pad="1"/>
 <contactref element="R3" pad="1"/>
 <wire x1="-40.7" y1="-3.05" x2="-40.7" y2="-4.5" width="0.4064" layer="16"/>
 <wire x1="-40.7" y1="-4.5" x2="-40.1" y2="-5.1" width="0.4064" layer="16"/>
-<wire x1="-29.6" y1="-0.35" x2="-30.45" y2="-1.2" width="0.4064" layer="16"/>
 <wire x1="-30.45" y1="-1.2" x2="-33.1" y2="-1.2" width="0.4064" layer="16"/>
 <via x="-33.1" y="-1.2" extent="1-16" drill="0.8"/>
@@
 <wire x1="-14.6" y1="-12.4" x2="-14.6" y2="-6.4" width="0.4064" layer="16"/>
 <wire x1="-14.6" y1="-6.4" x2="-20.65" y2="-0.35" width="0.4064" layer="16"/>
-<wire x1="-20.65" y1="-0.35" x2="-29.6" y2="-0.35" width="0.4064" layer="16"/>
+<contactref element="R4" pad="1"/>
+<wire x1="-40.7" y1="-3.05" x2="-43.25" y2="-3.1" width="0" layer="19" extent="16-16"/>
+<wire x1="-20.65" y1="-0.35" x2="-30.45" y2="-1.2" width="0" layer="19" extent="16-16"/>
 </signal>
 <signal name="N$10">
@@
 <signal name="N$19">
 </signal>
+<signal name="N$2">
+<contactref element="Q1" pad="1"/>
+<contactref element="R1" pad="2"/>
+<wire x1="-29.6" y1="1.55" x2="-32.75" y2="1.8" width="0" layer="19" extent="16-16"/>
+</signal>
+<signal name="N$3">
+<contactref element="R4" pad="2"/>
+<contactref element="Q2" pad="1"/>
+<wire x1="-45.05" y1="1.8" x2="-45.15" y2="-3.1" width="0" layer="19" extent="16-16"/>
+</signal>
 </signals>
