File: POVBase.sch (EAGLE design)
At the start: 25 parts, among them IC2 PIC16F876SO, Q5 IRF540, Q6 IRF540

Commit message: sdgs
Connections:
- net N$1: now also Q5.G; no longer Q6.G
- net N$4: now also Q6.G; no longer Q5.G
- net N$7: now also R1.1; no longer R4.1
- net N$8: now also R4.1; no longer R1.1
Other:
- moved on the sheet: R1, R4
Changed lines of the file:
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@@
 <instance part="P+1" gate="1" x="22.86" y="35.56"/>
 <instance part="SUPPLY1" gate="GND" x="22.86" y="25.4" rot="R180"/>
-<instance part="R1" gate="G$1" x="20.32" y="17.78" rot="R180"/>
+<instance part="R1" gate="G$1" x="12.7" y="17.78"/>
 <instance part="R2" gate="G$1" x="7.62" y="30.48" rot="R90"/>
 <instance part="R3" gate="G$1" x="38.1" y="30.48" rot="R90"/>
-<instance part="R4" gate="G$1" x="25.4" y="20.32"/>
+<instance part="R4" gate="G$1" x="33.02" y="17.78" rot="R180"/>
 <instance part="Q5" gate="G$1" x="15.24" y="48.26" smashed="yes" rot="MR270"/>
 <instance part="Q6" gate="G$1" x="30.48" y="48.26" smashed="yes" rot="R270"/>
@@
 <pinref part="Q3" gate="G$1" pin="C"/>
 <wire x1="10.16" y1="22.86" x2="10.16" y2="33.02" width="0.1524" layer="91"/>
-<wire x1="7.62" y1="63.5" x2="7.62" y2="40.64" width="0.1524" layer="91"/>
-<pinref part="Q6" gate="G$1" pin="G"/>
+<wire x1="7.62" y1="63.5" x2="7.62" y2="50.8" width="0.1524" layer="91"/>
+<wire x1="7.62" y1="50.8" x2="7.62" y2="40.64" width="0.1524" layer="91"/>
 <wire x1="7.62" y1="40.64" x2="10.16" y2="40.64" width="0.1524" layer="91"/>
-<wire x1="10.16" y1="40.64" x2="27.94" y2="40.64" width="0.1524" layer="91"/>
-<wire x1="27.94" y1="40.64" x2="27.94" y2="50.8" width="0.1524" layer="91"/>
 <wire x1="10.16" y1="33.02" x2="10.16" y2="40.64" width="0.1524" layer="91"/>
-<junction x="10.16" y="40.64"/>
 <junction x="10.16" y="33.02"/>
 <pinref part="Q7" gate="G$1" pin="G"/>
 <wire x1="7.62" y1="63.5" x2="17.78" y2="63.5" width="0.1524" layer="91"/>
+<pinref part="Q5" gate="G$1" pin="G"/>
+<wire x1="17.78" y1="50.8" x2="7.62" y2="50.8" width="0.1524" layer="91"/>
 </segment>
 </net>
 <net name="N$4" class="0">
 <segment>
-<wire x1="38.1" y1="63.5" x2="38.1" y2="53.34" width="0.1524" layer="91"/>
 <pinref part="Q2" gate="G$1" pin="C"/>
 <pinref part="Q4" gate="G$1" pin="C"/>
-<wire x1="38.1" y1="53.34" x2="38.1" y2="40.64" width="0.1524" layer="91"/>
+<wire x1="38.1" y1="63.5" x2="38.1" y2="50.8" width="0.1524" layer="91"/>
+<wire x1="38.1" y1="50.8" x2="38.1" y2="40.64" width="0.1524" layer="91"/>
 <wire x1="35.56" y1="22.86" x2="35.56" y2="33.02" width="0.1524" layer="91"/>
 <wire x1="38.1" y1="40.64" x2="35.56" y2="40.64" width="0.1524" layer="91"/>
 <wire x1="35.56" y1="40.64" x2="35.56" y2="33.02" width="0.1524" layer="91"/>
 <junction x="35.56" y="33.02"/>
-<pinref part="Q5" gate="G$1" pin="G"/>
-<wire x1="17.78" y1="50.8" x2="17.78" y2="53.34" width="0.1524" layer="91"/>
-<wire x1="17.78" y1="53.34" x2="38.1" y2="53.34" width="0.1524" layer="91"/>
-<junction x="38.1" y="53.34"/>
 <pinref part="Q9" gate="G$1" pin="G"/>
 <wire x1="27.94" y1="63.5" x2="38.1" y2="63.5" width="0.1524" layer="91"/>
+<pinref part="Q6" gate="G$1" pin="G"/>
+<wire x1="27.94" y1="50.8" x2="38.1" y2="50.8" width="0.1524" layer="91"/>
 </segment>
 </net>
@@
 </segment>
 </net>
-<net name="N$2" class="0">
-<segment>
-<pinref part="Q1" gate="G$1" pin="B"/>
-<pinref part="R1" gate="G$1" pin="2"/>
-<wire x1="15.24" y1="27.94" x2="15.24" y2="17.78" width="0.1524" layer="91"/>
-</segment>
-</net>
-<net name="N$3" class="0">
-<segment>
-<pinref part="Q2" gate="G$1" pin="B"/>
-<pinref part="R4" gate="G$1" pin="2"/>
-<wire x1="30.48" y1="27.94" x2="30.48" y2="20.32" width="0.1524" layer="91"/>
-</segment>
-</net>
 <net name="N$7" class="0">
 <segment>
 <pinref part="R2" gate="G$1" pin="1"/>
-<wire x1="7.62" y1="25.4" x2="7.62" y2="20.32" width="0.1524" layer="91"/>
-<pinref part="R4" gate="G$1" pin="1"/>
-<wire x1="7.62" y1="20.32" x2="20.32" y2="20.32" width="0.1524" layer="91"/>
-<wire x1="7.62" y1="20.32" x2="7.62" y2="12.7" width="0.1524" layer="91"/>
+<wire x1="7.62" y1="25.4" x2="7.62" y2="17.78" width="0.1524" layer="91"/>
+<wire x1="7.62" y1="17.78" x2="7.62" y2="12.7" width="0.1524" layer="91"/>
 <wire x1="7.62" y1="12.7" x2="66.04" y2="12.7" width="0.1524" layer="91"/>
 <pinref part="IC2" gate="G$1" pin="RC3/SCK"/>
 <wire x1="66.04" y1="12.7" x2="66.04" y2="27.94" width="0.1524" layer="91"/>
 <wire x1="66.04" y1="27.94" x2="114.3" y2="27.94" width="0.1524" layer="91"/>
+<pinref part="R1" gate="G$1" pin="1"/>
+<junction x="7.62" y="17.78"/>
 </segment>
 </net>
 <net name="N$8" class="0">
 <segment>
-<pinref part="R1" gate="G$1" pin="1"/>
 <pinref part="R3" gate="G$1" pin="1"/>
-<wire x1="25.4" y1="17.78" x2="38.1" y2="17.78" width="0.1524" layer="91"/>
+<wire x1="38.1" y1="15.24" x2="38.1" y2="17.78" width="0.1524" layer="91"/>
 <wire x1="38.1" y1="17.78" x2="38.1" y2="25.4" width="0.1524" layer="91"/>
-<wire x1="38.1" y1="17.78" x2="38.1" y2="15.24" width="0.1524" layer="91"/>
 <wire x1="38.1" y1="15.24" x2="63.5" y2="15.24" width="0.1524" layer="91"/>
 <wire x1="63.5" y1="15.24" x2="63.5" y2="30.48" width="0.1524" layer="91"/>
 <pinref part="IC2" gate="G$1" pin="RC2/CCP1"/>
 <wire x1="63.5" y1="30.48" x2="114.3" y2="30.48" width="0.1524" layer="91"/>
+<pinref part="R4" gate="G$1" pin="1"/>
+<junction x="38.1" y="17.78"/>
 </segment>
 </net>
@@
 </segment>
 </net>
+<net name="N$2" class="0">
+<segment>
+<pinref part="Q1" gate="G$1" pin="B"/>
+<wire x1="15.24" y1="27.94" x2="15.24" y2="20.32" width="0.1524" layer="91"/>
+<pinref part="R1" gate="G$1" pin="2"/>
+<wire x1="15.24" y1="20.32" x2="17.78" y2="20.32" width="0.1524" layer="91"/>
+<wire x1="17.78" y1="20.32" x2="17.78" y2="17.78" width="0.1524" layer="91"/>
+</segment>
+</net>
+<net name="N$3" class="0">
+<segment>
+<pinref part="R4" gate="G$1" pin="2"/>
+<wire x1="27.94" y1="17.78" x2="27.94" y2="20.32" width="0.1524" layer="91"/>
+<pinref part="Q2" gate="G$1" pin="B"/>
+<wire x1="27.94" y1="20.32" x2="30.48" y2="20.32" width="0.1524" layer="91"/>
+<wire x1="30.48" y1="20.32" x2="30.48" y2="27.94" width="0.1524" layer="91"/>
+</segment>
+</net>
