File: POVRotor.brd (EAGLE design)
At the start: 57.1 x 28 mm, 11 parts, among them IC1 LM2576S, U1 PIC32MZ2048EFH064-I/PT

Commit message: gfjfgj
Parts:
- removed JP1: (no value), pinhead:1X02
- added C3: (no value), resistor:E2,5-6E
- added C4, C5, C6, C7, C8: (no value), resistor:C0805
- added IC2: (no value), lm2576:SOT223
- added JP2: (no value), pinhead:1X05
- added R1: (no value), resistor:R0805
- added R2, R4, R5: (no value), resistor:R0603
- C1: device resistor:E5-10,5 -> resistor:E2,5-6E
- C2: device resistor:153CLV-1012 -> resistor:C0805
- moved IC1 36.0 mm to (-1.70, -15.9), flipped to the top
- moved D4 31.9 mm to (14.0, 16.1), turned to 180 degrees
- moved D3 24.9 mm to (14.0, 10.1), turned to 0 degrees
- moved D1 24.2 mm to (-11.1, -5.11), flipped to the top, turned to 180 degrees
- moved U1 22.3 mm to (-2.10, 14.7)
- moved C2 19.5 mm to (-11.2, 15.5), flipped to the top
- moved C1 19.1 mm to (-12.6, -19.8)
- moved L1 18.4 mm to (-10.7, 4.88), flipped to the top
- moved D5 15.2 mm to (18.6, 2.10), turned to 90 degrees
- moved D2 3.81 mm to (12.5, 2.10), turned to 270 degrees
Connections:
- removed net AVDD: U1.19
- removed net AVSS: U1.20
- removed net VDD: U1.26, U1.39, U1.54, U1.60, U1.8
- removed net VSS: U1.25, U1.35, U1.40, U1.55, U1.59, U1.7
- removed net VUSB3V3: U1.34
- new net +3V3: C2.1, C4.1, C5.1, C6.1, C7.1, C8.1, IC2.2, JP2.4, R1.1, R2.1, U1.19, U1.26, U1.39, U1.54, U1.60, U1.8
- new net N$12: JP2.2, U1.16
- new net N$13: JP2.1, U1.15
- new net N$14: JP2.5, R1.2, U1.9
- new net N$16: R4.2
- new net N$18: R5.2
- new net N$19: R5.1, U1.49
- new net N$21: R4.1, U1.44
- new net N$24: R2.2, U1.64
- net +15V: now also C3.+; no longer C1.+
- net +5V: now also C1.+, IC2.3; no longer C2.+
- net GND: now also C2.2, C3.-, C4.2, C5.2, C6.2, C7.2, C8.2, IC2.1, JP2.3, U1.20, U1.25, U1.34, U1.35, U1.40, U1.55, U1.59, U1.7; no longer C2.-
- net N$1: no longer JP1.2
- net N$2: no longer JP1.1
Routing:
- net GND: track 41.1 -> 189.2 mm
- net +3V3: track 0.00 -> 139.4 mm
- net N$3: track 62.6 -> 20.2 mm
- net +15V: track 27.9 -> 63.1 mm
- net +5V: track 21.9 -> 45.3 mm
- net N$23: track 0.00 -> 18.5 mm
- net N$14: track 0.00 -> 11.8 mm
- net N$13: track 0.00 -> 8.68 mm
- net N$16: track 0.00 -> 7.05 mm
- net N$12: track 0.00 -> 6.79 mm
- net N$1: track 22.0 -> 26.7 mm, vias 0 -> 1
- net N$22: track 0.00 -> 3.92 mm
- net N$21: track 0.00 -> 3.43 mm
- net N$26: track 0.00 -> 3.19 mm
- net N$24: track 0.00 -> 2.51 mm
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- added copper zone on layer 1, net GND
Other:
- board size 57.1 x 28 mm -> 56 x 85.3 mm

Commit message: asd
Parts:
- moved R5 112.0 mm to (-107.1, 35.6)
- moved R4 110.3 mm to (-103.3, 30.4)
- moved JP2 104.8 mm to (-115.4, 45.2)
- moved R2 96.0 mm to (-101.6, 43.7)
- moved R1 95.5 mm to (-107.9, 44.0)
- moved C7 77.5 mm to (-67.9, -8.00), turned to 0 degrees
- moved C6 73.9 mm to (-73.3, 0.30), turned to 90 degrees
- moved C5 68.3 mm to (-64.5, -8.00), turned to 180 degrees
- moved C8 66.1 mm to (-66.7, 7.60), turned to 0 degrees
- moved U1 64.8 mm to (-65.2, -0.20)
- moved C1 61.2 mm to (42.2, 7.40), turned to 270 degrees
- moved C4 59.2 mm to (-63.3, 7.60), turned to 180 degrees
- moved L1 58.9 mm to (48.1, 1.68)
- moved D1 58.5 mm to (47.4, -6.26), turned to 90 degrees
- moved C3 57.8 mm to (-44.9, -6.60)
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Routing:
- net +3V3: track 139.4 -> 0.00 mm
- net +5V: track 45.3 -> 118.5 mm, vias 0 -> 1
- net +15V: track 63.1 -> 115.0 mm, vias 0 -> 1
- net GND: track 189.2 -> 168.1 mm
- net N$1: track 26.7 -> 6.00 mm, vias 1 -> 0
- net N$23: track 18.5 -> 0.00 mm
- net N$2: track 20.7 -> 6.00 mm, vias 1 -> 0
- net N$14: track 11.8 -> 0.00 mm
- net N$13: track 8.68 -> 0.00 mm
- net N$16: track 7.05 -> 0.00 mm
- net N$12: track 6.79 -> 0.00 mm
- net N$3: track 20.2 -> 16.1 mm
- net N$22: track 3.92 -> 0.00 mm
- net N$21: track 3.43 -> 0.00 mm
- net N$26: track 3.19 -> 0.00 mm
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- removed copper zone on layer 1, net GND
Other:
- board size 56 x 85.3 mm -> 331.4 x 22.7 mm

Commit message: hgkjhgk
Parts:
- removed L1: (no value), rcl:6000-XXXX-RC
- added L2: (no value), resistor:L4532P
- added LED1, LED10, LED11, LED12, LED13, LED14, LED15, LED16, LED17, LED18, LED19, LED2, LED20, LED21, LED22, LED23, LED24, LED25, LED26, LED27, LED28, LED29, LED3, LED30, LED31, LED32, LED33, LED34, LED35, LED36, LED37, LED38, LED39, LED4, LED5, LED6, LED7, LED8, LED9: LP2C63-ST-RGB-SR0, led:LP2C63-ST-RGB-SR0
- moved C3 100.7 mm to (55.8, -6.20)
- moved JP2 66.3 mm to (-74.3, -6.80), turned to 0 degrees
- moved R1 65.5 mm to (-66.6, -6.80)
- moved R5 51.4 mm to (-65.2, 5.80), turned to 180 degrees
- moved R2 48.0 mm to (-81.9, -0.10), turned to 90 degrees
- moved R4 44.6 mm to (-65.2, 7.20), turned to 180 degrees
- moved C7 18.6 mm to (-50.1, -2.70), turned to 90 degrees
- moved C5 16.8 mm to (-50.1, 0.70), turned to 270 degrees
- moved C6 12.1 mm to (-63.6, -6.90)
- moved C8 9.53 mm to (-65.9, -1.90), turned to 90 degrees
- moved C2 8.70 mm to (-57.3, 7.90), turned to 180 degrees
- moved U1 7.30 mm to (-57.9, 0.00), turned to 90 degrees
- moved IC2 7.00 mm to (-45.9, 0.10)
- moved C4 6.63 mm to (-65.9, 1.50), turned to 270 degrees
- moved D2 0.40 mm to (-31.6, -5.60)
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Connections:
- removed net N$24: R2.2, U1.64
- new net N$11: LED1.4, LED1.5, LED1.6, LED15.4, LED15.5, LED15.6, LED9.4, LED9.5, LED9.6
- new net N$27: LED19.4, LED19.5, LED19.6, LED25.4, LED25.5, LED25.6, LED31.4, LED31.5, LED31.6
- new net N$28: LED20.4, LED20.5, LED20.6, LED26.4, LED26.5, LED32.4, LED32.5, LED32.6
- new net N$31: LED10.4, LED10.5, LED10.6, LED3.4, LED3.5, LED3.6, LED37.4, LED37.5, LED37.6
- new net N$38: LED11.4, LED11.5, LED11.6, LED38.4, LED38.5, LED38.6, LED5.4, LED5.5, LED5.6
- new net N$39: LED24.4, LED24.5, LED24.6, LED30.4, LED30.5, LED30.6, LED36.4, LED36.5, LED36.6
- new net N$4: LED13.4, LED13.5, LED13.6, LED2.4, LED2.5, LED2.6, LED7.4, LED7.5, LED7.6
- new net N$44: LED23.4, LED23.5, LED23.6, LED29.4, LED29.5, LED29.6, LED35.4, LED35.5, LED35.6
- new net N$45: LED1.3, LED18.3, LED19.3, LED2.3, LED20.3, LED21.3, LED22.3, LED23.3, LED24.3, LED37.3, LED38.3, LED39.3, LED4.3
- new net N$47: LED1.1, LED18.1, LED19.1, LED2.1, LED20.1, LED21.1, LED22.1, LED23.1, LED24.1, LED37.1, LED38.1, LED39.1, LED4.1
- new net N$48: LED17.3, LED26.3, LED27.3, LED28.3, LED29.3, LED3.3, LED30.3, LED5.3, LED6.3, LED8.3, LED9.3
- new net N$49: LED17.2, LED25.2, LED26.2, LED27.2, LED28.2, LED29.2, LED3.2, LED30.2, LED5.2, LED6.2, LED7.2, LED8.2, LED9.2
- new net N$5: R2.2, U1.50
- new net N$50: LED17.1, LED25.1, LED26.1, LED27.1, LED28.1, LED29.1, LED3.1, LED30.1, LED5.1, LED6.1, LED7.1, LED8.1, LED9.1
- new net N$51: LED10.1, LED11.1, LED12.1, LED13.1, LED14.1, LED15.1, LED16.1, LED31.1, LED32.1, LED33.1, LED34.1, LED35.1, LED36.1
- new net N$52: LED10.2, LED11.2, LED12.2, LED13.2, LED14.2, LED15.2, LED16.2, LED31.2, LED32.2, LED33.2, LED34.2, LED35.2, LED36.2
- new net N$53: LED10.3, LED11.3, LED12.3, LED13.3, LED14.3, LED15.3, LED16.3, LED31.3, LED32.3, LED33.3, LED34.3, LED35.3, LED36.3
- new net N$55: LED12.4, LED12.5, LED12.6, LED39.4, LED39.5, LED39.6, LED6.4, LED6.5, LED6.6
- new net N$56: LED16.4, LED16.5, LED16.6, LED17.4, LED17.5, LED17.6, LED18.4, LED18.5, LED18.6
- new net N$58: LED26.6
- new net N$61: LED21.4, LED21.5, LED21.6, LED27.4, LED27.5, LED27.6, LED33.4, LED33.5, LED33.6
- new net N$64: LED22.4, LED22.5, LED22.6, LED28.4, LED28.5, LED28.6, LED34.4, LED34.5, LED34.6
- new net N$7: LED1.2, LED18.2, LED19.2, LED2.2, LED20.2, LED21.2, LED22.2, LED23.2, LED24.2, LED37.2, LED38.2, LED39.2, LED4.2
- new net N$8: LED14.4, LED14.5, LED14.6, LED4.4, LED4.5, LED4.6, LED8.4, LED8.5, LED8.6
- net +5V: now also L2.2; no longer L1.2
- net N$3: now also L2.1; no longer L1.1
Routing:
- net +3V3: track 0.00 -> 101.9 mm
- net GND: track 168.1 -> 262.1 mm, vias 0 -> 1
- net N$12: track 0.00 -> 41.4 mm
- net N$18: track 0.00 -> 33.2 mm, vias 0 -> 1
- net N$16: track 0.00 -> 32.8 mm, vias 0 -> 1
- net N$13: track 0.00 -> 30.1 mm
- net N$5: track 0.00 -> 19.7 mm
- net N$14: track 0.00 -> 15.8 mm
- net +5V: track 118.5 -> 111.4 mm
- net N$21: track 0.00 -> 5.88 mm
- net +15V: track 115.0 -> 120.8 mm, vias 1 -> 2
- net N$19: track 0.00 -> 2.36 mm
Other:
- board size 331.4 x 22.7 mm -> 195 x 22.7 mm

Commit message: cvbn
Parts:
- removed LED1, LED10, LED11, LED12, LED13, LED14, LED15, LED16, LED17, LED18, LED19, LED2, LED20, LED21, LED22, LED23, LED24, LED25, LED26, LED27, LED28, LED29, LED3, LED30, LED31, LED32, LED33, LED34, LED35, LED36, LED37, LED38, LED39, LED4, LED5, LED6, LED7, LED8, LED9: LP2C63-ST-RGB-SR0, led:LP2C63-ST-RGB-SR0
- added U$1, U$10, U$11, U$12, U$13, U$14, U$15, U$16, U$17, U$18, U$19, U$2, U$20, U$21, U$22, U$23, U$24, U$25, U$26, U$27, U$28, U$29, U$3, U$30, U$31, U$32, U$33, U$34, U$35, U$36, U$37, U$38, U$39, U$4, U$40, U$41, U$42, U$43, U$44, U$45, U$46, U$47, U$48, U$49, U$5, U$50, U$51, U$52, U$53, U$54, U$55, U$56, U$57, U$58, U$59, U$6, U$60, U$61, U$62, U$63, U$64, U$65, U$66, U$67, U$68, U$69, U$7, U$70, U$71, U$72, U$73, U$8, U$9: 2020LED, APA2020:2020LED
- moved C6 0.61 mm to (-63.7, -6.30)
- moved R1 0.50 mm to (-66.6, -6.30)
Connections:
- removed net N$4: LED13.4, LED13.5, LED13.6, LED2.4, LED2.5, LED2.6, LED7.4, LED7.5, LED7.6
- removed net N$47: LED1.1, LED18.1, LED19.1, LED2.1, LED20.1, LED21.1, LED22.1, LED23.1, LED24.1, LED37.1, LED38.1, LED39.1, LED4.1
- removed net N$50: LED17.1, LED25.1, LED26.1, LED27.1, LED28.1, LED29.1, LED3.1, LED30.1, LED5.1, LED6.1, LED7.1, LED8.1, LED9.1
- new net N$100: U$40.SDO, U$41.SDI
- new net N$101: U$40.CLKO, U$41.CLKI
- new net N$102: U$41.SDO, U$42.SDI
- new net N$103: U$41.CLKO, U$42.CLKI
- new net N$104: U$42.SDO, U$43.SDI
- new net N$105: U$42.CLKO, U$43.CLKI
- new net N$106: U$43.SDO, U$44.SDI
- new net N$107: U$43.CLKO, U$44.CLKI
- new net N$108: U$44.SDO, U$45.SDI
- new net N$109: U$44.CLKO, U$45.CLKI
- new net N$110: U$45.SDO, U$46.SDI
- new net N$111: U$45.CLKO, U$46.CLKI
- new net N$113: U$46.SDO, U$47.SDI
- new net N$114: U$46.CLKO, U$47.CLKI
- new net N$115: U$47.SDO, U$48.SDI
- new net N$116: U$47.CLKO, U$48.CLKI
- new net N$117: U$48.SDO, U$49.SDI
- new net N$118: U$48.CLKO, U$49.CLKI
- new net N$119: U$49.SDO, U$50.SDI
- new net N$120: U$49.CLKO, U$50.CLKI
- new net N$121: U$50.SDO, U$51.SDI
- new net N$122: U$50.CLKO, U$51.CLKI
- new net N$123: U$51.SDO, U$52.SDI
- new net N$124: U$51.CLKO, U$52.CLKI
- new net N$125: U$52.SDO, U$53.SDI
- new net N$126: U$52.CLKO, U$53.CLKI
- new net N$127: U$53.SDO, U$54.SDI
- new net N$128: U$53.CLKO, U$54.CLKI
- new net N$129: U$54.SDO, U$55.SDI
- new net N$130: U$54.CLKO, U$55.CLKI
- new net N$131: U$55.SDO, U$56.SDI
- new net N$132: U$55.CLKO, U$56.CLKI
- new net N$133: U$56.SDO, U$57.SDI
- new net N$134: U$56.CLKO, U$57.CLKI
- new net N$135: U$57.SDO, U$58.SDI
- new net N$136: U$57.CLKO, U$58.CLKI
- new net N$137: U$58.SDO, U$59.SDI
- new net N$138: U$58.CLKO, U$59.CLKI
- new net N$139: U$59.SDO, U$60.SDI
- new net N$140: U$59.CLKO, U$60.CLKI
- new net N$141: U$60.SDO, U$61.SDI
- new net N$142: U$60.CLKO, U$61.CLKI
- new net N$143: U$61.SDO, U$62.SDI
- new net N$144: U$61.CLKO, U$62.CLKI
- new net N$145: U$62.SDO, U$63.SDI
- new net N$146: U$62.CLKO, U$63.CLKI
- new net N$147: U$63.SDO, U$64.SDI
- new net N$148: U$63.CLKO, U$64.CLKI
- new net N$149: U$64.SDO, U$65.SDI
- new net N$150: U$64.CLKO, U$65.CLKI
- new net N$151: U$65.SDO, U$66.SDI
- new net N$152: U$65.CLKO, U$66.CLKI
- new net N$153: U$66.SDO, U$67.SDI
- new net N$154: U$66.CLKO, U$67.CLKI
- new net N$155: U$67.SDO, U$68.SDI
- new net N$156: U$67.CLKO, U$68.CLKI
- new net N$157: U$68.SDO, U$69.SDI
- new net N$158: U$68.CLKO, U$69.CLKI
- new net N$159: U$69.SDO, U$70.SDI
- new net N$160: U$69.CLKO, U$70.CLKI
- new net N$161: U$70.SDO, U$71.SDI
- new net N$162: U$70.CLKO, U$71.CLKI
- new net N$163: U$71.SDO, U$72.SDI
- new net N$164: U$71.CLKO, U$72.CLKI
- new net N$165: U$72.SDO, U$73.SDI
- new net N$166: U$72.CLKO, U$73.CLKI
- new net N$17: U$1.SDO, U$3.SDI
- new net N$20: U$1.CLKO, U$3.CLKI
- new net N$24: U$11.CLKO, U$12.CLKI
- new net N$25: U$12.SDO, U$13.SDI
- new net N$29: U$3.SDO, U$4.SDI
- new net N$30: U$3.CLKO, U$4.CLKI
- new net N$32: U$14.SDO, U$15.SDI
- new net N$33: U$14.CLKO, U$15.CLKI
- new net N$34: U$4.SDO, U$5.SDI
- new net N$35: U$4.CLKO, U$5.CLKI
- new net N$36: U$15.SDO, U$16.SDI
- new net N$37: U$15.CLKO, U$16.CLKI
- new net N$40: U$5.SDO, U$6.SDI
- new net N$41: U$5.CLKO, U$6.CLKI
- new net N$42: U$17.SDO, U$18.SDI
- new net N$43: U$17.CLKO, U$18.CLKI
- new net N$46: U$6.SDO, U$7.SDI
- new net N$54: U$6.CLKO, U$7.CLKI
- new net N$57: U$22.CLKO, U$23.CLKI
- new net N$59: U$23.CLKO, U$24.CLKI
- new net N$6: U$1.SDI, U$2.SDO
- new net N$60: U$7.SDO, U$8.SDI
- new net N$62: U$7.CLKO, U$8.CLKI
- new net N$63: U$24.CLKO, U$25.CLKI
- new net N$65: U$25.CLKO, U$26.CLKI
- new net N$66: U$8.SDO, U$9.SDI
- new net N$67: U$8.CLKO, U$9.CLKI
- new net N$68: U$26.SDO, U$27.SDI
- new net N$69: U$26.CLKO, U$27.CLKI
- new net N$70: U$10.SDI, U$9.SDO
- new net N$71: U$10.CLKI, U$9.CLKO
- new net N$72: U$27.SDO, U$28.SDI
- new net N$73: U$27.CLKO, U$28.CLKI
- new net N$75: U$28.SDO, U$29.SDI
- new net N$76: U$28.CLKO, U$29.CLKI
- new net N$77: U$29.SDO, U$30.SDI
- new net N$78: U$29.CLKO, U$30.CLKI
- new net N$79: U$30.SDO, U$31.SDI
- new net N$80: U$30.CLKO, U$31.CLKI
- new net N$81: U$31.SDO, U$32.SDI
- new net N$82: U$31.CLKO, U$32.CLKI
- new net N$83: U$32.SDO, U$33.SDI
- new net N$84: U$32.CLKO, U$33.CLKI
- new net N$85: U$33.SDO, U$34.SDI
- new net N$86: U$33.CLKO, U$34.CLKI
- new net N$87: U$34.SDO, U$35.SDI
- new net N$88: U$34.CLKO, U$35.CLKI
- new net N$89: U$35.SDO, U$36.SDI
- new net N$9: U$1.CLKI, U$2.CLKO
- new net N$90: U$35.CLKO, U$36.CLKI
- new net N$91: U$36.SDO, U$37.SDI
- new net N$92: U$36.CLKO, U$37.CLKI
- new net N$93: U$37.SDO, U$38.SDI
- new net N$94: U$37.CLKO, U$38.CLKI
- new net N$96: U$38.SDO, U$39.SDI
- new net N$97: U$38.CLKO, U$39.CLKI
- new net N$98: U$39.SDO, U$40.SDI
- new net N$99: U$39.CLKO, U$40.CLKI
- net +5V: now also U$1.VCC, U$10.VCC, U$11.VCC, U$12.VCC, U$13.VCC, U$14.VCC, U$15.VCC, U$16.VCC, U$17.VCC, U$18.VCC, U$19.VCC, U$2.VCC, U$20.VCC, U$21.VCC, U$22.VCC, U$23.VCC, U$24.VCC, U$25.VCC, U$26.VCC, U$27.VCC, U$28.VCC, U$29.VCC, U$3.VCC, U$30.VCC, U$31.VCC, U$32.VCC, U$33.VCC, U$34.VCC, U$35.VCC, U$36.VCC, U$37.VCC, U$38.VCC, U$39.VCC, U$4.VCC, U$40.VCC, U$41.VCC, U$42.VCC, U$43.VCC, U$44.VCC, U$45.VCC, U$46.VCC, U$47.VCC, U$48.VCC, U$49.VCC, U$5.VCC, U$50.VCC, U$51.VCC, U$52.VCC, U$53.VCC, U$54.VCC, U$55.VCC, U$56.VCC, U$57.VCC, U$58.VCC, U$59.VCC, U$6.VCC, U$60.VCC, U$61.VCC, U$62.VCC, U$63.VCC, U$64.VCC, U$65.VCC, U$66.VCC, U$67.VCC, U$68.VCC, U$69.VCC, U$7.VCC, U$70.VCC, U$71.VCC, U$72.VCC, U$73.VCC, U$8.VCC, U$9.VCC
- net GND: now also U$1.GND, U$10.GND, U$11.GND, U$12.GND, U$13.GND, U$14.GND, U$15.GND, U$16.GND, U$17.GND, U$18.GND, U$19.GND, U$2.GND, U$20.GND, U$21.GND, U$22.GND, U$23.GND, U$24.GND, U$25.GND, U$26.GND, U$27.GND, U$28.GND, U$29.GND, U$3.GND, U$30.GND, U$31.GND, U$32.GND, U$33.GND, U$34.GND, U$35.GND, U$36.GND, U$37.GND, U$38.GND, U$39.GND, U$4.GND, U$40.GND, U$41.GND, U$42.GND, U$43.GND, U$44.GND, U$45.GND, U$46.GND, U$47.GND, U$48.GND, U$49.GND, U$5.GND, U$50.GND, U$51.GND, U$52.GND, U$53.GND, U$54.GND, U$55.GND, U$56.GND, U$57.GND, U$58.GND, U$59.GND, U$6.GND, U$60.GND, U$61.GND, U$62.GND, U$63.GND, U$64.GND, U$65.GND, U$66.GND, U$67.GND, U$68.GND, U$69.GND, U$7.GND, U$70.GND, U$71.GND, U$72.GND, U$73.GND, U$8.GND, U$9.GND
- net N$11: now also U$11.SDO, U$12.SDI; no longer LED1.4, LED1.5, LED1.6, LED15.4, LED15.5, LED15.6, LED9.4, LED9.5, LED9.6
- net N$16: now also U$2.SDI
- net N$18: now also U$2.CLKI
- net N$27: now also U$12.CLKO, U$13.CLKI; no longer LED19.4, LED19.5, LED19.6, LED25.4, LED25.5, LED25.6, LED31.4, LED31.5, LED31.6
- net N$28: now also U$13.SDO, U$14.SDI; no longer LED20.4, LED20.5, LED20.6, LED26.4, LED26.5, LED32.4, LED32.5, LED32.6
- net N$31: now also U$13.CLKO, U$14.CLKI; no longer LED10.4, LED10.5, LED10.6, LED3.4, LED3.5, LED3.6, LED37.4, LED37.5, LED37.6
- net N$38: now also U$16.SDO, U$17.SDI; no longer LED11.4, LED11.5, LED11.6, LED38.4, LED38.5, LED38.6, LED5.4, LED5.5, LED5.6
- net N$39: now also U$16.CLKO, U$17.CLKI; no longer LED24.4, LED24.5, LED24.6, LED30.4, LED30.5, LED30.6, LED36.4, LED36.5, LED36.6
- net N$44: now also U$18.SDO, U$19.SDI; no longer LED23.4, LED23.5, LED23.6, LED29.4, LED29.5, LED29.6, LED35.4, LED35.5, LED35.6
- net N$45: now also U$18.CLKO, U$19.CLKI; no longer LED1.3, LED18.3, LED19.3, LED2.3, LED20.3, LED21.3, LED22.3, LED23.3, LED24.3, LED37.3, LED38.3, LED39.3, LED4.3
- net N$48: now also U$19.SDO, U$20.SDI; no longer LED17.3, LED26.3, LED27.3, LED28.3, LED29.3, LED3.3, LED30.3, LED5.3, LED6.3, LED8.3, LED9.3
- net N$49: now also U$19.CLKO, U$20.CLKI; no longer LED17.2, LED25.2, LED26.2, LED27.2, LED28.2, LED29.2, LED3.2, LED30.2, LED5.2, LED6.2, LED7.2, LED8.2, LED9.2
- net N$51: now also U$20.SDO, U$21.SDI; no longer LED10.1, LED11.1, LED12.1, LED13.1, LED14.1, LED15.1, LED16.1, LED31.1, LED32.1, LED33.1, LED34.1, LED35.1, LED36.1
- net N$52: now also U$20.CLKO, U$21.CLKI; no longer LED10.2, LED11.2, LED12.2, LED13.2, LED14.2, LED15.2, LED16.2, LED31.2, LED32.2, LED33.2, LED34.2, LED35.2, LED36.2
- net N$53: now also U$21.SDO, U$22.SDI; no longer LED10.3, LED11.3, LED12.3, LED13.3, LED14.3, LED15.3, LED16.3, LED31.3, LED32.3, LED33.3, LED34.3, LED35.3, LED36.3
- net N$55: now also U$21.CLKO, U$22.CLKI; no longer LED12.4, LED12.5, LED12.6, LED39.4, LED39.5, LED39.6, LED6.4, LED6.5, LED6.6
- net N$56: now also U$22.SDO, U$23.SDI; no longer LED16.4, LED16.5, LED16.6, LED17.4, LED17.5, LED17.6, LED18.4, LED18.5, LED18.6
- net N$58: now also U$23.SDO, U$24.SDI; no longer LED26.6
- net N$61: now also U$24.SDO, U$25.SDI; no longer LED21.4, LED21.5, LED21.6, LED27.4, LED27.5, LED27.6, LED33.4, LED33.5, LED33.6
- net N$64: now also U$25.SDO, U$26.SDI; no longer LED22.4, LED22.5, LED22.6, LED28.4, LED28.5, LED28.6, LED34.4, LED34.5, LED34.6
- net N$7: now also U$10.SDO, U$11.SDI; no longer LED1.2, LED18.2, LED19.2, LED2.2, LED20.2, LED21.2, LED22.2, LED23.2, LED24.2, LED37.2, LED38.2, LED39.2, LED4.2
- net N$8: now also U$10.CLKO, U$11.CLKI; no longer LED14.4, LED14.5, LED14.6, LED4.4, LED4.5, LED4.6, LED8.4, LED8.5, LED8.6
Routing:
- net GND: track 262.1 -> 919.8 mm, vias 1 -> 2
- net +5V: track 111.4 -> 381.7 mm
- net N$16: track 32.8 -> 40.9 mm
- net N$14: track 15.8 -> 14.3 mm
- net N$13: track 30.1 -> 28.8 mm
- net N$12: track 41.4 -> 40.0 mm
- net N$9: track 0.00 -> 1.10 mm
- net N$6: track 0.00 -> 1.10 mm
- net N$8: track 0.00 -> 0.90 mm
- net N$7: track 0.00 -> 0.90 mm
- net N$67: track 0.00 -> 0.90 mm
- net N$66: track 0.00 -> 0.90 mm
- net N$62: track 0.00 -> 0.90 mm
- net N$60: track 0.00 -> 0.90 mm
- net N$52: track 0.00 -> 0.90 mm
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Other:
- board size 195 x 22.7 mm -> 195 x 22.6 mm
