File: POVRotor.sch (EAGLE design)
At the start: 11 parts, among them IC1 LM2576S, U1 PIC32MZ2048EFH064-I/PT

Commit message: gfjfgj
Parts:
- removed JP1: (no value), pinhead:PINHD-1X2
- added C3: (no value), resistor:CPOL-USE2,5-6E
- added C4, C5, C6, C7, C8: (no value), resistor:C-USC0805
- added IC2: (no value), lm2576:LM1117
- added JP2: (no value), pinhead:PINHD-1X5
- added R1: (no value), resistor:R-US_R0805
- added R2, R4, R5: (no value), resistor:R-US_R0603
- C1: device resistor:CPOL-USE5-10.5 -> resistor:CPOL-USE2,5-6E
- C2: device resistor:CPOL-US153CLV-1012 -> resistor:C-USC0805
Connections:
- new net +3V3: C2.1, C4.1, C5.1, C6.1, C7.1, C8.1, IC2.OUT, JP2.4, R1.1, R2.1, U1.AVDD, U1.VDD, U1.VDD@1, U1.VDD@2, U1.VDD@3, U1.VDD@4
- new net N$12: JP2.2, U1.PGED1/VREF+/CVREF+/AN0/RPB0/PMA6/RB0
- new net N$13: JP2.1, U1.PGEC1/VREF-/CVREF-/AN1/RPB1/RB1
- new net N$14: JP2.5, R1.2, U1.MCLR
- new net N$16: R4.2
- new net N$18: R5.2
- new net N$19: R5.1, U1.EMDIO/AEMDIO/RPD1/SCK1/RD1
- new net N$21: R4.1, U1.ECOL/RPD10/SCL1/SCK4/RD10
- new net N$24: R2.2, U1.AN18/ERXERR/PMD4/RE4
- net +15V: now also C3.+; no longer C1.+
- net +5V: now also C1.+, IC2.IN; no longer C2.+
- net GND: now also C2.2, C3.-, C4.2, C5.2, C6.2, C7.2, C8.2, IC2.GND, JP2.3, U1.AVSS, U1.VSS, U1.VSS@1, U1.VSS@2, U1.VSS@3, U1.VSS@4, U1.VSS@5, U1.VUSB3V3; no longer C2.-
- net N$1: no longer JP1.2
- net N$2: no longer JP1.1
Other:
- moved on the sheet: C1

Commit message: hgkjhgk
Parts:
- removed L1: (no value), rcl:L-US6000-XXX-RC
- added L2: (no value), resistor:L-USL4532P
- added LED1, LED10, LED11, LED12, LED13, LED14, LED15, LED16, LED17, LED18, LED19, LED2, LED20, LED21, LED22, LED23, LED24, LED25, LED26, LED27, LED28, LED29, LED3, LED30, LED31, LED32, LED33, LED34, LED35, LED36, LED37, LED38, LED39, LED4, LED5, LED6, LED7, LED8, LED9: LP2C63-ST-RGB-SR0, led:LP2C63-ST-RGB-SR0
Connections:
- removed net N$24: R2.2, U1.AN18/ERXERR/PMD4/RE4
- new net N$11: LED15B.C, LED15G.C, LED15R.C, LED1B.C, LED1G.C, LED1R.C, LED9B.C, LED9G.C, LED9R.C
- new net N$27: LED19B.C, LED19G.C, LED19R.C, LED25B.C, LED25G.C, LED25R.C, LED31B.C, LED31G.C, LED31R.C
- new net N$28: LED20B.C, LED20G.C, LED20R.C, LED26B.C, LED26R.C, LED32B.C, LED32G.C, LED32R.C
- new net N$31: LED10B.C, LED10G.C, LED10R.C, LED37B.C, LED37G.C, LED37R.C, LED3B.C, LED3G.C, LED3R.C
- new net N$38: LED11B.C, LED11G.C, LED11R.C, LED38B.C, LED38G.C, LED38R.C, LED5B.C, LED5G.C, LED5R.C
- new net N$39: LED24B.C, LED24G.C, LED24R.C, LED30B.C, LED30G.C, LED30R.C, LED36B.C, LED36G.C, LED36R.C
- new net N$4: LED13B.C, LED13G.C, LED13R.C, LED2B.C, LED2G.C, LED2R.C, LED7B.C, LED7G.C, LED7R.C
- new net N$44: LED23B.C, LED23G.C, LED23R.C, LED29B.C, LED29G.C, LED29R.C, LED35B.C, LED35G.C, LED35R.C
- new net N$45: LED18B.A, LED19B.A, LED1B.A, LED20B.A, LED21B.A, LED22B.A, LED23B.A, LED24B.A, LED2B.A, LED37B.A, LED38B.A, LED39B.A, LED4B.A
- new net N$47: LED18G.A, LED19G.A, LED1G.A, LED20G.A, LED21G.A, LED22G.A, LED23G.A, LED24G.A, LED2G.A, LED37G.A, LED38G.A, LED39G.A, LED4G.A
- new net N$48: LED17B.A, LED26B.A, LED27B.A, LED28B.A, LED29B.A, LED30B.A, LED3B.A, LED5B.A, LED6B.A, LED8B.A, LED9B.A
- new net N$49: LED17R.A, LED25R.A, LED26R.A, LED27R.A, LED28R.A, LED29R.A, LED30R.A, LED3R.A, LED5R.A, LED6R.A, LED7R.A, LED8R.A, LED9R.A
- new net N$5: R2.2, U1.ETXERR/AETXEN/RPD2/SDA3/RD2
- new net N$50: LED17G.A, LED25G.A, LED26G.A, LED27G.A, LED28G.A, LED29G.A, LED30G.A, LED3G.A, LED5G.A, LED6G.A, LED7G.A, LED8G.A, LED9G.A
- new net N$51: LED10G.A, LED11G.A, LED12G.A, LED13G.A, LED14G.A, LED15G.A, LED16G.A, LED31G.A, LED32G.A, LED33G.A, LED34G.A, LED35G.A, LED36G.A
- new net N$52: LED10R.A, LED11R.A, LED12R.A, LED13R.A, LED14R.A, LED15R.A, LED16R.A, LED31R.A, LED32R.A, LED33R.A, LED34R.A, LED35R.A, LED36R.A
- new net N$53: LED10B.A, LED11B.A, LED12B.A, LED13B.A, LED14B.A, LED15B.A, LED16B.A, LED31B.A, LED32B.A, LED33B.A, LED34B.A, LED35B.A, LED36B.A
- new net N$55: LED12B.C, LED12G.C, LED12R.C, LED39B.C, LED39G.C, LED39R.C, LED6B.C, LED6G.C, LED6R.C
- new net N$56: LED16B.C, LED16G.C, LED16R.C, LED17B.C, LED17G.C, LED17R.C, LED18B.C, LED18G.C, LED18R.C
- new net N$58: LED26G.C
- new net N$61: LED21B.C, LED21G.C, LED21R.C, LED27B.C, LED27G.C, LED27R.C, LED33B.C, LED33G.C, LED33R.C
- new net N$64: LED22B.C, LED22G.C, LED22R.C, LED28B.C, LED28G.C, LED28R.C, LED34B.C, LED34G.C, LED34R.C
- new net N$7: LED18R.A, LED19R.A, LED1R.A, LED20R.A, LED21R.A, LED22R.A, LED23R.A, LED24R.A, LED2R.A, LED37R.A, LED38R.A, LED39R.A, LED4R.A
- new net N$8: LED14B.C, LED14G.C, LED14R.C, LED4B.C, LED4G.C, LED4R.C, LED8B.C, LED8G.C, LED8R.C
- net +5V: now also L2.2; no longer L1.2
- net N$3: now also L2.1; no longer L1.1
Other:
- moved on the sheet: R2

Commit message: cvbn
Parts:
- removed LED1, LED10, LED11, LED12, LED13, LED14, LED15, LED16, LED17, LED18, LED19, LED2, LED20, LED21, LED22, LED23, LED24, LED25, LED26, LED27, LED28, LED29, LED3, LED30, LED31, LED32, LED33, LED34, LED35, LED36, LED37, LED38, LED39, LED4, LED5, LED6, LED7, LED8, LED9: LP2C63-ST-RGB-SR0, led:LP2C63-ST-RGB-SR0
- added U$1, U$10, U$11, U$12, U$13, U$14, U$15, U$16, U$17, U$18, U$19, U$2, U$20, U$21, U$22, U$23, U$24, U$25, U$26, U$27, U$28, U$29, U$3, U$30, U$31, U$32, U$33, U$34, U$35, U$36, U$37, U$38, U$39, U$4, U$40, U$41, U$42, U$43, U$44, U$45, U$46, U$47, U$48, U$49, U$5, U$50, U$51, U$52, U$53, U$54, U$55, U$56, U$57, U$58, U$59, U$6, U$60, U$61, U$62, U$63, U$64, U$65, U$66, U$67, U$68, U$69, U$7, U$70, U$71, U$72, U$73, U$8, U$9: 2020LED, APA2020:2020LED
Connections:
- removed net N$4: LED13B.C, LED13G.C, LED13R.C, LED2B.C, LED2G.C, LED2R.C, LED7B.C, LED7G.C, LED7R.C
- removed net N$47: LED18G.A, LED19G.A, LED1G.A, LED20G.A, LED21G.A, LED22G.A, LED23G.A, LED24G.A, LED2G.A, LED37G.A, LED38G.A, LED39G.A, LED4G.A
- removed net N$50: LED17G.A, LED25G.A, LED26G.A, LED27G.A, LED28G.A, LED29G.A, LED30G.A, LED3G.A, LED5G.A, LED6G.A, LED7G.A, LED8G.A, LED9G.A
- new net N$100: U$40.SDO, U$41.SDI
- new net N$101: U$40.CLKO, U$41.CLKI
- new net N$102: U$41.SDO, U$42.SDI
- new net N$103: U$41.CLKO, U$42.CLKI
- new net N$104: U$42.SDO, U$43.SDI
- new net N$105: U$42.CLKO, U$43.CLKI
- new net N$106: U$43.SDO, U$44.SDI
- new net N$107: U$43.CLKO, U$44.CLKI
- new net N$108: U$44.SDO, U$45.SDI
- new net N$109: U$44.CLKO, U$45.CLKI
- new net N$110: U$45.SDO, U$46.SDI
- new net N$111: U$45.CLKO, U$46.CLKI
- new net N$113: U$46.SDO, U$47.SDI
- new net N$114: U$46.CLKO, U$47.CLKI
- new net N$115: U$47.SDO, U$48.SDI
- new net N$116: U$47.CLKO, U$48.CLKI
- new net N$117: U$48.SDO, U$49.SDI
- new net N$118: U$48.CLKO, U$49.CLKI
- new net N$119: U$49.SDO, U$50.SDI
- new net N$120: U$49.CLKO, U$50.CLKI
- new net N$121: U$50.SDO, U$51.SDI
- new net N$122: U$50.CLKO, U$51.CLKI
- new net N$123: U$51.SDO, U$52.SDI
- new net N$124: U$51.CLKO, U$52.CLKI
- new net N$125: U$52.SDO, U$53.SDI
- new net N$126: U$52.CLKO, U$53.CLKI
- new net N$127: U$53.SDO, U$54.SDI
- new net N$128: U$53.CLKO, U$54.CLKI
- new net N$129: U$54.SDO, U$55.SDI
- new net N$130: U$54.CLKO, U$55.CLKI
- new net N$131: U$55.SDO, U$56.SDI
- new net N$132: U$55.CLKO, U$56.CLKI
- new net N$133: U$56.SDO, U$57.SDI
- new net N$134: U$56.CLKO, U$57.CLKI
- new net N$135: U$57.SDO, U$58.SDI
- new net N$136: U$57.CLKO, U$58.CLKI
- new net N$137: U$58.SDO, U$59.SDI
- new net N$138: U$58.CLKO, U$59.CLKI
- new net N$139: U$59.SDO, U$60.SDI
- new net N$140: U$59.CLKO, U$60.CLKI
- new net N$141: U$60.SDO, U$61.SDI
- new net N$142: U$60.CLKO, U$61.CLKI
- new net N$143: U$61.SDO, U$62.SDI
- new net N$144: U$61.CLKO, U$62.CLKI
- new net N$145: U$62.SDO, U$63.SDI
- new net N$146: U$62.CLKO, U$63.CLKI
- new net N$147: U$63.SDO, U$64.SDI
- new net N$148: U$63.CLKO, U$64.CLKI
- new net N$149: U$64.SDO, U$65.SDI
- new net N$150: U$64.CLKO, U$65.CLKI
- new net N$151: U$65.SDO, U$66.SDI
- new net N$152: U$65.CLKO, U$66.CLKI
- new net N$153: U$66.SDO, U$67.SDI
- new net N$154: U$66.CLKO, U$67.CLKI
- new net N$155: U$67.SDO, U$68.SDI
- new net N$156: U$67.CLKO, U$68.CLKI
- new net N$157: U$68.SDO, U$69.SDI
- new net N$158: U$68.CLKO, U$69.CLKI
- new net N$159: U$69.SDO, U$70.SDI
- new net N$160: U$69.CLKO, U$70.CLKI
- new net N$161: U$70.SDO, U$71.SDI
- new net N$162: U$70.CLKO, U$71.CLKI
- new net N$163: U$71.SDO, U$72.SDI
- new net N$164: U$71.CLKO, U$72.CLKI
- new net N$165: U$72.SDO, U$73.SDI
- new net N$166: U$72.CLKO, U$73.CLKI
- new net N$17: U$1.SDO, U$3.SDI
- new net N$20: U$1.CLKO, U$3.CLKI
- new net N$24: U$11.CLKO, U$12.CLKI
- new net N$25: U$12.SDO, U$13.SDI
- new net N$29: U$3.SDO, U$4.SDI
- new net N$30: U$3.CLKO, U$4.CLKI
- new net N$32: U$14.SDO, U$15.SDI
- new net N$33: U$14.CLKO, U$15.CLKI
- new net N$34: U$4.SDO, U$5.SDI
- new net N$35: U$4.CLKO, U$5.CLKI
- new net N$36: U$15.SDO, U$16.SDI
- new net N$37: U$15.CLKO, U$16.CLKI
- new net N$40: U$5.SDO, U$6.SDI
- new net N$41: U$5.CLKO, U$6.CLKI
- new net N$42: U$17.SDO, U$18.SDI
- new net N$43: U$17.CLKO, U$18.CLKI
- new net N$46: U$6.SDO, U$7.SDI
- new net N$54: U$6.CLKO, U$7.CLKI
- new net N$57: U$22.CLKO, U$23.CLKI
- new net N$59: U$23.CLKO, U$24.CLKI
- new net N$6: U$1.SDI, U$2.SDO
- new net N$60: U$7.SDO, U$8.SDI
- new net N$62: U$7.CLKO, U$8.CLKI
- new net N$63: U$24.CLKO, U$25.CLKI
- new net N$65: U$25.CLKO, U$26.CLKI
- new net N$66: U$8.SDO, U$9.SDI
- new net N$67: U$8.CLKO, U$9.CLKI
- new net N$68: U$26.SDO, U$27.SDI
- new net N$69: U$26.CLKO, U$27.CLKI
- new net N$70: U$10.SDI, U$9.SDO
- new net N$71: U$10.CLKI, U$9.CLKO
- new net N$72: U$27.SDO, U$28.SDI
- new net N$73: U$27.CLKO, U$28.CLKI
- new net N$75: U$28.SDO, U$29.SDI
- new net N$76: U$28.CLKO, U$29.CLKI
- new net N$77: U$29.SDO, U$30.SDI
- new net N$78: U$29.CLKO, U$30.CLKI
- new net N$79: U$30.SDO, U$31.SDI
- new net N$80: U$30.CLKO, U$31.CLKI
- new net N$81: U$31.SDO, U$32.SDI
- new net N$82: U$31.CLKO, U$32.CLKI
- new net N$83: U$32.SDO, U$33.SDI
- new net N$84: U$32.CLKO, U$33.CLKI
- new net N$85: U$33.SDO, U$34.SDI
- new net N$86: U$33.CLKO, U$34.CLKI
- new net N$87: U$34.SDO, U$35.SDI
- new net N$88: U$34.CLKO, U$35.CLKI
- new net N$89: U$35.SDO, U$36.SDI
- new net N$9: U$1.CLKI, U$2.CLKO
- new net N$90: U$35.CLKO, U$36.CLKI
- new net N$91: U$36.SDO, U$37.SDI
- new net N$92: U$36.CLKO, U$37.CLKI
- new net N$93: U$37.SDO, U$38.SDI
- new net N$94: U$37.CLKO, U$38.CLKI
- new net N$96: U$38.SDO, U$39.SDI
- new net N$97: U$38.CLKO, U$39.CLKI
- new net N$98: U$39.SDO, U$40.SDI
- new net N$99: U$39.CLKO, U$40.CLKI
- net +5V: now also U$1.VCC, U$10.VCC, U$11.VCC, U$12.VCC, U$13.VCC, U$14.VCC, U$15.VCC, U$16.VCC, U$17.VCC, U$18.VCC, U$19.VCC, U$2.VCC, U$20.VCC, U$21.VCC, U$22.VCC, U$23.VCC, U$24.VCC, U$25.VCC, U$26.VCC, U$27.VCC, U$28.VCC, U$29.VCC, U$3.VCC, U$30.VCC, U$31.VCC, U$32.VCC, U$33.VCC, U$34.VCC, U$35.VCC, U$36.VCC, U$37.VCC, U$38.VCC, U$39.VCC, U$4.VCC, U$40.VCC, U$41.VCC, U$42.VCC, U$43.VCC, U$44.VCC, U$45.VCC, U$46.VCC, U$47.VCC, U$48.VCC, U$49.VCC, U$5.VCC, U$50.VCC, U$51.VCC, U$52.VCC, U$53.VCC, U$54.VCC, U$55.VCC, U$56.VCC, U$57.VCC, U$58.VCC, U$59.VCC, U$6.VCC, U$60.VCC, U$61.VCC, U$62.VCC, U$63.VCC, U$64.VCC, U$65.VCC, U$66.VCC, U$67.VCC, U$68.VCC, U$69.VCC, U$7.VCC, U$70.VCC, U$71.VCC, U$72.VCC, U$73.VCC, U$8.VCC, U$9.VCC
- net GND: now also U$1.GND, U$10.GND, U$11.GND, U$12.GND, U$13.GND, U$14.GND, U$15.GND, U$16.GND, U$17.GND, U$18.GND, U$19.GND, U$2.GND, U$20.GND, U$21.GND, U$22.GND, U$23.GND, U$24.GND, U$25.GND, U$26.GND, U$27.GND, U$28.GND, U$29.GND, U$3.GND, U$30.GND, U$31.GND, U$32.GND, U$33.GND, U$34.GND, U$35.GND, U$36.GND, U$37.GND, U$38.GND, U$39.GND, U$4.GND, U$40.GND, U$41.GND, U$42.GND, U$43.GND, U$44.GND, U$45.GND, U$46.GND, U$47.GND, U$48.GND, U$49.GND, U$5.GND, U$50.GND, U$51.GND, U$52.GND, U$53.GND, U$54.GND, U$55.GND, U$56.GND, U$57.GND, U$58.GND, U$59.GND, U$6.GND, U$60.GND, U$61.GND, U$62.GND, U$63.GND, U$64.GND, U$65.GND, U$66.GND, U$67.GND, U$68.GND, U$69.GND, U$7.GND, U$70.GND, U$71.GND, U$72.GND, U$73.GND, U$8.GND, U$9.GND
- net N$11: now also U$11.SDO, U$12.SDI; no longer LED15B.C, LED15G.C, LED15R.C, LED1B.C, LED1G.C, LED1R.C, LED9B.C, LED9G.C, LED9R.C
- net N$16: now also U$2.SDI
- net N$18: now also U$2.CLKI
- net N$27: now also U$12.CLKO, U$13.CLKI; no longer LED19B.C, LED19G.C, LED19R.C, LED25B.C, LED25G.C, LED25R.C, LED31B.C, LED31G.C, LED31R.C
- net N$28: now also U$13.SDO, U$14.SDI; no longer LED20B.C, LED20G.C, LED20R.C, LED26B.C, LED26R.C, LED32B.C, LED32G.C, LED32R.C
- net N$31: now also U$13.CLKO, U$14.CLKI; no longer LED10B.C, LED10G.C, LED10R.C, LED37B.C, LED37G.C, LED37R.C, LED3B.C, LED3G.C, LED3R.C
- net N$38: now also U$16.SDO, U$17.SDI; no longer LED11B.C, LED11G.C, LED11R.C, LED38B.C, LED38G.C, LED38R.C, LED5B.C, LED5G.C, LED5R.C
- net N$39: now also U$16.CLKO, U$17.CLKI; no longer LED24B.C, LED24G.C, LED24R.C, LED30B.C, LED30G.C, LED30R.C, LED36B.C, LED36G.C, LED36R.C
- net N$44: now also U$18.SDO, U$19.SDI; no longer LED23B.C, LED23G.C, LED23R.C, LED29B.C, LED29G.C, LED29R.C, LED35B.C, LED35G.C, LED35R.C
- net N$45: now also U$18.CLKO, U$19.CLKI; no longer LED18B.A, LED19B.A, LED1B.A, LED20B.A, LED21B.A, LED22B.A, LED23B.A, LED24B.A, LED2B.A, LED37B.A, LED38B.A, LED39B.A, LED4B.A
- net N$48: now also U$19.SDO, U$20.SDI; no longer LED17B.A, LED26B.A, LED27B.A, LED28B.A, LED29B.A, LED30B.A, LED3B.A, LED5B.A, LED6B.A, LED8B.A, LED9B.A
- net N$49: now also U$19.CLKO, U$20.CLKI; no longer LED17R.A, LED25R.A, LED26R.A, LED27R.A, LED28R.A, LED29R.A, LED30R.A, LED3R.A, LED5R.A, LED6R.A, LED7R.A, LED8R.A, LED9R.A
- net N$51: now also U$20.SDO, U$21.SDI; no longer LED10G.A, LED11G.A, LED12G.A, LED13G.A, LED14G.A, LED15G.A, LED16G.A, LED31G.A, LED32G.A, LED33G.A, LED34G.A, LED35G.A, LED36G.A
- net N$52: now also U$20.CLKO, U$21.CLKI; no longer LED10R.A, LED11R.A, LED12R.A, LED13R.A, LED14R.A, LED15R.A, LED16R.A, LED31R.A, LED32R.A, LED33R.A, LED34R.A, LED35R.A, LED36R.A
- net N$53: now also U$21.SDO, U$22.SDI; no longer LED10B.A, LED11B.A, LED12B.A, LED13B.A, LED14B.A, LED15B.A, LED16B.A, LED31B.A, LED32B.A, LED33B.A, LED34B.A, LED35B.A, LED36B.A
- net N$55: now also U$21.CLKO, U$22.CLKI; no longer LED12B.C, LED12G.C, LED12R.C, LED39B.C, LED39G.C, LED39R.C, LED6B.C, LED6G.C, LED6R.C
- net N$56: now also U$22.SDO, U$23.SDI; no longer LED16B.C, LED16G.C, LED16R.C, LED17B.C, LED17G.C, LED17R.C, LED18B.C, LED18G.C, LED18R.C
- net N$58: now also U$23.SDO, U$24.SDI; no longer LED26G.C
- net N$61: now also U$24.SDO, U$25.SDI; no longer LED21B.C, LED21G.C, LED21R.C, LED27B.C, LED27G.C, LED27R.C, LED33B.C, LED33G.C, LED33R.C
- net N$64: now also U$25.SDO, U$26.SDI; no longer LED22B.C, LED22G.C, LED22R.C, LED28B.C, LED28G.C, LED28R.C, LED34B.C, LED34G.C, LED34R.C
- net N$7: now also U$10.SDO, U$11.SDI; no longer LED18R.A, LED19R.A, LED1R.A, LED20R.A, LED21R.A, LED22R.A, LED23R.A, LED24R.A, LED2R.A, LED37R.A, LED38R.A, LED39R.A, LED4R.A
- net N$8: now also U$10.CLKO, U$11.CLKI; no longer LED14B.C, LED14G.C, LED14R.C, LED4B.C, LED4G.C, LED4R.C, LED8B.C, LED8G.C, LED8R.C
