File: Quad/Quad.brd (EAGLE design)
At the start: 62 x 33.5 mm, 11 parts, among them U1 PIC32MZ2048EFH064-I/PT, U2 PCA9685PW,118, U3 LM2576HVS-ADJ/NOPB, U4 MPU-6050, U5 MS561101BA03-50

Commit message: dfg
Parts:
- removed LED1: RGBLED5050, adafruit:RGBLED5050
- removed XB1: XBEE-PRO, maxstream:XBEE-PRO
- added C1, C10, C12, C14, C16, C18, C27, C4, C5, C6, C7, C8, C9: 0.1uF, rcl:C0603
- added C11: 0.22uF, rcl:C0603
- added C13: 4.7uF, rcl:C0603
- added C15, C19, C20, C23: (no value), rcl:C0805
- added C17: (no value), rcl:E2-4
- added C2: 2.2nF, rcl:C0603
- added C21, C22, C24, C25, C26: (no value), rcl:B/3528-21W
- added C3: 10nF, rcl:C0603
- added JP4, JP5: (no value), pinhead:2X03
- added JP6: (no value), pinhead:1X04
- added JP7: (no value), pinhead:1X02/90
- added L1: 4.7uH, rcl:L1812
- added L3: (no value), rcl:L1812
- added LED2: RGBLED5050, adafruit:RGBLED5050
- added R1: 75k, rcl:R0603
- added R10, R11, R12, R13, R14, R17, R18, R19, R20, R7, R8: 33, rcl:R0603
- added R15, R16: 330, rcl:R0603
- added R2: 41k, rcl:R0603
- added R21: 220, rcl:R0603
- added R3: 7.6k, rcl:R0603
- added R4, R5: 4.7k, rcl:R0603
- added R6: 1k, rcl:R0603
- added R9: 22, rcl:R0603
- added T4, T5, T6: (no value), transistor:SOT23-EBC
- added U$2: AP65211A, SOT95P280X140-6N:SOT95P280X140-6N
- added U6, U7, U8: TLV75533PDBVR, TLV75533PDBVR:SOT95P280X145-5N
- added XB2: XBEE-PRO, maxstream:XBEE-PRO
- JP1: device pinhead:1X04 -> pinhead:1X06
- JP3: device pinhead:1X08 -> pinhead:1X06/90
- U2: value PCA9685PW,118 -> TLV75533PDBVR; device PCA9685PW_118:SOP65P640X110-28N -> TLV75533PDBVR:SOT95P280X145-5N
- U3: value LM2576HVS-ADJ/NOPB -> NEO-6M-GPS; device LM2576HVS-ADJ_NOPB:REG_LM2576HVS-ADJ/NOPB -> NEO-6M-GPS:XCVR_NEO-6M-GPS
- moved JP1 63.7 mm to (25.9, -32.9)
- moved U3 45.9 mm to (37.1, -18.9), turned to 0 degrees
- moved JP2 33.6 mm to (25.9, 2.70), turned to 0 degrees
- moved U$1 26.8 mm to (10.1, 7.00)
- moved JP3 26.5 mm to (59.5, 9.70), turned to 270 degrees
- moved U2 25.0 mm to (29.4, 27.8), flipped to the top
- moved U5 16.0 mm to (21.6, 21.7), turned to 0 degrees
- moved U4 7.89 mm to (22.9, 12.0)
- moved U1 5.09 mm to (39.6, 12.7), flipped to the top, turned to 180 degrees
Connections:
- removed net AVDD: U1.19
- removed net AVSS: U1.20
- removed net VDD: U1.26, U1.39, U1.54, U1.60, U1.8, U2.28, U4.13, U5.1
- removed net VLOGIC: U4.8
- removed net VSS: U1.25, U1.35, U1.40, U1.55, U1.59, U1.7
- removed net VUSB3V3: U1.34
- new net +12V: C17.+, JP7.2, U$2.3, U$2.5
- new net +3V3: C10.1, C20.1, C5.1, C6.1, C7.1, C8.1, C9.1, JP3.2, R4.2, R5.2, R6.2, U1.19, U1.26, U1.39, U1.54, U1.60, U1.8, U2.5
- new net +5V: C21.+, C24.+, C25.+, JP2.1, JP4.3, JP4.4, JP5.3, JP5.4, JP6.4, L1.2, R2.2, U2.1, U2.3, U6.1, U6.3
- new net +5V/1: C22.+, C26.+, JP1.1, LED2.1, LED2.2, LED2.3, U7.1, U7.3, U8.1, U8.3
- new net ANT: L3.2, U3.11
- new net DGND: C15.2, C18.2, C19.2, C22.-, C26.-, C27.2, JP1.2, T4.E, T5.E, T6.E, U3.10, U3.12, U3.13, U3.24, U3.7, U7.2, U8.2, XB2.10
- new net ESC_1: JP5.1, R19.2
- new net ESC_2: JP5.2, R17.2
- new net ESC_3: JP4.1, R18.2
- new net ESC_4: JP4.2, R20.2
- new net GPS_RX: JP2.3, R14.1
- new net GPS_RX_J: JP1.5, U3.21
- new net GPS_TX: JP2.4, R13.1
- new net GPS_TX_J: JP1.6, U3.20
- new net LED_BLUE: R11.2, T4.B
- new net LED_GREEN: R10.2, T5.B
- new net LED_RED: R12.2, T6.B
- new net MCLR: JP3.1, R6.1, U1.9
- new net N$1: C1.1, U4.10
- new net N$10: R1.1, U$2.4
- new net N$11: R1.2, R2.1, R3.2
- new net N$12: R7.2, U1.48
- new net N$13: R8.2, U1.47
- new net N$14: L3.1, R9.2
- new net N$16: R9.1, U3.9
- new net N$18: R13.2, U1.45
- new net N$19: R14.2, U1.44
- new net N$2: C2.1, U4.20
- new net N$20: LED2.4, R21.2
- new net N$21: R10.1, U1.17
- new net N$22: LED2.6, R15.2
- new net N$23: R17.1, U1.11
- new net N$24: R18.1, U1.13
- new net N$25: R19.1, U1.10
- new net N$26: R20.1, U1.14
- new net N$27: LED2.5, R16.2
- new net N$28: R16.1, T6.C
- new net N$29: R15.1, T5.C
- new net N$3: C11.1, U$1.8
- new net N$30: R21.1, T4.C
- new net N$4: C11.2, U$1.12
- new net N$5: R11.1, U1.30
- new net N$6: C13.1, U$1.10
- new net N$7: R12.1, U1.29
- new net N$8: C16.1, L1.1, U$2.2
- new net N$9: C16.2, U$2.6
- new net PGC: JP3.5, U1.15
- new net PGD: JP3.4, U1.16
- new net SCL: JP6.1, R4.1, U$1.1, U1.42, U4.23, U5.8
- new net SDA: JP6.2, R5.1, U$1.16, U1.41, U4.24, U5.7
- new net V+: C15.1, C18.1, C19.1, C27.1, U3.23, U7.5, U8.5, XB2.1
- new net V_BCKP: U3.22
- new net XBEE_RX: JP2.5, R8.1
- new net XBEE_RX_J: JP1.3, XB2.3
- new net XBEE_TX: JP2.6, R7.1
- new net XBEE_TX_J: JP1.4, XB2.2
- net GND: now also C1.2, C10.2, C12.2, C13.2, C14.2, C17.-, C2.2, C20.2, C21.-, C23.2, C24.-, C25.-, C3.2, C4.2, C5.2, C6.2, C7.2, C8.2, C9.2, JP2.2, JP3.3, JP4.5, JP4.6, JP5.5, JP5.6, JP6.3, JP7.1, R3.1, U$1.11, U$1.9, U$2.1, U1.20, U1.25, U1.34, U1.35, U1.40, U1.55, U1.59, U1.7, U2.2, U4.1, U4.9, U5.4, U5.5, U6.2; no longer U3.3, U3.6, U3.7, XB1.10
- net VCC: now also C12.1, C14.1, C23.1, C3.1, C4.1, U$1.13, U$1.2, U$1.4, U4.13, U4.8, U5.1, U5.2, U6.5; no longer XB1.1
Routing:
- net GND: track 0.00 -> 289.4 mm, vias 0 -> 16
- net +5V: track 0.00 -> 103.6 mm, vias 0 -> 1
- net +3V3: track 0.00 -> 90.7 mm, vias 0 -> 3
- net SCL: track 0.00 -> 73.0 mm, vias 0 -> 2
- net SDA: track 0.00 -> 70.7 mm, vias 0 -> 4
- net VCC: track 0.00 -> 65.6 mm
- net DGND: track 0.00 -> 41.8 mm, vias 0 -> 4
- net XBEE_TX_J: track 0.00 -> 38.2 mm
- net MCLR: track 0.00 -> 36.2 mm
- net XBEE_RX_J: track 0.00 -> 34.6 mm
- net V+: track 0.00 -> 18.9 mm
- net PGC: track 0.00 -> 17.7 mm, vias 0 -> 1
- net PGD: track 0.00 -> 16.4 mm, vias 0 -> 1
- net N$8: track 0.00 -> 16.0 mm
- net +5V/1: track 0.00 -> 15.0 mm
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- added copper zone on layer 1, net GND
- added copper zone on layer 16, net GND
Other:
- board size 62 x 33.5 mm -> 62 x 69.1 mm

Commit message: a
Parts:
- removed JP6: (no value), pinhead:1X04
- removed L1: 4.7uH, rcl:L1812
- removed L3: (no value), rcl:L1812
- removed LED2: RGBLED5050, adafruit:RGBLED5050
- removed U$1: HMC5883L, HMC5883L:LPCC-16
- removed U3: NEO-6M-GPS, NEO-6M-GPS:XCVR_NEO-6M-GPS
- added HMC5883: HMC5883L, HMC5883L:LPCC-16
- added JP10, JP12, JP13, JP14, JP15: (no value), pinhead:1X02
- added JP11, JP8, JP9: (no value), pinhead:1X04
- added JP16: (no value), pinhead:1X06
- added JP17: (no value), pinhead:1X04/90
- added LED: RGBLED5050, adafruit:RGBLED5050
- added PIC32MZ: PIC32MZ2048EFH064-I/PT, PIC32MZ2048EFH064-I_PT:QFP50P1200X1200X120-64N
- added R22: 22uH, rcl:R0805
- added R25, R26: 33, rcl:R0603
- added R27, R28: 330, rcl:R0603
- added R29: 220, rcl:R0603
- added UBLOX: NEO-6M-GPS, NEO-6M-GPS:XCVR_NEO-6M-GPS
- C17: device rcl:E2-4 -> rcl:C/6032-28R
- C25: value (none) -> 0.1uF; device rcl:B/3528-21W -> rcl:C0603
- JP1: device pinhead:1X06 -> pinhead:1X04
- JP2: device pinhead:1X06 -> pinhead:1X02
- R10: value 33 -> 4.7uH; device rcl:R0603 -> rcl:R0805
- R15, R16: value 330 -> 33
- R21: value 220 -> 33
- U1: value PIC32MZ2048EFH064-I/PT -> CAT24C02; device PIC32MZ2048EFH064-I_PT:QFP50P1200X1200X120-64N -> CAT24C02:SOT95P280X145-5N
- moved R3 103.1 mm to (7.10, 21.7), turned to 0 degrees
- moved R10 92.8 mm to (17.3, 26.9)
- moved R4 89.4 mm to (29.2, 19.9)
- moved R5 74.4 mm to (29.2, 17.8)
- moved C18 73.4 mm to (4.90, -6.90)
- moved C24 60.6 mm to (8.40, 19.4), turned to 0 degrees
- moved U1 48.5 mm to (8.00, -24.1), turned to 90 degrees
- moved R11 45.8 mm to (31.9, -5.40), flipped to the bottom
- moved C25 43.7 mm to (10.9, -24.0), turned to 270 degrees
- moved R12 43.4 mm to (34.5, -6.00), flipped to the bottom, turned to 270 degrees
- moved C22 42.1 mm to (27.3, -3.90), flipped to the bottom, turned to 270 degrees
- moved R16 37.3 mm to (50.1, 10.9), flipped to the bottom, turned to 270 degrees
- moved R21 37.3 mm to (48.0, 10.9), flipped to the bottom, turned to 270 degrees
- moved R15 36.3 mm to (50.1, 10.9), turned to 270 degrees
- moved C19 34.8 mm to (27.2, -13.9), flipped to the bottom, turned to 270 degrees
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- renumbered U4 to MPU6050, U5 to MS5611
Connections:
- removed net N$27: LED2.5, R16.2
- removed net N$28: R16.1, T6.C
- removed net N$29: R15.1, T5.C
- new net GPIO1: JP16.5, R16.2
- new net GPIO2: JP16.4, R21.2
- new net GPIO3: JP16.3, R26.2
- new net GPIO4: JP16.2, R15.2
- new net LED_BLUE1: R25.2, T5.B
- new net LED_GREEN1: R11.2, T4.B
- new net LED_RED1: R12.2, T6.B
- new net N$15: LED.4, R27.2
- new net N$17: JP8.2, R12.1
- new net N$31: PIC32MZ.6, R15.1
- new net N$41: JP8.1, R25.1
- new net N$42: R28.1, T6.C
- new net N$43: R29.1, T4.C
- new net N$44: R27.1, T5.C
- new net SCL_J: JP12.2, U1.1
- new net SDA_J: JP12.1, U1.3
- new net VDD: C19.1, C27.1, U8.5, UBLOX.23
- net +3V3: now also JP16.6, PIC32MZ.19, PIC32MZ.26, PIC32MZ.39, PIC32MZ.54, PIC32MZ.60, PIC32MZ.8; no longer U1.19, U1.26, U1.39, U1.54, U1.60, U1.8
- net +5V: now also JP10.1, JP17.4, R10.2; no longer C25.+, JP2.1, JP6.4, L1.2
- net +5V/1: now also JP13.1, LED.1, LED.2, LED.3; no longer JP1.1, LED2.1, LED2.2, LED2.3
- net ANT: now also R22.2, UBLOX.11; no longer L3.2, U3.11
- net DGND: now also C25.2, JP13.2, JP14.1, JP14.2, JP8.4, U1.2, UBLOX.10, UBLOX.12, UBLOX.13, UBLOX.24, UBLOX.7; no longer JP1.2, U3.10, U3.12, U3.13, U3.24, U3.7
- net GND: now also HMC5883.11, HMC5883.9, JP10.2, JP15.1, JP15.2, JP16.1, JP17.3, JP9.4, PIC32MZ.20, PIC32MZ.25, PIC32MZ.34, PIC32MZ.35, PIC32MZ.40, PIC32MZ.55, PIC32MZ.59, PIC32MZ.7; no longer C25.-, JP2.2, JP6.3, U$1.11, U$1.9, U1.20, U1.25, U1.34, U1.35, U1.40, U1.55, U1.59, U1.7
- net GPS_RX: now also JP11.1; no longer JP2.3
- net GPS_RX_J: now also JP1.3, UBLOX.21; no longer JP1.5, U3.21
- net GPS_TX: now also JP11.2; no longer JP2.4
- net GPS_TX_J: now also JP1.4, UBLOX.20; no longer JP1.6, U3.20
- net LED_BLUE: now also JP9.1, PIC32MZ.18; no longer R11.2, T4.B
- net LED_GREEN: now also JP9.3, PIC32MZ.30; no longer R10.2, T5.B
- net LED_RED: now also JP9.2, PIC32MZ.29; no longer R12.2, T6.B
- net MCLR: now also PIC32MZ.9; no longer U1.9
- net N$12: now also PIC32MZ.48; no longer U1.48
- net N$13: now also PIC32MZ.47; no longer U1.47
- net N$14: now also R22.1; no longer L3.1
- net N$16: now also UBLOX.9; no longer U3.9
- net N$18: now also PIC32MZ.45; no longer U1.45
- net N$19: now also PIC32MZ.44; no longer U1.44
- net N$20: now also JP8.3, R11.1; no longer LED2.4, R21.2
- net N$21: now also PIC32MZ.4, R16.1; no longer R10.1, U1.17
- net N$22: now also PIC32MZ.1, R21.1; no longer LED2.6, R15.2
- net N$23: now also PIC32MZ.11; no longer U1.11
- net N$24: now also PIC32MZ.13; no longer U1.13
- net N$25: now also PIC32MZ.10; no longer U1.10
- net N$26: now also PIC32MZ.14; no longer U1.14
- net N$3: now also HMC5883.8; no longer U$1.8
- net N$30: now also PIC32MZ.5, R26.1; no longer R21.1, T4.C
- net N$4: now also HMC5883.12; no longer U$1.12
- net N$5: now also LED.5, R29.2; no longer R11.1, U1.30
- net N$6: now also HMC5883.10; no longer U$1.10
- net N$7: now also LED.6, R28.2; no longer R12.1, U1.29
- net N$8: now also R10.1; no longer L1.1
- net PGC: now also PIC32MZ.15; no longer U1.15
- net PGD: now also PIC32MZ.16; no longer U1.16
- net SCL: now also HMC5883.1, JP17.1, JP2.2, PIC32MZ.42; no longer JP6.1, U$1.1, U1.42
- net SDA: now also HMC5883.16, JP17.2, JP2.1, PIC32MZ.41; no longer JP6.2, U$1.16, U1.41
- net V+: now also C25.1, U1.4; no longer C19.1, C27.1, U3.23, U8.5
- net VBUS: now also PIC32MZ.33; no longer U1.33
- net VCC: now also HMC5883.13, HMC5883.2, HMC5883.4; no longer U$1.13, U$1.2, U$1.4
- net V_BCKP: now also UBLOX.22; no longer U3.22
- net XBEE_RX: now also JP11.3; no longer JP2.5
- net XBEE_RX_J: now also JP1.1; no longer JP1.3
- net XBEE_TX: now also JP11.4; no longer JP2.6
- net XBEE_TX_J: now also JP1.2; no longer JP1.4
Routing:
- net DGND: track 41.8 -> 217.2 mm, vias 4 -> 3
- net GND: track 289.4 -> 343.9 mm, vias 16 -> 19
- net +5V/1: track 15.0 -> 67.8 mm, vias 0 -> 2
- net MCLR: track 36.2 -> 10.8 mm
- net GPS_RX_J: track 0.00 -> 21.1 mm
- net GPS_TX_J: track 0.00 -> 20.4 mm
- net +5V: track 103.6 -> 84.0 mm, vias 1 -> 2
- net GPIO1: track 0.00 -> 19.2 mm
- net LED_BLUE: track 0.00 -> 14.6 mm
- net LED_RED1: track 0.00 -> 11.3 mm, vias 0 -> 1
- net N$29: track 1.59 -> 12.8 mm
- net SCL: track 73.0 -> 62.9 mm
- net VCC: track 65.6 -> 56.0 mm
- net V+: track 18.9 -> 28.1 mm
- net LED_GREEN: track 0.07 -> 9.19 mm
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- added copper zone on layer 1, net DGND
- added copper zone on layer 16, net DGND
Other:
- board size 62 x 69.1 mm -> 62 x 67 mm
- board text added: "+"
- board text added: "+3.3"
- board text added: "+5V"
- board text added: "GND"
- board text added: "RE5"
- board text added: "RG6"
- board text added: "RG7"
- board text added: "RG8"
- board text added: "SCL"
- board text added: "SDA"
- board text added: "v4"
