File: Quad/Quad.sch (EAGLE design)
At the start: 11 parts, among them U1 PIC32MZ2048EFH064-I/PT, U2 PCA9685PW,118, U3 LM2576HVS-ADJ/NOPB, U4 MPU-6050, U5 MS561101BA03-50

Commit message: dfg
Parts:
- removed LED1: RGBLED5050, adafruit:RGBLED5050
- removed XB1: XBEE-PRO, maxstream:XBEE-PRO
- added C1, C10, C12, C14, C16, C18, C27, C4, C5, C6, C7, C8, C9: 0.1uF, rcl:C-EUC0603
- added C11: 0.22uF, rcl:C-EUC0603
- added C13: 4.7uF, rcl:C-EUC0603
- added C15, C19, C20, C23: (no value), rcl:C-USC0805
- added C17: (no value), rcl:CPOL-USE2-4
- added C2: 2.2nF, rcl:C-EUC0603
- added C21, C22, C24, C25, C26: (no value), rcl:CPOL-USB/3528-21W
- added C3: 10nF, rcl:C-EUC0603
- added JP4, JP5: (no value), pinhead:PINHD-2X3
- added JP6: (no value), pinhead:PINHD-1X4
- added JP7: (no value), pinhead:PINHD-1X2/90
- added L1: 4.7uH, rcl:L-USL1812
- added L3: (no value), rcl:L-USL1812
- added LED2: RGBLED5050, adafruit:RGBLED5050
- added R1: 75k, rcl:R-US_R0603
- added R10, R11, R12, R13, R14, R17, R18, R19, R20, R7, R8: 33, rcl:R-US_R0603
- added R15, R16: 330, rcl:R-US_R0603
- added R2: 41k, rcl:R-US_R0603
- added R21: 220, rcl:R-US_R0603
- added R3: 7.6k, rcl:R-US_R0603
- added R4, R5: 4.7k, rcl:R-US_R0603
- added R6: 1k, rcl:R-US_R0603
- added R9: 22, rcl:R-US_R0603
- added T4, T5, T6: (no value), transistor:-NPN-SOT23-EBC
- added U$2: AP65211A, SOT95P280X140-6N:AP65211A
- added U6, U7, U8: TLV75533PDBVR, TLV75533PDBVR:TLV75533PDBVR
- added XB2: XBEE-PRO, maxstream:XBEE-PRO
- JP1: device pinhead:PINHD-1X4 -> pinhead:PINHD-1X6
- JP3: device pinhead:PINHD-1X8 -> pinhead:PINHD-1X6/90
- U2: value PCA9685PW,118 -> TLV75533PDBVR; device PCA9685PW_118:PCA9685PW,118 -> TLV75533PDBVR:TLV75533PDBVR
- U3: value LM2576HVS-ADJ/NOPB -> NEO-6M-GPS; device LM2576HVS-ADJ_NOPB:LM2576HVS-ADJ/NOPB -> NEO-6M-GPS:NEO-6M-GPS
Connections:
- new net +12V: C17.+, JP7.2, U$2.EN, U$2.IN
- new net +3V3: C10.1, C20.1, C5.1, C6.1, C7.1, C8.1, C9.1, JP3.2, R4.2, R5.2, R6.2, U1.AVDD, U1.VDD, U1.VDD@1, U1.VDD@2, U1.VDD@3, U1.VDD@4, U2.OUT
- new net +5V: C21.+, C24.+, C25.+, JP2.1, JP4.3, JP4.4, JP5.3, JP5.4, JP6.4, L1.2, R2.2, U2.EN, U2.IN, U6.EN, U6.IN
- new net +5V/1: C22.+, C26.+, JP1.1, LED2.BLUE_A, LED2.GREEN_A, LED2.RED_A, U7.EN, U7.IN, U8.EN, U8.IN
- new net ANT: L3.2, U3.RF_IN
- new net DGND: C15.2, C18.2, C19.2, C22.-, C26.-, C27.2, JP1.2, T4.E, T5.E, T6.E, U3.GND, U3.VDDUSB, U7.GND, U8.GND, XB2.GND
- new net ESC_1: JP5.1, R19.2
- new net ESC_2: JP5.2, R17.2
- new net ESC_3: JP4.1, R18.2
- new net ESC_4: JP4.2, R20.2
- new net GND: C1.2, C10.2, C12.2, C13.2, C14.2, C17.-, C2.2, C20.2, C21.-, C23.2, C24.-, C25.-, C3.2, C4.2, C5.2, C6.2, C7.2, C8.2, C9.2, JP2.2, JP3.3, JP4.5, JP4.6, JP5.5, JP5.6, JP6.3, JP7.1, R3.1, U$1.GND, U$2.GND, U1.AVSS, U1.VSS, U1.VSS@1, U1.VSS@2, U1.VSS@3, U1.VSS@4, U1.VSS@5, U1.VUSB3V3, U2.GND, U4.AD0, U4.CLKIN, U4.GND, U5.!CSB, U5.GND, U6.GND
- new net GPS_RX: JP2.3, R14.1
- new net GPS_RX_J: JP1.5, U3.RXD1
- new net GPS_TX: JP2.4, R13.1
- new net GPS_TX_J: JP1.6, U3.TXD1
- new net LED_BLUE: R11.2, T4.B
- new net LED_GREEN: R10.2, T5.B
- new net LED_RED: R12.2, T6.B
- new net MCLR: JP3.1, R6.1, U1.MCLR
- new net N$1: C1.1, U4.REGOUT
- new net N$10: R1.1, U$2.FB
- new net N$11: R1.2, R2.1, R3.2
- new net N$12: R7.2, U1.SOSCO/RPC14/T1CK/RC14
- new net N$13: R8.2, U1.SOSCI/RPC13/RC13
- new net N$14: L3.1, R9.2
- new net N$16: R9.1, U3.VCC_RF
- new net N$18: R13.2, U1.AERXCLK/AEREFCLK/ECRS/RPD11/PMCS1/PMA14/RD11
- new net N$19: R14.2, U1.ECOL/RPD10/SCL1/SCK4/RD10
- new net N$2: C2.1, U4.CPOUT
- new net N$20: LED2.BLUE_C, R21.2
- new net N$21: R10.1, U1.PGEC2/AN46/RPB6/RB6
- new net N$22: LED2.GREEN_C, R15.2
- new net N$23: R17.1, U1.AN45/C1INA/RPB5/RB5
- new net N$24: R18.1, U1.AN3/C2INA/RPB3/RB3
- new net N$25: R19.1, U1.AN11/C2INC/RPG9/PMA2/RG9
- new net N$26: R20.1, U1.AN2/C2INB/RPB2/RB2
- new net N$27: LED2.RED_C, R16.2
- new net N$28: R16.1, T6.C
- new net N$29: R15.1, T5.C
- new net N$3: C11.1, U$1.SETP
- new net N$30: R21.1, T4.C
- new net N$4: C11.2, U$1.SETC
- new net N$5: R11.1, U1.AN10/EMDC/AEMDC/RPB15/OCFB/PMA0/RB15
- new net N$6: C13.1, U$1.C1
- new net N$7: R12.1, U1.AN9/RPB14/SCK3/PMA1/RB14
- new net N$8: C16.1, L1.1, U$2.SW
- new net N$9: C16.2, U$2.BST
- new net PGC: JP3.5, U1.PGEC1/VREF-/CVREF-/AN1/RPB1/RB1
- new net PGD: JP3.4, U1.PGED1/VREF+/CVREF+/AN0/RPB0/PMA6/RB0
- new net SCL: JP6.1, R4.1, U$1.SCL, U1.RPF5/SCL5/PMA8/RF5, U4.SCL, U5.SCLK
- new net SDA: JP6.2, R5.1, U$1.SDA, U1.RPF4/SDA5/PMA9/RF4, U4.SDA, U5.SDI/SDA
- new net V+: C15.1, C18.1, C19.1, C27.1, U3.VCC, U7.OUT, U8.OUT, XB2.VCC
- new net VCC: C12.1, C14.1, C23.1, C3.1, C4.1, U$1.S1, U$1.VDD, U$1.VDDIO, U4.VDD, U4.VLOGIC, U5.PS, U5.VDD, U6.OUT
- new net XBEE_RX: JP2.5, R8.1
- new net XBEE_RX_J: JP1.3, XB2.DIN/!CONFIG
- new net XBEE_TX: JP2.6, R7.1
- new net XBEE_TX_J: JP1.4, XB2.DOUT
Other:
- note added: "HMC5883 Magnetometer"
- note added: "MPU6050 Accelerometer/Gyroscope"
- note added: "MS5611 Barometer"

Commit message: a
Parts:
- removed JP6: (no value), pinhead:PINHD-1X4
- removed L1: 4.7uH, rcl:L-USL1812
- removed L3: (no value), rcl:L-USL1812
- removed LED2: RGBLED5050, adafruit:RGBLED5050
- added JP10, JP12, JP13, JP14, JP15: (no value), pinhead:PINHD-1X2
- added JP11, JP8, JP9: (no value), pinhead:PINHD-1X4
- added JP16: (no value), pinhead:PINHD-1X6
- added JP17: (no value), pinhead:PINHD-1X4/90
- added LED: RGBLED5050, adafruit:RGBLED5050
- added PIC32MZ: PIC32MZ2048EFH064-I/PT, PIC32MZ2048EFH064-I_PT:PIC32MZ2048EFH064-I/PT
- added R22: 22uH, rcl:R-EU_R0805
- added R25, R26: 33, rcl:R-US_R0603
- added R27, R28: 330, rcl:R-US_R0603
- added R29: 220, rcl:R-US_R0603
- C17: device rcl:CPOL-USE2-4 -> rcl:CPOL-USC/6032-28R
- C25: value (none) -> 0.1uF; device rcl:CPOL-USB/3528-21W -> rcl:C-EUC0603
- JP1: device pinhead:PINHD-1X6 -> pinhead:PINHD-1X4
- JP2: device pinhead:PINHD-1X6 -> pinhead:PINHD-1X2
- R10: value 33 -> 4.7uH; device rcl:R-US_R0603 -> rcl:R-EU_R0805
- R15, R16: value 330 -> 33
- R21: value 220 -> 33
- U1: value PIC32MZ2048EFH064-I/PT -> CAT24C02; device PIC32MZ2048EFH064-I_PT:PIC32MZ2048EFH064-I/PT -> CAT24C02:CAT24C02
- renumbered U$1 to HMC5883, U3 to UBLOX, U4 to MPU6050, U5 to MS5611
Connections:
- removed net N$27: LED2.RED_C, R16.2
- removed net N$28: R16.1, T6.C
- removed net N$29: R15.1, T5.C
- new net GPIO1: JP16.5, R16.2
- new net GPIO2: JP16.4, R21.2
- new net GPIO3: JP16.3, R26.2
- new net GPIO4: JP16.2, R15.2
- new net LED_BLUE1: R25.2, T5.B
- new net LED_GREEN1: R11.2, T4.B
- new net LED_RED1: R12.2, T6.B
- new net N$15: LED.BLUE_C, R27.2
- new net N$17: JP8.2, R12.1
- new net N$31: PIC32MZ.AN12/C2IND/RPG8/SCL4/PMA3/RG8, R15.1
- new net N$41: JP8.1, R25.1
- new net N$42: R28.1, T6.C
- new net N$43: R29.1, T4.C
- new net N$44: R27.1, T5.C
- new net SCL_J: JP12.2, U1.SCL
- new net SDA_J: JP12.1, U1.SDA
- new net VDD: C19.1, C27.1, U8.OUT, UBLOX.VCC
- net +3V3: now also JP16.6, PIC32MZ.AVDD, PIC32MZ.VDD, PIC32MZ.VDD@1, PIC32MZ.VDD@2, PIC32MZ.VDD@3, PIC32MZ.VDD@4; no longer U1.AVDD, U1.VDD, U1.VDD@1, U1.VDD@2, U1.VDD@3, U1.VDD@4
- net +5V: now also JP10.1, JP17.4, R10.2; no longer C25.+, JP2.1, JP6.4, L1.2
- net +5V/1: now also JP13.1, LED.BLUE_A, LED.GREEN_A, LED.RED_A; no longer JP1.1, LED2.BLUE_A, LED2.GREEN_A, LED2.RED_A
- net ANT: now also R22.2; no longer L3.2
- net DGND: now also C25.2, JP13.2, JP14.1, JP14.2, JP8.4, U1.VSS; no longer JP1.2
- net GND: now also JP10.2, JP15.1, JP15.2, JP16.1, JP17.3, JP9.4, PIC32MZ.AVSS, PIC32MZ.VSS, PIC32MZ.VSS@1, PIC32MZ.VSS@2, PIC32MZ.VSS@3, PIC32MZ.VSS@4, PIC32MZ.VSS@5, PIC32MZ.VUSB3V3; no longer C25.-, JP2.2, JP6.3, U1.AVSS, U1.VSS, U1.VSS@1, U1.VSS@2, U1.VSS@3, U1.VSS@4, U1.VSS@5, U1.VUSB3V3
- net GPS_RX: now also JP11.1; no longer JP2.3
- net GPS_RX_J: now also JP1.3; no longer JP1.5
- net GPS_TX: now also JP11.2; no longer JP2.4
- net GPS_TX_J: now also JP1.4; no longer JP1.6
- net LED_BLUE: now also JP9.1, PIC32MZ.PGED2/AN47/RPB7/RB7; no longer R11.2, T4.B
- net LED_GREEN: now also JP9.3, PIC32MZ.AN10/EMDC/AEMDC/RPB15/OCFB/PMA0/RB15; no longer R10.2, T5.B
- net LED_RED: now also JP9.2, PIC32MZ.AN9/RPB14/SCK3/PMA1/RB14; no longer R12.2, T6.B
- net MCLR: now also PIC32MZ.MCLR; no longer U1.MCLR
- net N$12: now also PIC32MZ.SOSCO/RPC14/T1CK/RC14; no longer U1.SOSCO/RPC14/T1CK/RC14
- net N$13: now also PIC32MZ.SOSCI/RPC13/RC13; no longer U1.SOSCI/RPC13/RC13
- net N$14: now also R22.1; no longer L3.1
- net N$18: now also PIC32MZ.AERXCLK/AEREFCLK/ECRS/RPD11/PMCS1/PMA14/RD11; no longer U1.AERXCLK/AEREFCLK/ECRS/RPD11/PMCS1/PMA14/RD11
- net N$19: now also PIC32MZ.ECOL/RPD10/SCL1/SCK4/RD10; no longer U1.ECOL/RPD10/SCL1/SCK4/RD10
- net N$20: now also JP8.3, R11.1; no longer LED2.BLUE_C, R21.2
- net N$21: now also PIC32MZ.AN14/C1IND/RPG6/SCK2/PMA5/RG6, R16.1; no longer R10.1, U1.PGEC2/AN46/RPB6/RB6
- net N$22: now also PIC32MZ.AN17/ETXEN/RPE5/PMD5/RE5, R21.1; no longer LED2.GREEN_C, R15.2
- net N$23: now also PIC32MZ.AN45/C1INA/RPB5/RB5; no longer U1.AN45/C1INA/RPB5/RB5
- net N$24: now also PIC32MZ.AN3/C2INA/RPB3/RB3; no longer U1.AN3/C2INA/RPB3/RB3
- net N$25: now also PIC32MZ.AN11/C2INC/RPG9/PMA2/RG9; no longer U1.AN11/C2INC/RPG9/PMA2/RG9
- net N$26: now also PIC32MZ.AN2/C2INB/RPB2/RB2; no longer U1.AN2/C2INB/RPB2/RB2
- net N$30: now also PIC32MZ.AN13/C1INC/RPG7/SDA4/PMA4/RG7, R26.1; no longer R21.1, T4.C
- net N$5: now also LED.RED_C, R29.2; no longer R11.1, U1.AN10/EMDC/AEMDC/RPB15/OCFB/PMA0/RB15
- net N$7: now also LED.GREEN_C, R28.2; no longer R12.1, U1.AN9/RPB14/SCK3/PMA1/RB14
- net N$8: now also R10.1; no longer L1.1
- net PGC: now also PIC32MZ.PGEC1/VREF-/CVREF-/AN1/RPB1/RB1; no longer U1.PGEC1/VREF-/CVREF-/AN1/RPB1/RB1
- net PGD: now also PIC32MZ.PGED1/VREF+/CVREF+/AN0/RPB0/PMA6/RB0; no longer U1.PGED1/VREF+/CVREF+/AN0/RPB0/PMA6/RB0
- net SCL: now also JP17.1, JP2.2, PIC32MZ.RPF5/SCL5/PMA8/RF5; no longer JP6.1, U1.RPF5/SCL5/PMA8/RF5
- net SDA: now also JP17.2, JP2.1, PIC32MZ.RPF4/SDA5/PMA9/RF4; no longer JP6.2, U1.RPF4/SDA5/PMA9/RF4
- net V+: now also C25.1, U1.VCC; no longer C19.1, C27.1, U8.OUT, UBLOX.VCC
- net XBEE_RX: now also JP11.3; no longer JP2.5
- net XBEE_RX_J: now also JP1.1; no longer JP1.3
- net XBEE_TX: now also JP11.4; no longer JP2.6
- net XBEE_TX_J: now also JP1.2; no longer JP1.4
Other:
- moved on the sheet: T4, T5, T6
