File: Quad/Quad-4layer.brd (EAGLE design)
At the start: 62 x 68 mm, 94 parts, among them U1 CAT24C02, U2 TLV75533PDBVR, U6 TLV75533PDBVR, U7 TLV75533PDBVR, U8 TLV75533PDBVR

Commit message: a
Parts:
- removed R22: 22uH, rcl:R0805
- removed UBLOX: NEO-6M-GPS, NEO-6M-GPS:XCVR_NEO-6M-GPS
- added C31, C33, C35: 0.1uF, rcl:C0603
- added C32: (no value), rcl:085CS_1AR
- added C34: 10uF, rcl:C1206
- added FB1: 30Ω/1.8A, SparkFun-Coils:0603
- added LED1: (no value), adafruit:CHIPLED_0603
- added SJ1, SJ2, SJ3, SJ4: (no value), jumper:SJ
- added U3: SAM-M8Q, SAM-M8Q:XCVR_SAM-M8Q
- C15, C19, C20, C23: value (none) -> 1uF
- C17: value (none) -> 0.1uF; device rcl:C/6032-28R -> rcl:C0603
- C21, C22, C24: value (none) -> 10uF; device rcl:B/3528-21W -> rcl:C1206
- C26: value (none) -> 0.1uF; device rcl:B/3528-21W -> rcl:C0603
- R9: value 22 -> 1k
- moved C17 28.6 mm to (32.1, 22.8), turned to 180 degrees
- moved C27 27.7 mm to (57.3, -20.5), flipped to the top, turned to 270 degrees
- moved R9 14.8 mm to (50.5, -8.50), flipped to the top, turned to 270 degrees
- moved C24 12.0 mm to (18.1, 26.5), turned to 270 degrees
- moved C21 8.33 mm to (28.0, 30.5), turned to 180 degrees
- moved JP10 7.90 mm to (19.0, 30.8)
- moved JP13 7.80 mm to (19.0, -3.70)
- moved R27 4.93 mm to (32.9, -11.3)
- moved L2 4.65 mm to (14.0, 28.8), turned to 270 degrees
- moved T5 4.12 mm to (35.3, -8.50), turned to 90 degrees
- moved C30 3.96 mm to (13.0, 16.8)
- moved C26 3.70 mm to (15.5, -23.1), turned to 0 degrees
- moved R3 3.62 mm to (11.0, 20.7)
- moved C14 3.61 mm to (18.3, 17.6), turned to 0 degrees
- moved R2 3.50 mm to (14.1, 21.0)
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Connections:
- removed net ANT: R22.2, UBLOX.11
- removed net V_BCKP: UBLOX.22
- new net N$29: JP4.4, SJ4.1
- new net N$39: C20.1, FB1.1, U2.5
- new net N$40: JP5.3, SJ1.1
- new net N$41: JP4.3, SJ2.1
- new net N$45: JP5.4, SJ3.1
- net +12V: now also C32.+; no longer C17.+
- net +3V3: now also C17.1, FB1.2; no longer C20.1, U2.5
- net +5V: now also C21.1, C24.1, SJ1.2, SJ2.2, SJ3.2, SJ4.2; no longer C21.+, C24.+, JP4.3, JP4.4, JP5.3, JP5.4
- net +5V/1: now also C22.1, C26.1, C34.1, C35.1; no longer C22.+, C26.+
- net DGND: now also C22.2, C26.2, C31.2, C33.2, C34.2, C35.2, LED1.C, U3.1, U3.10, U3.11, U3.15, U3.16, U3.20, U3.4, U3.5, U3.6; no longer C22.-, C26.-, UBLOX.10, UBLOX.12, UBLOX.13, UBLOX.24, UBLOX.7
- net GND: now also C17.2, C21.2, C24.2, C32.-; no longer C17.-, C21.-, C24.-
- net GPS_RX_J: now also U3.14; no longer UBLOX.21
- net GPS_TX_J: now also U3.13; no longer UBLOX.20
- net N$14: now also U3.7; no longer R22.1
- net N$16: now also LED1.A; no longer UBLOX.9
- net SCL_J: now also U3.12
- net SDA_J: now also U3.9
- net VDD: now also C31.1, C33.1, U3.17, U3.2, U3.3; no longer UBLOX.23
Routing:
- net GND: track 344.6 -> 127.9 mm, vias 19 -> 28
- net DGND: track 223.3 -> 131.0 mm, vias 6 -> 21
- net SDA_J: track 7.30 -> 59.3 mm
- net SCL_J: track 7.92 -> 56.1 mm, vias 0 -> 1
- net +5V: track 82.1 -> 39.1 mm, vias 2 -> 14
- net N$38: track 0.00 -> 12.8 mm
- net N$37: track 0.00 -> 12.8 mm
- net +3V3: track 90.0 -> 78.4 mm, vias 5 -> 0
- net VDD: track 8.61 -> 19.9 mm, vias 0 -> 8
- net ANT: track 10.2 -> 0.00 mm, vias 1 -> 0
- net +5V/1: track 73.7 -> 64.0 mm
- net SCL: track 62.9 -> 55.5 mm
- net N$29: track 12.8 -> 5.69 mm
- net SDA: track 62.9 -> 57.3 mm
- net N$45: track 0.00 -> 5.65 mm
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- added copper zone on layer 1, net +12V
- added copper zone on layer 1, net +3V3
- added copper zone on layer 15, net +5V
- added copper zone on layer 2, net DGND
- added copper zone on layer 2, net GND
- added copper zone on layer 15, net V+
- added copper zone on layer 15, net VDD
- removed copper zone on layer 16, net DGND
- removed copper zone on layer 16, net GND
- removed copper zone on layer 1, net N$8
Other:
- board text added: "5V"
- board text added: "5V jumper"
- board text added: "v5"
- board text removed: "+5V"
- board text removed: "v4"
