File: Quad/Quad-4layer.sch (EAGLE design)
At the start: 94 parts, among them U1 CAT24C02, U2 TLV75533PDBVR, U6 TLV75533PDBVR, U7 TLV75533PDBVR, U8 TLV75533PDBVR

Commit message: a
Parts:
- removed R22: 22uH, rcl:R-EU_R0805
- removed UBLOX: NEO-6M-GPS, NEO-6M-GPS:NEO-6M-GPS
- added C31, C33, C35: 0.1uF, rcl:C-EUC0603
- added C32: (no value), rcl:CPOL-US085CS-1AR
- added C34: 10uF, rcl:C-EUC1206
- added FB1: 30Ω/1.8A, SparkFun-Coils:FERRITE_BEAD-0603
- added LED1: (no value), adafruit:LEDCHIPLED_0603
- added SJ1, SJ2, SJ3, SJ4: (no value), jumper:SJ
- added U3: SAM-M8Q, SAM-M8Q:SAM-M8Q
- C15, C19, C20, C23: value (none) -> 1uF
- C17: value (none) -> 0.1uF; device rcl:CPOL-USC/6032-28R -> rcl:C-EUC0603
- C21, C22, C24: value (none) -> 10uF; device rcl:CPOL-USB/3528-21W -> rcl:C-EUC1206
- C26: value (none) -> 0.1uF; device rcl:CPOL-USB/3528-21W -> rcl:C-EUC0603
- R9: value 22 -> 1k
Connections:
- removed net ANT: R22.2, UBLOX.RF_IN
- new net N$29: JP4.4, SJ4.1
- new net N$39: C20.1, FB1.1, U2.OUT
- new net N$40: JP5.3, SJ1.1
- new net N$41: JP4.3, SJ2.1
- new net N$45: JP5.4, SJ3.1
- net +12V: now also C32.+; no longer C17.+
- net +3V3: now also C17.1, FB1.2; no longer C20.1, U2.OUT
- net +5V: now also C21.1, C24.1, SJ1.2, SJ2.2, SJ3.2, SJ4.2; no longer C21.+, C24.+, JP4.3, JP4.4, JP5.3, JP5.4
- net +5V/1: now also C22.1, C26.1, C34.1, C35.1; no longer C22.+, C26.+
- net DGND: now also C22.2, C26.2, C31.2, C33.2, C34.2, C35.2, LED1.C, U3.GND; no longer C22.-, C26.-, UBLOX.GND, UBLOX.VDDUSB
- net GND: now also C17.2, C21.2, C24.2, C32.-; no longer C17.-, C21.-, C24.-
- net GPS_RX_J: now also U3.RXD; no longer UBLOX.RXD1
- net GPS_TX_J: now also U3.TXD; no longer UBLOX.TXD1
- net N$14: now also U3.TIMEPULSE; no longer R22.1
- net N$16: now also LED1.A; no longer UBLOX.VCC_RF
- net SCL_J: now also U3.SCL
- net SDA_J: now also U3.SDA
- net VDD: now also C31.1, C33.1, U3.VCC, U3.VCC_IO, U3.V_BCKP; no longer UBLOX.VCC
Other:
- moved on the sheet: C27, R9

Commit message: sdf
Parts:
- removed JP17: (no value), pinhead:PINHD-1X4/90
- removed JP3: (no value), pinhead:PINHD-1X6/90
- added C36: 0.1uF, rcl:C-EUC0603
- added JP6: (no value), pinhead:PINHD-1X4
- added JP7: (no value), pinhead:PINHD-1X6
- C24: value 10uF -> 0.1uF; device rcl:C-EUC1206 -> rcl:C-EUC0603
Connections:
- net +3V3: now also JP7.2; no longer JP3.2, R4.2, R5.2
- net +5V: now also C36.1, JP6.4; no longer JP17.4
- net GND: now also C36.2, JP6.3, JP7.3; no longer JP17.3, JP3.3
- net MCLR: now also JP7.1; no longer JP3.1
- net PGC: now also JP7.5; no longer JP3.5
- net PGD: now also JP7.4; no longer JP3.4
- net SCL: now also JP6.1; no longer JP17.1
- net SDA: now also JP6.2; no longer JP17.2
- net VCC: now also R4.2, R5.2
Other:
- moved on the sheet: C16, C21, C28, C32, L2, R1, R2, R3, R32
