File: Quad/Quad-4layerV2.brd (EAGLE design)
At the start: 58 x 67 mm, 105 parts, among them U1 CAT24C02, U2 TLV75533PDBVR, U3 SAM-M8Q, U6 TLV75533PDBVR, U7 TLV75533PDBVR, U8 TLV75533PDBVR

Commit message: gjh
Parts:
- removed CN1: (no value), adafruit:JST-PH-2-THM-RA
- removed JP1, JP11, JP8, JP9: (no value), pinhead:1X04
- removed JP10, JP12, JP13, JP14, JP15: (no value), pinhead:1X02
- removed JP7: (no value), pinhead:1X06
- removed L2: 4.7uH, rcl:L2825P
- added PRGM: (no value), pinhead:1X06
- added R10: 4.7uH, rcl:R1210
- added VIN: (no value), adafruit:JST-PH-2-THM-RA
- C16: value 0.1uF -> 1uF
- moved R23 103.5 mm to (-73.7, 32.3)
- moved C34 93.8 mm to (-61.7, 28.9)
- moved C25 90.8 mm to (-65.6, 24.9)
- moved C15 90.4 mm to (-69.6, 22.4)
- moved C26 89.1 mm to (-62.0, 21.8)
- moved U7 84.7 mm to (-57.0, 29.0)
- moved C18 82.7 mm to (-72.8, 19.9)
- moved U1 78.2 mm to (-50.5, 27.8)
- moved U3 72.5 mm to (46.2, 55.7)
- moved LED 67.5 mm to (12.0, 48.0)
- moved C11 66.7 mm to (80.4, -14.3)
- moved C14 66.7 mm to (81.9, -2.60)
- moved C19 66.7 mm to (91.9, -33.1)
- moved C22 66.7 mm to (90.9, -23.9)
- moved C30 66.7 mm to (76.9, -3.40)
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Connections:
- removed net GPS_RX_J: JP1.3, U3.14
- removed net GPS_TX_J: JP1.4, U3.13
- removed net LED_BLUE1: JP8.1, T5.B
- removed net LED_GREEN1: JP8.2, T4.B
- removed net N$35: JP8.3, T6.B
- removed net XBEE_RX_J: JP1.2, XB2.3
- removed net XBEE_TX_J: JP1.1, XB2.2
- net +12V: now also VIN.1; no longer CN1.1
- net +3V3: now also PRGM.2; no longer JP7.2
- net +5V: now also C22.1, C26.1, C34.1, C35.1, R10.2, R23.2, R24.2, U7.1, U8.1; no longer JP10.1, L2.1
- net +5V/1: no longer C22.1, C26.1, C34.1, C35.1, JP13.1, R23.2, R24.2, U7.1, U8.1
- net DGND: no longer C15.2, C18.2, C19.2, C22.2, C25.2, C26.2, C27.2, C31.2, C33.2, C34.2, C35.2, JP13.2, JP14.1, JP14.2, JP8.4, LED1.C, U1.2, U3.1, U3.10, U3.11, U3.15, U3.16, U3.20, U3.4, U3.5, U3.6, U7.2, U8.2, XB2.10
- net GND: now also C15.2, C18.2, C19.2, C22.2, C25.2, C26.2, C27.2, C31.2, C33.2, C34.2, C35.2, LED1.C, PRGM.3, U1.2, U3.1, U3.10, U3.11, U3.15, U3.16, U3.20, U3.4, U3.5, U3.6, U7.2, U8.2, VIN.2, XB2.10; no longer CN1.2, JP10.2, JP15.1, JP15.2, JP7.3, JP9.4
- net GPS_RX: now also U3.14; no longer JP11.1
- net GPS_TX: now also U3.13; no longer JP11.2
- net LED_BLUE: now also T5.B; no longer JP9.1
- net LED_GREEN: now also T6.B; no longer JP9.3
- net LED_RED: now also T4.B; no longer JP9.2
- net MCLR: now also PRGM.1; no longer JP7.1
- net N$8: now also R10.1; no longer L2.2
- net PGC: now also PRGM.5; no longer JP7.5
- net PGD: now also PRGM.4; no longer JP7.4
- net SCL_J: no longer JP12.2, U3.12
- net SDA_J: no longer JP12.1, U3.9
- net XBEE_RX: now also XB2.3; no longer JP11.3
- net XBEE_TX: now also XB2.2; no longer JP11.4
Routing:
- net DGND: track 131.9 -> 0.00 mm, vias 21 -> 0
- net GND: track 119.1 -> 32.7 mm, vias 35 -> 1
- net +3V3: track 80.5 -> 0.00 mm, vias 8 -> 0
- net +5V/1: track 64.0 -> 0.00 mm, vias 2 -> 0
- net SDA_J: track 58.9 -> 0.00 mm
- net SCL_J: track 57.7 -> 0.00 mm, vias 1 -> 0
- net VCC: track 56.3 -> 0.00 mm, vias 1 -> 0
- net SCL: track 49.3 -> 0.00 mm, vias 3 -> 0
- net SDA: track 45.8 -> 0.00 mm, vias 2 -> 0
- net XBEE_RX_J: track 38.0 -> 0.00 mm, vias 1 -> 0
- net XBEE_TX_J: track 37.9 -> 0.00 mm
- net V+: track 30.5 -> 0.00 mm, vias 4 -> 0
- net VDD: track 19.9 -> 0.00 mm, vias 8 -> 0
- net PGC: track 19.5 -> 0.00 mm, vias 1 -> 0
- net GPS_TX_J: track 18.7 -> 0.00 mm, vias 1 -> 0
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- removed copper zone on layer 1, net +12V
- removed copper zone on layer 1, net +3V3
- removed copper zone on layer 15, net +3V3
- removed copper zone on layer 1, net +5V
- removed copper zone on layer 15, net +5V
- removed copper zone on layer 1, net DGND
- removed copper zone on layer 2, net DGND
- removed copper zone on layer 1, net GND
- removed copper zone on layer 2, net GND
- removed copper zone on layer 15, net V+
- removed copper zone on layer 15, net VDD
Other:
- board size 58 x 67 mm -> 40 x 40 mm
- board text removed: "+"
- board text removed: "+3.3"
- board text removed: "5V"
- board text removed: "5V jumper"
- board text removed: "GND"
- board text removed: "RE5"
- board text removed: "RG6"
- board text removed: "RG7"
- board text removed: "RG8"
- board text removed: "SCL"
- board text removed: "SDA"
- board text removed: "v5"
