File: POVBase/POVBase.brd (EAGLE design)
At the start: 79.6 x 79.6 mm, 29 parts, among them IC1 LM2576S, IC2 PIC16F876SO, Q5 IRF540, Q6 IRF540, T2 2SC1306

Commit message: a
Routing:
- net +12V: track 168.0 -> 188.5 mm
- net GND: track 225.7 -> 215.6 mm
- added copper zone on layer 16, net +12V
Changed lines of the file:
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@@
 <?xml version="1.0" encoding="utf-8"?>
 <!DOCTYPE eagle SYSTEM "eagle.dtd">
-<eagle version="8.6.3">
+<eagle version="9.4.2">
 <drawing>
 <settings>
@@
 <layer number="23" name="tOrigins" color="15" fill="1" visible="yes" active="yes"/>
 <layer number="24" name="bOrigins" color="15" fill="1" visible="yes" active="yes"/>
-<layer number="25" name="tNames" color="7" fill="1" visible="yes" active="yes"/>
-<layer number="26" name="bNames" color="7" fill="1" visible="yes" active="yes"/>
-<layer number="27" name="tValues" color="7" fill="1" visible="yes" active="yes"/>
-<layer number="28" name="bValues" color="7" fill="1" visible="yes" active="yes"/>
-<layer number="29" name="tStop" color="7" fill="3" visible="yes" active="yes"/>
-<layer number="30" name="bStop" color="7" fill="6" visible="yes" active="yes"/>
-<layer number="31" name="tCream" color="7" fill="4" visible="yes" active="yes"/>
-<layer number="32" name="bCream" color="7" fill="5" visible="yes" active="yes"/>
-<layer number="33" name="tFinish" color="6" fill="3" visible="yes" active="yes"/>
-<layer number="34" name="bFinish" color="6" fill="6" visible="yes" active="yes"/>
-<layer number="35" name="tGlue" color="7" fill="4" visible="yes" active="yes"/>
-<layer number="36" name="bGlue" color="7" fill="5" visible="yes" active="yes"/>
-<layer number="37" name="tTest" color="7" fill="1" visible="yes" active="yes"/>
-<layer number="38" name="bTest" color="7" fill="1" visible="yes" active="yes"/>
-<layer number="39" name="tKeepout" color="4" fill="11" visible="yes" active="yes"/>
-<layer number="40" name="bKeepout" color="1" fill="11" visible="yes" active="yes"/>
-<layer number="41" name="tRestrict" color="4" fill="10" visible="yes" active="yes"/>
-<layer number="42" name="bRestrict" color="1" fill="10" visible="yes" active="yes"/>
-<layer number="43" name="vRestrict" color="2" fill="10" visible="yes" active="yes"/>
-<layer number="44" name="Drills" color="7" fill="1" visible="yes" active="yes"/>
-<layer number="45" name="Holes" color="7" fill="1" visible="yes" active="yes"/>
-<layer number="46" name="Milling" color="3" fill="1" visible="yes" active="yes"/>
-<layer number="47" name="Measures" color="7" fill="1" visible="yes" active="yes"/>
-<layer number="48" name="Document" color="7" fill="1" visible="yes" active="yes"/>
-<layer number="49" name="Reference" color="7" fill="1" visible="yes" active="yes"/>
-<layer number="50" name="dxf" color="7" fill="1" visible="yes" active="yes"/>
+<layer number="25" name="tNames" color="7" fill="1" visible="no" active="yes"/>
+<layer number="26" name="bNames" color="7" fill="1" visible="no" active="yes"/>
+<layer number="27" name="tValues" color="7" fill="1" visible="no" active="yes"/>
+<layer number="28" name="bValues" color="7" fill="1" visible="no" active="yes"/>
+<layer number="29" name="tStop" color="7" fill="3" visible="no" active="yes"/>
+<layer number="30" name="bStop" color="7" fill="6" visible="no" active="yes"/>
+<layer number="31" name="tCream" color="7" fill="4" visible="no" active="yes"/>
+<layer number="32" name="bCream" color="7" fill="5" visible="no" active="yes"/>
+<layer number="33" name="tFinish" color="6" fill="3" visible="no" active="yes"/>
+<layer number="34" name="bFinish" color="6" fill="6" visible="no" active="yes"/>
+<layer number="35" name="tGlue" color="7" fill="4" visible="no" active="yes"/>
+<layer number="36" name="bGlue" color="7" fill="5" visible="no" active="yes"/>
+<layer number="37" name="tTest" color="7" fill="1" visible="no" active="yes"/>
+<layer number="38" name="bTest" color="7" fill="1" visible="no" active="yes"/>
+<layer number="39" name="tKeepout" color="4" fill="11" visible="no" active="yes"/>
+<layer number="40" name="bKeepout" color="1" fill="11" visible="no" active="yes"/>
+<layer number="41" name="tRestrict" color="4" fill="10" visible="no" active="yes"/>
+<layer number="42" name="bRestrict" color="1" fill="10" visible="no" active="yes"/>
+<layer number="43" name="vRestrict" color="2" fill="10" visible="no" active="yes"/>
+<layer number="44" name="Drills" color="7" fill="1" visible="no" active="yes"/>
+<layer number="45" name="Holes" color="7" fill="1" visible="no" active="yes"/>
+<layer number="46" name="Milling" color="3" fill="1" visible="no" active="yes"/>
+<layer number="47" name="Measures" color="7" fill="1" visible="no" active="yes"/>
+<layer number="48" name="Document" color="7" fill="1" visible="no" active="yes"/>
+<layer number="49" name="Reference" color="7" fill="1" visible="no" active="yes"/>
+<layer number="50" name="dxf" color="7" fill="1" visible="no" active="yes"/>
 <layer number="51" name="tDocu" color="7" fill="1" visible="yes" active="yes"/>
 <layer number="52" name="bDocu" color="7" fill="1" visible="yes" active="yes"/>
@@
 <layer number="98" name="Guide" color="6" fill="1" visible="no" active="no"/>
 <layer number="99" name="SpiceOrder" color="5" fill="1" visible="no" active="no"/>
-<layer number="200" name="200bmp" color="7" fill="1" visible="yes" active="yes"/>
-<layer number="231" name="Eagle3D_PG1" color="7" fill="1" visible="yes" active="yes"/>
-<layer number="232" name="Eagle3D_PG2" color="7" fill="1" visible="yes" active="yes"/>
-<layer number="233" name="Eagle3D_PG3" color="7" fill="1" visible="yes" active="yes"/>
-<layer number="250" name="Descript" color="7" fill="1" visible="yes" active="yes"/>
-<layer number="251" name="SMDround" color="7" fill="1" visible="yes" active="yes"/>
+<layer number="200" name="200bmp" color="7" fill="1" visible="no" active="yes"/>
+<layer number="231" name="Eagle3D_PG1" color="7" fill="1" visible="no" active="yes"/>
+<layer number="232" name="Eagle3D_PG2" color="7" fill="1" visible="no" active="yes"/>
+<layer number="233" name="Eagle3D_PG3" color="7" fill="1" visible="no" active="yes"/>
+<layer number="250" name="Descript" color="7" fill="1" visible="no" active="yes"/>
+<layer number="251" name="SMDround" color="7" fill="1" visible="no" active="yes"/>
 </layers>
 <board>
@@
 <param name="checkStop" value="0"/>
 <param name="checkValues" value="0"/>
+<param name="checkNames" value="1"/>
+<param name="checkWireStubs" value="1"/>
+<param name="checkPolygonWidth" value="0"/>
 <param name="useDiameter" value="13"/>
 <param name="maxErrors" value="50"/>
@@
 <wire x1="12.8" y1="34.2" x2="-10.5" y2="34.2" width="0.254" layer="16"/>
 <wire x1="-10.5" y1="34.2" x2="-12.407896875" y2="32.292103125" width="0.254" layer="16"/>
+<polygon width="0.15" layer="16">
+<vertex x="-18" y="3"/>
+<vertex x="-22" y="3"/>
+<vertex x="-22" y="-3"/>
+<vertex x="-18" y="-3"/>
+</polygon>
+<wire x1="-16.407896875" y1="20" x2="-15.3" y2="18.892103125" width="0.8128" layer="16"/>
+<wire x1="-19.5" y1="12.5" x2="-19.5" y2="1.7" width="0.8128" layer="16"/>
+<wire x1="-15.3" y1="18.892103125" x2="-15.3" y2="16.7" width="0.8128" layer="16"/>
+<wire x1="-15.3" y1="16.7" x2="-19.5" y2="12.5" width="0.8128" layer="16"/>
 </signal>
 <signal name="GND">
@@
 <contactref element="C4" pad="-"/>
 <wire x1="-3.8" y1="23.63" x2="-6" y2="25.83" width="0.4064" layer="1"/>
-<polygon width="0.15" layer="16">
-<vertex x="-18" y="3"/>
-<vertex x="-22" y="3"/>
-<vertex x="-22" y="-3"/>
-<vertex x="-18" y="-3"/>
-</polygon>
 <wire x1="-31.2" y1="11.3" x2="-31.2" y2="3.81" width="0.4064" layer="1"/>
 <wire x1="-12.95" y1="29.55" x2="-31.2" y2="11.3" width="0.4064" layer="1"/>
@@
 <wire x1="29.16" y1="2.54" x2="27.94" y2="2.54" width="0.254" layer="1"/>
 <wire x1="-31.2" y1="3.81" x2="-24.4" y2="3.81" width="0.254" layer="1"/>
-<wire x1="-24.4" y1="3.81" x2="-21.89" y2="3.81" width="0.254" layer="1"/>
-<wire x1="-21.89" y1="3.81" x2="-20.9" y2="4.8" width="0.254" layer="1"/>
-<via x="-20.9" y="4.8" extent="1-16" drill="0.6"/>
+<wire x1="-24.4" y1="3.81" x2="-22.79" y2="3.81" width="0.254" layer="1"/>
+<wire x1="-22.79" y1="3.81" x2="-21.8" y2="4.8" width="0.254" layer="1"/>
+<via x="-21.8" y="4.8" extent="1-16" drill="0.6"/>
 <wire x1="-24.4" y1="3.81" x2="-24.4" y2="0.9" width="0.254" layer="1"/>
-<wire x1="-20.9" y1="4.8" x2="-20.4" y2="4.3" width="0.4064" layer="16"/>
-<wire x1="-20.4" y1="4.3" x2="-20.4" y2="-4.2" width="0.4064" layer="16"/>
 <wire x1="15.3" y1="-18.892103125" x2="16.407896875" y2="-20" width="0.4064" layer="1"/>
 <wire x1="20" y1="2.54" x2="20" y2="-11.8" width="0.4064" layer="1"/>
@@
 </signal>
 </signals>
+<mfgpreviewcolors>
+<mfgpreviewcolor name="soldermaskcolor" color="0xC8008000"/>
+<mfgpreviewcolor name="silkscreencolor" color="0xFFFEFEFE"/>
+<mfgpreviewcolor name="backgroundcolor" color="0xFF282828"/>
+<mfgpreviewcolor name="coppercolor" color="0xFFFFBF00"/>
+<mfgpreviewcolor name="substratecolor" color="0xFF786E46"/>
+</mfgpreviewcolors>
 <errors>
 </errors>
