File: POVBaseV2/POVBase.brd (EAGLE design)
At the start: 36 x 36 mm, 50 parts, among them J1 MEM2075-00-140-01-A, U1 ZXGD3005E6TA, U2 ZXGD3005E6TA, U3 ZXGD3005E6TA, U4 ZXGD3005E6TA, U5 TLV75533PDBVR

Commit message: a
Parts:
- added R19, R21, R22, R23: (no value), rcl:R0603
- added T2, T6, T7, T8: (no value), transistor:SOT23-EBC
- moved C11 195.2 mm to (41.8, 17.1)
- moved C20 144.6 mm to (21.0, 20.1), turned to 270 degrees
- moved C17 143.7 mm to (33.3, 25.2)
- moved C21 142.4 mm to (25.1, 25.5)
- moved C7 94.0 mm to (-15.4, -1.20), turned to 90 degrees
- moved R13 91.0 mm to (-29.3, 0.10), turned to 90 degrees
- moved R10 88.9 mm to (-24.2, 0.10), turned to 90 degrees
- moved R8 85.5 mm to (-21.9, 0.10), turned to 90 degrees
- moved U4 84.0 mm to (-28.1, -4.70), turned to 90 degrees
- moved C8 77.3 mm to (-12.6, -5.10), turned to 270 degrees
- moved U3 76.5 mm to (-23.1, -4.70), turned to 90 degrees
- moved R12 74.0 mm to (-27.0, 0.10), turned to 90 degrees
- moved R11 73.9 mm to (-22.9, -8.10)
- moved R3 70.7 mm to (-20.2, -18.4), turned to 90 degrees
- moved R4 68.5 mm to (-28.9, -21.7), turned to 180 degrees
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Connections:
- removed net +12V1: C7.2, U3.1
- removed net +12V2: C8.2, U4.1
- removed net +12V3: C9.2, U2.1
- new net +24V: C7.2, C8.2, U3.1, U4.1
- new net IN_H1_R: R11.1, T6.C
- new net IN_H2_R: R14.1, T2.C
- new net IN_L1_R: R3.1, T7.C
- new net IN_L2_R: R7.1, T8.C
- new net N$14: R19.1, T2.B
- new net N$15: R21.1, T6.B
- new net N$24: R22.1, T7.B
- new net N$25: R23.1, T8.B
- net +12V: now also C9.2, U2.1
- net GND: now also T2.E, T6.E, T7.E, T8.E
- net IN_H1: now also R21.2; no longer R11.1
- net IN_H2: now also R19.2; no longer R14.1
- net IN_L1: now also R22.2; no longer R3.1
- net IN_L2: now also R23.2; no longer R7.1
Routing:
- net GND: track 118.9 -> 242.4 mm, vias 13 -> 21
- net +12V: track 105.1 -> 186.2 mm, vias 20 -> 22
- net GATE_H2: track 53.9 -> 27.5 mm, vias 0 -> 2
- net GATE_H1: track 39.5 -> 21.5 mm, vias 0 -> 2
- net N$14: track 0.00 -> 15.5 mm
- net N$15: track 0.00 -> 10.6 mm
- net N$24: track 0.00 -> 3.18 mm
- net N$1: track 0.00 -> 3.12 mm
- net GATE_L2: track 25.1 -> 28.2 mm
- net GATE_L1: track 10.4 -> 13.5 mm
- net N$6: track 0.00 -> 2.87 mm
- net N$9: track 0.00 -> 2.54 mm
- net +3V3: track 107.5 -> 109.9 mm
- net N$23: track 0.00 -> 2.40 mm
- net N$25: track 0.00 -> 2.29 mm
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
Commit message: a
Parts:
- added C12: 0.047uF, rcl:C0603
- added C13: 100pF, rcl:C0603
- added C14: 0.1uF, rcl:C0603
- added C15, C18, C19: 4.7uF, rcl:C0805
- added D1: GF1, diode:SMA-DO214AC
- added L1: 10uH, rcl:POWER-CHOKE_WE-TPC
- added R24, R25: 2.55k, rcl:R0603
- added R26, R27: 10k, rcl:R0603
- added R28: 187k, rcl:R0603
- added U6: TPS55340RTER, TPS55340RTER:QFN50P300X300X100-17N
- moved C17 26.2 mm to (7.20, 22.5), turned to 270 degrees
- moved C8 18.1 mm to (-30.7, -6.00), turned to 90 degrees
- moved C11 11.2 mm to (31.1, 13.8)
- moved C7 10.2 mm to (-25.6, -2.00), turned to 270 degrees
- moved C21 4.47 mm to (21.1, 23.5), turned to 180 degrees
- moved C16 4.10 mm to (12.3, 23.3)
- moved C20 4.10 mm to (25.1, 20.1)
- moved R15 4.10 mm to (16.6, 20.8)
- moved R16 4.10 mm to (17.6, 18.2)
- moved R9 4.10 mm to (12.3, 18.4)
- moved R17 4.10 mm to (12.4, 25.1)
- moved R18 4.10 mm to (18.2, 20.8)
- moved R5 4.10 mm to (15.0, 19.0)
- moved U$2 4.10 mm to (12.2, 20.8)
- moved U5 4.10 mm to (21.9, 20.4)
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Connections:
- removed net SHIELD: J1.SH1, J1.SH2, J1.SH3, J1.SH4
- new net BST_COMP: C13.1, R24.2, U6.7
- new net BST_COMP_R: C14.1, R24.1
- new net BST_EN: R26.1, U6.3
- new net BST_FB: R27.1, R28.2, U6.8
- new net BST_FREQ: R25.1, U6.9
- new net BST_SS: C12.1, U6.4
- new net BST_SW: D1.A, L1.2, U6.1, U6.15, U6.16
- net +12V: now also L1.1, R26.2, U6.2
- net +24V: now also C15.1, C18.1, C19.1, D1.K, R28.1
- net GND: now also C12.2, C13.2, C14.2, C15.2, C18.2, C19.2, J1.SH1, J1.SH2, J1.SH3, J1.SH4, R25.2, R27.2, U6.11, U6.12, U6.13, U6.17, U6.5, U6.6
Routing:
- net GND: track 242.4 -> 298.3 mm, vias 21 -> 26
- net +24V: track 0.00 -> 38.0 mm
- net +12V: track 186.2 -> 207.9 mm, vias 22 -> 28
- net BST_SW: track 0.00 -> 9.22 mm
- net BST_COMP: track 0.00 -> 6.04 mm, vias 0 -> 1
- net BST_FB: track 0.00 -> 4.01 mm
- net BST_SS: track 0.00 -> 2.58 mm
- net +5V: track 9.70 -> 11.6 mm
- net BST_EN: track 0.00 -> 1.78 mm
- net +3V3: track 109.9 -> 108.2 mm
- net BST_COMP_R: track 0.00 -> 1.67 mm
- net BST_FREQ: track 0.00 -> 1.51 mm

Commit message: a
Parts:
- removed JP1, JP4: (no value), pinhead:1X01
- added R29, R31: 90k, rcl:R0603
- added R30, R32: 10k, rcl:R0603
- added R33, R35: 45k, rcl:R0603
- added R34, R36: 5k, rcl:R0603
- added R37, R38, R39, R40: (no value), rcl:R0603
- moved C11 25.0 mm to (48.5, -4.10), flipped to the bottom, turned to 180 degrees
- moved R21 5.80 mm to (-17.3, -12.2)
- moved R19 5.59 mm to (-17.3, -14.1)
- moved R4 2.70 mm to (-28.8, -19.0)
- moved R6 2.70 mm to (-28.8, -21.3)
- moved R2 2.70 mm to (-28.9, -16.7)
- moved U1 2.60 mm to (-24.4, -15.7)
- moved R1 2.60 mm to (-28.9, -14.5)
- moved U2 2.30 mm to (-24.4, -20.2)
- moved R3 2.11 mm to (-18.4, -17.3)
- moved R11 1.97 mm to (-21.2, -9.10), turned to 90 degrees
- moved R23 1.70 mm to (-11.9, -22.2)
- moved T7 1.65 mm to (-15.7, -18.1)
- moved T8 1.61 mm to (-15.7, -21.5)
- moved R14 1.56 mm to (-29.2, -9.20), turned to 90 degrees
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Connections:
- new net N$26: R29.1, R30.2
- new net N$27: R31.1, R32.2
- new net N$28: R33.1, R34.2
- new net N$29: R35.1, R36.2
- net +12V: now also R37.2, R38.2
- net +24V: now also R39.2, R40.2
- net GATE_H1: now also R29.2
- net GATE_H2: now also R31.2
- net GATE_L1: now also R33.2
- net GATE_L2: now also R35.2
- net GND: now also R30.1, R32.1, R34.1, R36.1
- net H_OUT1: no longer JP1.1
- net H_OUT2: no longer JP4.1
- net IN_H1_R: now also R39.1
- net IN_H2_R: now also R40.1
- net IN_L1_R: now also R37.1
- net IN_L2_R: now also R38.1
Routing:
- net GND: track 298.3 -> 372.7 mm, vias 26 -> 35
- net +3V3: track 108.2 -> 123.8 mm, vias 0 -> 1
- net H_OUT2: track 0.00 -> 15.3 mm, vias 12 -> 13
- net H_OUT1: track 0.00 -> 15.0 mm, vias 12 -> 13
- net IN_H1: track 0.00 -> 12.8 mm
- net IN_H2: track 0.00 -> 12.2 mm
- net +12V: track 207.9 -> 217.2 mm
- net N$14: track 15.5 -> 9.35 mm
- net IN_L1: track 0.00 -> 6.02 mm
- net N$15: track 10.6 -> 4.74 mm
- net IN_L2: track 0.00 -> 5.21 mm
- net +24V: track 38.0 -> 42.0 mm
- net IN_H1_R: track 1.72 -> 4.83 mm
- net IN_H2_R: track 1.86 -> 4.31 mm
- net GATE_L1: track 13.5 -> 15.6 mm
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- added copper zone on layer 1, net GND
- added copper zone on layer 16, net GND

Commit message: a
Parts:
- added R41, R42, R43, R44: (no value), rcl:R0603
- moved R36 50.7 mm to (-51.7, -20.9)
- moved R35 49.8 mm to (-51.7, -19.4), turned to 180 degrees
- moved R29 48.3 mm to (-20.3, 4.10), turned to 270 degrees
- moved R32 47.4 mm to (-26.4, 5.10)
- moved R31 44.2 mm to (-26.4, 3.70), turned to 180 degrees
- moved R30 41.7 mm to (-21.7, 4.10), turned to 90 degrees
- moved R34 34.1 mm to (-34.5, -19.9)
- moved R33 28.9 mm to (-34.5, -18.5), turned to 180 degrees
- moved C9 28.3 mm to (-46.6, -16.2), turned to 270 degrees
- moved R38 24.8 mm to (-42.9, -17.6), turned to 180 degrees
- moved T8 24.2 mm to (-39.4, -16.8), turned to 0 degrees
- moved R7 23.3 mm to (-42.9, -16.2), turned to 180 degrees
- moved R4 23.0 mm to (-51.4, -14.9)
- moved R6 23.0 mm to (-51.4, -17.3)
- moved U2 22.6 mm to (-46.6, -16.2)
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Connections:
- net +3V3: now also R41.2, R42.2, R43.2, R44.2
- net IN_H1: now also PIC32MZ.61, R42.1
- net IN_H2: now also PIC32MZ.62, R43.1
- net IN_L1: now also PIC32MZ.63, R41.1
- net IN_L2: now also PIC32MZ.64, R44.1
Routing:
- net IN_L2: track 5.21 -> 57.5 mm
- net IN_L1: track 6.02 -> 54.4 mm, vias 0 -> 1
- net IN_H2: track 12.2 -> 57.5 mm, vias 0 -> 1
- net GND: track 372.7 -> 417.5 mm, vias 35 -> 36
- net IN_H1: track 12.8 -> 53.3 mm
- net GATE_L2: track 27.2 -> 10.3 mm
- net +12V: track 217.2 -> 201.4 mm
- net N$25: track 2.94 -> 17.8 mm
- net H_OUT1: track 15.0 -> 25.1 mm
- net +3V3: track 123.8 -> 132.3 mm, vias 1 -> 2
- net GATE_H2: track 27.0 -> 35.3 mm
- net H_OUT2: track 15.3 -> 20.6 mm
- net GATE_H1: track 21.7 -> 27.0 mm
- net GATE_L1: track 15.6 -> 10.8 mm
- net +24V: track 42.0 -> 45.6 mm
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
Commit message: a
Parts:
- moved R44 11.6 mm to (24.6, -8.60)
- moved R32 2.16 mm to (-28.2, 6.30)
- moved R31 2.11 mm to (-28.2, 4.80)
- moved C2 1.46 mm to (29.6, -11.0), turned to 90 degrees
- moved R11 0.81 mm to (-21.1, -9.90)
- moved R41 0.45 mm to (24.0, -5.50)
Connections:
- removed net N$26: R29.1, R30.2
- removed net N$27: R31.1, R32.2
- removed net N$28: R33.1, R34.2
- removed net N$29: R35.1, R36.2
- new net GATE_H1_V: PIC32MZ.1, R29.1, R30.2
- new net GATE_H2_V: PIC32MZ.2, R31.1, R32.2
- new net GATE_L1_V: PIC32MZ.3, R33.1, R34.2
- new net GATE_L2_V: PIC32MZ.4, R35.1, R36.2
Routing:
- net GATE_H2_V: track 0.00 -> 91.4 mm, vias 0 -> 2
- net GATE_L2_V: track 0.00 -> 90.6 mm
- net GATE_H1_V: track 0.00 -> 82.6 mm, vias 0 -> 2
- net GATE_L1_V: track 0.00 -> 74.4 mm, vias 0 -> 2
- net IN_L2: track 57.5 -> 54.2 mm
- net GND: track 417.5 -> 420.6 mm
- net N$28: track 1.82 -> 0.00 mm
- net N$29: track 1.50 -> 0.00 mm
- net MCLR: track 18.5 -> 17.1 mm
- net N$27: track 1.40 -> 0.00 mm
- net N$26: track 1.40 -> 0.00 mm
- net N$9: track 2.46 -> 3.30 mm
- net GATE_H2: track 35.3 -> 34.5 mm
- net IN_H1: track 53.3 -> 54.1 mm
- net IN_L1: track 54.4 -> 53.7 mm
