File: POVBaseV2/POVBase.brd (EAGLE design)
At the start: 36 x 36 mm, 72 parts, among them J1 MEM2075-00-140-01-A, U1 ZXGD3005E6TA, U2 ZXGD3005E6TA, U3 ZXGD3005E6TA, U4 ZXGD3005E6TA, U5 TLV75533PDBVR, U6 TPS55340RTER

Commit message: sdf
Parts:
- removed D1: GF1, diode:SMA-DO214AC
- removed L1: 10uH, rcl:POWER-CHOKE_WE-TPC
- added C22, C23: (no value), rcl:C0603
- added R29: (no value), rcl:R0603
- added U7: CHL8510CRT, CHL8510CRT:10-VFDFN
- C12: value 0.047uF -> (none)
- C13: value 100pF -> (none)
- C14: value 0.1uF -> (none)
- C15, C18, C19: value 4.7uF -> (none); device rcl:C0805 -> rcl:C0603
- R24, R25: value 2.55k -> (none); device rcl:R0603 -> rcl:R1206
- R26: value 10k -> (none)
- R27: value 10k -> (none); device rcl:R0603 -> rcl:R1206
- R28: value 187k -> (none); device rcl:R0603 -> rcl:R1206
- U6: value TPS55340RTER -> CHL8510CRT; device TPS55340RTER:QFN50P300X300X100-17N -> CHL8510CRT:10-VFDFN
- moved C19 94.6 mm to (-113.0, -23.0), turned to 0 degrees
- moved R27 91.5 mm to (-112.0, -19.0), turned to 0 degrees
- moved R25 91.2 mm to (-112.0, -5.00), turned to 90 degrees
- moved C15 89.1 mm to (-110.0, 1.00), turned to 0 degrees
- moved C13 88.7 mm to (-110.0, -1.00), flipped to the top, turned to 0 degrees
- moved R24 88.2 mm to (-109.0, -5.00), flipped to the top, turned to 90 degrees
- moved C14 87.5 mm to (-106.0, -3.00), flipped to the top, turned to 0 degrees
- moved R28 86.2 mm to (-107.0, -19.0)
- moved R26 85.0 mm to (-106.0, 1.00), turned to 0 degrees
- moved C12 83.4 mm to (-106.0, -1.00), turned to 0 degrees
- moved C18 81.7 mm to (-103.0, -18.0), turned to 0 degrees
- moved U6 79.0 mm to (-99.0, -4.00), turned to 0 degrees
- moved T1 44.6 mm to (-82.0, 10.0)
- moved T5 38.5 mm to (-70.0, 10.0)
- moved T3 37.0 mm to (-82.0, -7.00)
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Connections:
- removed net BST_COMP: C13.1, R24.2, U6.7
- removed net BST_COMP_R: C14.1, R24.1
- removed net BST_EN: R26.1, U6.3
- removed net BST_FB: R27.1, R28.2, U6.8
- removed net BST_FREQ: R25.1, U6.9
- removed net BST_SS: C12.1, U6.4
- removed net BST_SW: D1.A, L1.2, U6.1, U6.15, U6.16
- new net N$26: C11.1, J1.P4
- new net N$27: R25.1, U6.6
- new net N$28: R24.1, U6.10
- new net N$29: C15.2, R26.2
- new net N$30: R26.1, U6.1
- new net N$31: R28.1, U7.6
- new net N$32: R27.1, U7.10
- new net N$33: C23.2, R29.2
- new net N$34: R29.1, U7.1
- net +12V: now also C12.1, C13.1, C14.1, C18.1, C19.1, C22.1, U6.4, U6.5, U7.2, U7.4, U7.5; no longer L1.1, R26.2
- net +24V: no longer C15.1, C18.1, C19.1, D1.K, R28.1
- net +3V3: no longer C11.1, J1.P4
- net GATE_H1: now also R24.2
- net GATE_H2: now also R27.2
- net GATE_L1: now also R25.2
- net GATE_L2: now also R28.2
- net GND: now also C22.2, U6.7, U6.8, U7.11, U7.7, U7.8; no longer C15.2, R25.2, R27.2, U6.12, U6.13, U6.17, U6.5, U6.6
- net H_OUT1: now also C15.1, U6.9
- net H_OUT2: now also C23.1, U7.9
Routing:
- net GND: track 300.2 -> 0.32 mm, vias 26 -> 0
- net +12V: track 207.9 -> 0.12 mm, vias 28 -> 0
- net +3V3: track 110.1 -> 0.00 mm
- net +24V: track 38.0 -> 0.00 mm
- net GATE_L2: track 28.2 -> 0.00 mm
- net GATE_H2: track 27.0 -> 0.00 mm, vias 2 -> 0
- net GATE_H1: track 21.7 -> 0.00 mm, vias 2 -> 0
- net PGD: track 18.8 -> 0.00 mm
- net MCLR: track 18.1 -> 0.00 mm
- net N$14: track 15.5 -> 0.00 mm
- net GATE_L1: track 13.5 -> 0.00 mm
- net PGC: track 11.8 -> 0.00 mm
- net +5V: track 11.6 -> 0.00 mm, vias 1 -> 0
- net N$15: track 10.6 -> 0.00 mm
- net BST_SW: track 9.22 -> 0.00 mm
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- removed copper zone on layer 1, net +12V
- removed copper zone on layer 1, net H_OUT1
- removed copper zone on layer 16, net H_OUT1
- removed copper zone on layer 1, net H_OUT2
- removed copper zone on layer 16, net H_OUT2
