File: POVBaseV2/POVBase.sch (EAGLE design)
At the start: 29 parts, among them IC1 LM2576S, IC2 PIC16F876SO, Q5 IRF540, Q6 IRF540, T2 2SC1306

Commit message: a
Parts:
- removed D2: (no value), eagle-ltspice:DIODE_E-SMC
- removed IC1: LM2576S, lm2576:LM2576S
- removed IC2: PIC16F876SO, microchip:PIC16F876SO
- removed L1: 82114R, inductors:82114R
- removed Q1, Q2: (no value), semicon-smd-ipc:NPN-TRANSISTOR_SOT23
- removed Q3, Q4: (no value), semicon-smd-ipc:PNP-TRANSISTOR_SOT23
- removed Q5, Q6: IRF540, transistor-power:IRF540
- removed Q7, Q9: (no value), transistor-power:PMOSFET_PTO220BV
- removed Q8: (no value), special:XTAL/S
- removed T2: 2SC1306, transistor:2SC1306
- added C10, C11, C16: 0.1uF, rcl:C-EUC0603
- added C17: (no value), rcl:CPOL-USC/6032-28R
- added C20: (no value), rcl:C-USC0805
- added C21: (no value), rcl:CPOL-USB/3528-21W
- added C6, C7, C8, C9: 0.1uF, rcl:C-EUC0805
- added J1: MEM2075-00-140-01-A, MEM2075-00-140-01-A:MEM2075-00-140-01-A
- added PIC32MZ: PIC32MZ2048EFH064-I/PT, PIC32MZ2048EFH064-I_PT:PIC32MZ2048EFH064-I/PT
- added R10, R12, R13, R6, R8: (no value), rcl:R-US_R1206
- added R11, R14, R18, R7: (no value), rcl:R-US_R0603
- added R15: 41k, rcl:R-US_R0603
- added R16: 7.6k, rcl:R-US_R0603
- added R17: 4.7uH, rcl:R-EU_R0805
- added R20: 1k, rcl:R-US_R0603
- added T1, T3, T4, T5: (no value), we-transistor:MOSFET-N-D2PAK
- added U$2: AP65211A, SOT95P280X140-6N:AP65211A
- added U1, U2, U3, U4: ZXGD3005E6TA, ZXGD3005E6TA:ZXGD3005E6TA
- added U5: TLV75533PDBVR, TLV75533PDBVR:TLV75533PDBVR
- C1, C2, C3: value (none) -> 0.1uF; device resistor:C-EUC0805 -> rcl:C-EUC0603
- C4: value (none) -> 0.1uF; device rcl:CPOL-USE2.5-7 -> rcl:C-EUC0603
- C5: value (none) -> 0.1uF; device rcl:CPOL-USE1.8-4 -> rcl:C-EUC0603
- R1, R2, R4: device resistor:R-US_R0805 -> rcl:R-US_R1206
- R3, R9: device resistor:R-US_R0805 -> rcl:R-US_R0603
- R5: value (none) -> 75k; device resistor:R-US_R0805 -> rcl:R-US_R0603
Connections:
- removed net N$14: IC2.PGC/RB6, JP3.5
- removed net N$15: D2.A, IC1.OUT, L1.1
- removed net N$20: T2.C
- new net +12V1: C7.2, U3.VCC
- new net +12V2: C8.2, U4.VCC
- new net +12V3: C9.2, U2.VCC
- new net +3V3: C1.1, C10.1, C11.1, C2.1, C20.1, C3.1, C4.1, C5.1, J1.VDD, JP3.2, PIC32MZ.AVDD, PIC32MZ.VDD, PIC32MZ.VDD@1, PIC32MZ.VDD@2, PIC32MZ.VDD@3, PIC32MZ.VDD@4, R20.2, U5.OUT
- new net GATE_H1: R10.2, R8.2, T1.G
- new net GATE_H2: R12.2, R13.2, T3.G
- new net GATE_L1: R1.2, R2.2, T5.G
- new net GATE_L2: R4.2, R6.2, T4.G
- new net H_OUT1: JP1.1, T1.S, T5.D
- new net H_OUT2: JP4.1, T3.S, T4.D
- new net IN_H1: R11.1
- new net IN_H2: R14.1
- new net IN_L1: R3.1
- new net IN_L2: R7.1
- new net MCLR: JP3.1, PIC32MZ.MCLR, R20.1
- new net N$23: R14.2, U4.IN
- new net N$9: R11.2, U3.IN
- new net PGC: JP3.5, PIC32MZ.PGEC1/VREF-/CVREF-/AN1/RPB1/RB1
- new net PGD: JP3.4, PIC32MZ.PGED1/VREF+/CVREF+/AN0/RPB0/PMA6/RB0
- net +12V: now also C17.+, C6.2, R9.1, T1.D, T3.D, U$2.IN, U1.VCC; no longer C4.+, IC1.VIN, Q3.E, Q4.E, Q7.S, Q9.S
- net +5V: now also C21.+, R15.2, R17.2, R18.1, U5.IN; no longer C3.2, C5.+, IC1.FB, IC2.VDD, JP3.2, L1.2, R9.2
- net GND: now also C1.2, C10.2, C11.2, C17.-, C2.2, C20.2, C21.-, C3.2, C4.2, C5.2, C6.1, C7.1, C8.1, C9.1, J1.VSS, PIC32MZ.AVSS, PIC32MZ.VSS, PIC32MZ.VSS@1, PIC32MZ.VSS@2, PIC32MZ.VSS@3, PIC32MZ.VSS@4, PIC32MZ.VSS@5, PIC32MZ.VUSB3V3, R16.1, T4.S, T5.S, U$2.GND, U1.VEE, U2.VEE, U3.VEE, U4.VEE, U5.GND; no longer C1.1, C2.1, C3.1, C4.-, C5.-, D2.C, IC1.GND, IC1.OFF, IC2.VSS, IC2.VSS@1, Q1.E, Q2.E, Q5.S, Q6.S, T2.E
- net N$1: now also R3.2, U1.IN; no longer Q1.C, Q3.C, Q5.G, Q7.G
- net N$10: now also R12.1, U4.SINK; no longer JP4.1, Q6.D, Q9.D
- net N$11: now also R13.1, U4.SOURCE; no longer JP1.1, Q5.D, Q7.D
- net N$12: now also R9.2, U$2.EN; no longer IC2.!MCLR/THV, JP3.1, R9.1
- net N$13: now also R18.2, U5.EN; no longer IC2.PGD/RB7, JP3.4
- net N$16: now also C16.1, R17.1, U$2.SW; no longer C1.2, IC2.OSC2/CLKOUT, Q8.1
- net N$17: now also C16.2, U$2.BST; no longer C2.2, IC2.OSC1/CLKIN, Q8.2
- net N$2: now also R1.1, U1.SINK; no longer Q1.B, R1.2
- net N$21: now also U$2.FB; no longer IC2.RC1/T1OSI
- net N$22: now also R15.1, R16.2; no longer T2.B
- net N$3: now also R2.1, U1.SOURCE; no longer Q2.B, R4.2
- net N$4: now also R4.1, U2.SINK; no longer Q2.C, Q4.C, Q6.G, Q9.G
- net N$5: now also R6.1, U2.SOURCE; no longer Q3.B, R2.2
- net N$6: now also R7.2, U2.IN; no longer Q4.B, R3.2
- net N$7: now also R8.1, U3.SINK; no longer IC2.RC3/SCK, R1.1, R2.1
- net N$8: now also R10.1, U3.SOURCE; no longer IC2.RC2/CCP1, R3.1, R4.1
Other:
- moved on the sheet: C1, C2, C3, JP1, JP2, JP3, JP4, R1, R2, R3, R4, R5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

Commit message: a
Parts:
- added R19, R21, R22, R23: (no value), rcl:R-US_R0603
- added T2, T6, T7, T8: (no value), transistor:-NPN-SOT23-EBC
Connections:
- removed net +12V1: C7.2, U3.VCC
- removed net +12V2: C8.2, U4.VCC
- removed net +12V3: C9.2, U2.VCC
- new net +24V: C7.2, C8.2, U3.VCC, U4.VCC
- new net IN_H1_R: R11.1, T6.C
- new net IN_H2_R: R14.1, T2.C
- new net IN_L1_R: R3.1, T7.C
- new net IN_L2_R: R7.1, T8.C
- new net N$14: R19.1, T2.B
- new net N$15: R21.1, T6.B
- new net N$24: R22.1, T7.B
- new net N$25: R23.1, T8.B
- net +12V: now also C9.2, U2.VCC
- net GND: now also T2.E, T6.E, T7.E, T8.E
- net IN_H1: now also R21.2; no longer R11.1
- net IN_H2: now also R19.2; no longer R14.1
- net IN_L1: now also R22.2; no longer R3.1
- net IN_L2: now also R23.2; no longer R7.1
Other:
- moved on the sheet: C6, C7, C8, C9, R1, R10, R11, R12, R13, R14, R2, R3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

Commit message: a
Parts:
- added C12: 0.047uF, rcl:C-EUC0603
- added C13: 100pF, rcl:C-EUC0603
- added C14: 0.1uF, rcl:C-EUC0603
- added C15, C18, C19: 4.7uF, rcl:C-EUC0805
- added D1: GF1, diode:GF1
- added L1: 10uH, rcl:L-USWE-TPC
- added R24, R25: 2.55k, rcl:R-US_R0603
- added R26, R27: 10k, rcl:R-US_R0603
- added R28: 187k, rcl:R-US_R0603
- added U6: TPS55340RTER, TPS55340RTER:TPS55340RTER
Connections:
- new net BST_COMP: C13.1, R24.2, U6.COMP
- new net BST_COMP_R: C14.1, R24.1
- new net BST_EN: R26.1, U6.EN
- new net BST_FB: R27.1, R28.2, U6.FB
- new net BST_FREQ: R25.1, U6.FREQ
- new net BST_SS: C12.1, U6.SS
- new net BST_SW: D1.A, L1.2, U6.SW
- net +12V: now also L1.1, R26.2, U6.VIN
- net +24V: now also C15.1, C18.1, C19.1, D1.C, R28.1
- net GND: now also C12.2, C13.2, C14.2, C15.2, C18.2, C19.2, J1.SHIELD, R25.2, R27.2, U6.GND, U6.SYNC

Commit message: a
Parts:
- removed JP1, JP4: (no value), pinhead:PINHD-1X1
- added R29, R31: 90k, rcl:R-US_R0603
- added R30, R32: 10k, rcl:R-US_R0603
- added R33, R35: 45k, rcl:R-US_R0603
- added R34, R36: 5k, rcl:R-US_R0603
- added R37, R38, R39, R40: (no value), rcl:R-US_R0603
Connections:
- new net N$26: R29.1, R30.2
- new net N$27: R31.1, R32.2
- new net N$28: R33.1, R34.2
- new net N$29: R35.1, R36.2
- net +12V: now also R37.2, R38.2
- net +24V: now also R39.2, R40.2
- net GATE_H1: now also R29.2
- net GATE_H2: now also R31.2
- net GATE_L1: now also R33.2
- net GATE_L2: now also R35.2
- net GND: now also R30.1, R32.1, R34.1, R36.1
- net H_OUT1: no longer JP1.1
- net H_OUT2: no longer JP4.1
- net IN_H1_R: now also R39.1
- net IN_H2_R: now also R40.1
- net IN_L1_R: now also R37.1
- net IN_L2_R: now also R38.1
Other:
- moved on the sheet: C6, C7, C8, C9, R1, R10, R11, R12, R13, R14, R19, R2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

Commit message: a
Parts:
- added R41, R42, R43, R44: (no value), rcl:R-US_R0603
Connections:
- net +3V3: now also R41.2, R42.2, R43.2, R44.2
- net IN_H1: now also PIC32MZ.TRD1/SQID1/ERXD0/PMD1/RE1, R42.1
- net IN_H2: now also PIC32MZ.TRD2/SQID2/ERXDV/ECRSDV/AECRSDV/PMD2/RE2, R43.1
- net IN_L1: now also PIC32MZ.TRD3/SQID3/ERXCLK/EREFCLK/RPE3/PMD3/RE3, R41.1
- net IN_L2: now also PIC32MZ.AN18/ERXERR/PMD4/RE4, R44.1
Other:
- moved on the sheet: C6, C7, C8, C9, R1, R10, R11, R12, R13, R14, R19, R2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

Commit message: a
Connections:
- removed net N$26: R29.1, R30.2
- removed net N$27: R31.1, R32.2
- removed net N$28: R33.1, R34.2
- removed net N$29: R35.1, R36.2
- new net GATE_H1_V: PIC32MZ.AN17/ETXEN/RPE5/PMD5/RE5, R29.1, R30.2
- new net GATE_H2_V: PIC32MZ.AN16/ETXD0/PMD6/RE6, R31.1, R32.2
- new net GATE_L1_V: PIC32MZ.AN15/ETXD1/PMD7/RE7, R33.1, R34.2
- new net GATE_L2_V: PIC32MZ.AN14/C1IND/RPG6/SCK2/PMA5/RG6, R35.1, R36.2
Other:
- moved on the sheet: R29, R30, R33, R34
Changed lines of the file:
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@@
 </instance>
 <instance part="SUPPLY23" gate="GND" x="231.14" y="45.72" smashed="yes"/>
-<instance part="R29" gate="G$1" x="-78.74" y="40.64" smashed="yes" rot="R90">
-<attribute name="NAME" x="-84.582" y="41.1226" size="1.778" layer="95"/>
-<attribute name="VALUE" x="-84.074" y="38.862" size="1.778" layer="96"/>
-</instance>
-<instance part="R30" gate="G$1" x="-78.74" y="30.48" smashed="yes" rot="R90">
-<attribute name="NAME" x="-84.582" y="31.2166" size="1.778" layer="95"/>
-<attribute name="VALUE" x="-84.074" y="28.956" size="1.778" layer="96"/>
-</instance>
-<instance part="SUPPLY27" gate="GND" x="-78.74" y="22.86" smashed="yes"/>
+<instance part="R29" gate="G$1" x="-83.82" y="40.64" smashed="yes" rot="R90">
+<attribute name="NAME" x="-89.662" y="41.1226" size="1.778" layer="95"/>
+<attribute name="VALUE" x="-89.154" y="38.862" size="1.778" layer="96"/>
+</instance>
+<instance part="R30" gate="G$1" x="-83.82" y="30.48" smashed="yes" rot="R90">
+<attribute name="NAME" x="-89.662" y="31.2166" size="1.778" layer="95"/>
+<attribute name="VALUE" x="-89.154" y="28.956" size="1.778" layer="96"/>
+</instance>
+<instance part="SUPPLY27" gate="GND" x="-83.82" y="22.86" smashed="yes"/>
 <instance part="R31" gate="G$1" x="-60.96" y="40.64" smashed="yes" rot="R90">
 <attribute name="NAME" x="-66.802" y="41.1226" size="1.778" layer="95"/>
@@
 </instance>
 <instance part="SUPPLY28" gate="GND" x="-60.96" y="22.86" smashed="yes"/>
-<instance part="R33" gate="G$1" x="-78.74" y="10.16" smashed="yes" rot="R90">
-<attribute name="NAME" x="-84.582" y="10.6426" size="1.778" layer="95"/>
-<attribute name="VALUE" x="-84.074" y="8.382" size="1.778" layer="96"/>
-</instance>
-<instance part="R34" gate="G$1" x="-78.74" y="0" smashed="yes" rot="R90">
-<attribute name="NAME" x="-84.582" y="0.7366" size="1.778" layer="95"/>
-<attribute name="VALUE" x="-84.074" y="-1.524" size="1.778" layer="96"/>
-</instance>
-<instance part="SUPPLY29" gate="GND" x="-78.74" y="-7.62" smashed="yes"/>
+<instance part="R33" gate="G$1" x="-83.82" y="10.16" smashed="yes" rot="R90">
+<attribute name="NAME" x="-89.662" y="10.6426" size="1.778" layer="95"/>
+<attribute name="VALUE" x="-89.154" y="8.382" size="1.778" layer="96"/>
+</instance>
+<instance part="R34" gate="G$1" x="-83.82" y="0" smashed="yes" rot="R90">
+<attribute name="NAME" x="-89.662" y="0.7366" size="1.778" layer="95"/>
+<attribute name="VALUE" x="-89.154" y="-1.524" size="1.778" layer="96"/>
+</instance>
+<instance part="SUPPLY29" gate="GND" x="-83.82" y="-7.62" smashed="yes"/>
 <instance part="R35" gate="G$1" x="-60.96" y="10.16" smashed="yes" rot="R90">
 <attribute name="NAME" x="-66.802" y="10.6426" size="1.778" layer="95"/>
@@
 <segment>
 <pinref part="R29" gate="G$1" pin="2"/>
-<wire x1="-78.74" y1="45.72" x2="-88.9" y2="45.72" width="0.1524" layer="91"/>
-<label x="-88.9" y="45.72" size="1.778" layer="95"/>
+<wire x1="-83.82" y1="45.72" x2="-93.98" y2="45.72" width="0.1524" layer="91"/>
+<label x="-93.98" y="45.72" size="1.778" layer="95"/>
 </segment>
 </net>
@@
 <segment>
 <pinref part="R33" gate="G$1" pin="2"/>
-<wire x1="-78.74" y1="15.24" x2="-88.9" y2="15.24" width="0.1524" layer="91"/>
-<label x="-88.9" y="15.24" size="1.778" layer="95"/>
+<wire x1="-83.82" y1="15.24" x2="-93.98" y2="15.24" width="0.1524" layer="91"/>
+<label x="-93.98" y="15.24" size="1.778" layer="95"/>
 </segment>
 </net>
@@
 </segment>
 </net>
-<net name="N$26" class="0">
+<net name="GATE_H2_V" class="0">
+<segment>
+<pinref part="R32" gate="G$1" pin="2"/>
+<pinref part="R31" gate="G$1" pin="1"/>
+<wire x1="-60.96" y1="35.56" x2="-45.72" y2="35.56" width="0.1524" layer="91"/>
+<junction x="-60.96" y="35.56"/>
+<label x="-58.42" y="35.56" size="1.778" layer="95"/>
+</segment>
+<segment>
+<pinref part="PIC32MZ" gate="G$1" pin="AN16/ETXD0/PMD6/RE6"/>
+<wire x1="25.4" y1="58.42" x2="10.16" y2="58.42" width="0.1524" layer="91"/>
+<label x="10.16" y="58.42" size="1.778" layer="95"/>
+</segment>
+</net>
+<net name="GATE_L1_V" class="0">
+<segment>
+<pinref part="R34" gate="G$1" pin="2"/>
+<pinref part="R33" gate="G$1" pin="1"/>
+<wire x1="-83.82" y1="5.08" x2="-68.58" y2="5.08" width="0.1524" layer="91"/>
+<junction x="-83.82" y="5.08"/>
+<label x="-81.28" y="5.08" size="1.778" layer="95"/>
+</segment>
+<segment>
+<pinref part="PIC32MZ" gate="G$1" pin="AN15/ETXD1/PMD7/RE7"/>
+<wire x1="25.4" y1="55.88" x2="10.16" y2="55.88" width="0.1524" layer="91"/>
+<label x="10.16" y="55.88" size="1.778" layer="95"/>
+</segment>
+</net>
+<net name="GATE_L2_V" class="0">
+<segment>
+<pinref part="R36" gate="G$1" pin="2"/>
+<pinref part="R35" gate="G$1" pin="1"/>
+<wire x1="-60.96" y1="5.08" x2="-45.72" y2="5.08" width="0.1524" layer="91"/>
+<junction x="-60.96" y="5.08"/>
+<label x="-58.42" y="5.08" size="1.778" layer="95"/>
+</segment>
+<segment>
+<pinref part="PIC32MZ" gate="G$1" pin="AN14/C1IND/RPG6/SCK2/PMA5/RG6"/>
+<wire x1="25.4" y1="53.34" x2="10.16" y2="53.34" width="0.1524" layer="91"/>
+<label x="10.16" y="53.34" size="1.778" layer="95"/>
+</segment>
+</net>
+<net name="GATE_H1_V" class="0">
+<segment>
+<pinref part="PIC32MZ" gate="G$1" pin="AN17/ETXEN/RPE5/PMD5/RE5"/>
+<wire x1="25.4" y1="60.96" x2="10.16" y2="60.96" width="0.1524" layer="91"/>
+<label x="10.16" y="60.96" size="1.778" layer="95"/>
+</segment>
 <segment>
 <pinref part="R30" gate="G$1" pin="2"/>
 <pinref part="R29" gate="G$1" pin="1"/>
-<wire x1="-78.74" y1="35.56" x2="-68.58" y2="35.56" width="0.1524" layer="91"/>
-<junction x="-78.74" y="35.56"/>
-</segment>
-</net>
-<net name="N$27" class="0">
-<segment>
-<pinref part="R32" gate="G$1" pin="2"/>
-<pinref part="R31" gate="G$1" pin="1"/>
-<wire x1="-60.96" y1="35.56" x2="-50.8" y2="35.56" width="0.1524" layer="91"/>
-<junction x="-60.96" y="35.56"/>
-</segment>
-</net>
-<net name="N$28" class="0">
-<segment>
-<pinref part="R34" gate="G$1" pin="2"/>
-<pinref part="R33" gate="G$1" pin="1"/>
-<wire x1="-78.74" y1="5.08" x2="-68.58" y2="5.08" width="0.1524" layer="91"/>
-<junction x="-78.74" y="5.08"/>
-</segment>
-</net>
-<net name="N$29" class="0">
-<segment>
-<pinref part="R36" gate="G$1" pin="2"/>
-<pinref part="R35" gate="G$1" pin="1"/>
-<wire x1="-60.96" y1="5.08" x2="-50.8" y2="5.08" width="0.1524" layer="91"/>
-<junction x="-60.96" y="5.08"/>
-</segment>
-</net>
+<wire x1="-83.82" y1="35.56" x2="-68.58" y2="35.56" width="0.1524" layer="91"/>
+<junction x="-83.82" y="35.56"/>
+<label x="-81.28" y="35.56" size="1.778" layer="95"/>
+</segment>
+</net>
