File: POVBaseV2/POVBase.sch (EAGLE design)
At the start: 72 parts, among them J1 MEM2075-00-140-01-A, U1 ZXGD3005E6TA, U2 ZXGD3005E6TA, U3 ZXGD3005E6TA, U4 ZXGD3005E6TA, U5 TLV75533PDBVR, U6 TPS55340RTER

Commit message: sdf
Parts:
- removed D1: GF1, diode:GF1
- removed L1: 10uH, rcl:L-USWE-TPC
- added C22, C23: (no value), rcl:C-EUC0603
- added R29: (no value), rcl:R-US_R0603
- added U7: CHL8510CRT, CHL8510CRT:CHL8510CRT
- C12: value 0.047uF -> (none)
- C13: value 100pF -> (none)
- C14: value 0.1uF -> (none)
- C15, C18, C19: value 4.7uF -> (none); device rcl:C-EUC0805 -> rcl:C-EUC0603
- R24, R25: value 2.55k -> (none); device rcl:R-US_R0603 -> rcl:R-US_R1206
- R26: value 10k -> (none)
- R27: value 10k -> (none); device rcl:R-US_R0603 -> rcl:R-US_R1206
- R28: value 187k -> (none); device rcl:R-US_R0603 -> rcl:R-US_R1206
- U6: value TPS55340RTER -> CHL8510CRT; device TPS55340RTER:TPS55340RTER -> CHL8510CRT:CHL8510CRT
Connections:
- removed net BST_COMP: C13.1, R24.2, U6.COMP
- removed net BST_COMP_R: C14.1, R24.1
- removed net BST_EN: R26.1, U6.EN
- removed net BST_FB: R27.1, R28.2, U6.FB
- removed net BST_FREQ: R25.1, U6.FREQ
- removed net BST_SS: C12.1, U6.SS
- removed net BST_SW: D1.A, L1.2, U6.SW
- new net N$26: C11.1, J1.VDD
- new net N$27: R25.1, U6.LO
- new net N$28: R24.1, U6.HI
- new net N$29: C15.2, R26.2
- new net N$30: R26.1, U6.BOOT
- new net N$31: R28.1, U7.LO
- new net N$32: R27.1, U7.HI
- new net N$33: C23.2, R29.2
- new net N$34: R29.1, U7.BOOT
- net +12V: now also C12.1, C13.1, C14.1, C18.1, C19.1, C22.1, U6.VCC, U7.VCC; no longer L1.1, R26.2, U6.VIN
- net +24V: no longer C15.1, C18.1, C19.1, D1.C, R28.1
- net +3V3: no longer C11.1, J1.VDD
- net GATE_H1: now also R24.2
- net GATE_H2: now also R27.2
- net GATE_L1: now also R25.2
- net GATE_L2: now also R28.2
- net GND: now also C22.2, U6.MODE, U7.GND, U7.MODE; no longer C15.2, R25.2, R27.2, U6.SYNC
- net H_OUT1: now also C15.1, U6.SWITCH
- net H_OUT2: now also C23.1, U7.SWITCH
Other:
- moved on the sheet: C12, C13, C14, C15, C18, C19, R24, R25, R26, R27, R28
