File: POVRotorV2/POVRotor.brd (EAGLE design)
At the start: 195 x 22.6 mm, 102 parts, among them IC1 LM2576S, U1 PIC32MZ2048EFH064-I/PT

Commit message: a
Parts:
- removed C1, C3: (no value), resistor:E2,5-6E
- removed D1: (no value), telefunken:SOD106A
- removed IC1: LM2576S, lm2576:TO263-5
- removed L2: (no value), resistor:L4532P
- added C16: 0.1uF, rcl:C0603
- added C17: (no value), rcl:C/6032-28R
- added R10, R7, R8, R9: (no value), resistor:R0603
- added R11: 75k, rcl:R0603
- added R12: 41k, rcl:R0603
- added R13: 7.6k, rcl:R0603
- added R14: 4.7uH, rcl:R0805
- added U$74: AP65211A, SOT95P280X140-6N:SOT95P280X140-6N
- moved R3 67.7 mm to (-47.4, 16.5)
- moved R4 57.8 mm to (-4.20, 2.10)
- moved C12 56.8 mm to (-84.6, 28.6)
- moved C11 50.1 mm to (-84.4, 26.0)
- moved R6 48.3 mm to (-51.3, -15.7)
- moved C10 42.7 mm to (-84.4, 22.5)
- moved C9 36.2 mm to (-84.5, 20.0)
Connections:
- removed net N$3: D1.K, IC1.2, L2.1
- new net N$112: R10.2, U1.5
- new net N$129: C16.1, R14.1, U$74.2
- new net N$130: C16.2, U$74.6
- new net N$167: R11.1, U$74.4
- new net N$168: R11.2, R12.1, R13.2
- new net N$4: R7.1, U1.48
- new net N$47: R7.2, U$2.SDI
- new net N$50: R8.1, U1.45
- new net N$74: R8.2, U$37.SDI
- new net N$91: R9.1, U$19.SDI
- new net N$92: R9.2, U1.23
- new net N$95: R10.1, U$55.SDI
- net +15V: now also C17.+, U$74.3, U$74.5; no longer C3.+, IC1.1
- net +5V: now also R12.2, R14.2; no longer C1.+, IC1.4, L2.2
- net GND: now also C17.-, R13.1, U$74.1; no longer C1.-, C3.-, D1.A, IC1.3, IC1.5
Routing:
- net GND: track 906.9 -> 849.5 mm, vias 2 -> 3
- net +5V: track 296.1 -> 267.2 mm, vias 1 -> 2
- net +15V: track 122.3 -> 147.2 mm
- net N$3: track 16.3 -> 0.00 mm
- net N$129: track 0.00 -> 13.3 mm
- net N$168: track 0.00 -> 3.21 mm
- net N$21: track 2.61 -> 0.00 mm
- net N$167: track 0.00 -> 2.54 mm
- net N$130: track 0.00 -> 1.59 mm

Commit message: s
Parts:
- removed C10, C11, C12, C9: (no value), resistor:C0805
- removed IC2: (no value), lm2576:SOT223
- removed JP2: (no value), pinhead:1X04
- removed U$1, U$10, U$11, U$12, U$13, U$14, U$15, U$16, U$17, U$18, U$19, U$2, U$20, U$21, U$22, U$23, U$24, U$25, U$26, U$27, U$28, U$29, U$3, U$30, U$31, U$32, U$33, U$34, U$35, U$36, U$37, U$38, U$39, U$4, U$40, U$41, U$42, U$43, U$44, U$45, U$46, U$47, U$48, U$49, U$5, U$50, U$51, U$52, U$53, U$54, U$55, U$56, U$57, U$58, U$59, U$6, U$60, U$61, U$62, U$63, U$64, U$65, U$66, U$67, U$68, U$69, U$7, U$70, U$71, U$72, U$73, U$8, U$9: 2020LED, APA2020:2020LED
- added C20: (no value), rcl:C0805
- added C21: (no value), rcl:B/3528-21W
- added R15: 75k, rcl:R0603
- added U10, U11, U12, U13, U14, U15, U16, U17, U18, U19, U2, U20, U21, U22, U23, U24, U25, U26, U27, U28, U29, U30, U31, U32, U33, U34, U35, U36, U37, U38, U39, U40, U41, U42, U43, U44, U45, U46, U47, U48, U49, U5, U50, U51, U52, U53, U54, U55, U56, U57, U58, U59, U6, U60, U61, U62, U63, U64, U65, U66, U67, U68, U69, U7, U70, U71, U72, U73, U74, U75, U76, U8, U9: 3341, APA102:LED_3341
- added U3: TLV75533PDBVR, TLV75533PDBVR:SOT95P280X145-5N
- moved D3 75.3 mm to (37.7, 5.30)
- moved D5 75.3 mm to (37.7, -5.30)
- moved D2 63.3 mm to (31.7, -5.30)
- moved D4 63.3 mm to (31.7, 5.30)
- moved R4 44.5 mm to (-47.0, 14.2), turned to 90 degrees
- moved R8 41.5 mm to (-48.3, 14.2), turned to 90 degrees
- moved R7 32.7 mm to (-49.6, 14.2), turned to 270 degrees
- moved R9 14.0 mm to (-40.1, -14.3), turned to 90 degrees
- moved C16 13.3 mm to (46.2, 0.50)
- moved R11 13.3 mm to (51.1, 1.00)
- moved U$74 13.3 mm to (48.6, 0.50)
- moved R12 13.3 mm to (48.4, 3.30)
- moved R13 13.3 mm to (51.8, 3.30)
- moved R14 13.3 mm to (47.4, 5.10)
- moved C17 13.0 mm to (42.9, 0.40)
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Connections:
- removed net N$166: U$72.CLKO, U$73.CLKI
- removed net N$6: U$1.SDI, U$2.SDO
- new net N$3: R15.2, U3.3
- net +3V3: now also C20.1, U3.5; no longer IC2.2, JP2.1
- net +5V: now also C21.+, R15.1, U10.1, U10.8, U11.1, U11.8, U12.1, U12.8, U13.1, U13.8, U14.1, U14.8, U15.1, U15.8, U16.1, U16.8, U17.1, U17.8, U18.1, U18.8, U19.1, U19.8, U2.1, U2.8, U20.1, U20.8, U21.1, U21.8, U22.1, U22.8, U23.1, U23.8, U24.1, U24.8, U25.1, U25.8, U26.1, U26.8, U27.1, U27.8, U28.1, U28.8, U29.1, U29.8, U3.1, U30.1, U30.8, U31.1, U31.8, U32.1, U32.8, U33.1, U33.8, U34.1, U34.8, U35.1, U35.8, U36.1, U36.8, U37.1, U37.8, U38.1, U38.8, U39.1, U39.8, U40.1, U40.8, U41.1, U41.8, U42.1, U42.8, U43.1, U43.8, U44.1, U44.8, U45.1, U45.8, U46.1, U46.8, U47.1, U47.8, U48.1, U48.8, U49.1, U49.8, U5.1, U5.8, U50.1, U50.8, U51.1, U51.8, U52.1, U52.8, U53.1, U53.8, U54.1, U54.8, U55.1, U55.8, U56.1, U56.8, U57.1, U57.8, U58.1, U58.8, U59.1, U59.8, U6.1, U6.8, U60.1, U60.8, U61.1, U61.8, U62.1, U62.8, U63.1, U63.8, U64.1, U64.8, U65.1, U65.8, U66.1, U66.8, U67.1, U67.8, U68.1, U68.8, U69.1, U69.8, U7.1, U7.8, U70.1, U70.8, U71.1, U71.8, U72.1, U72.8, U73.1, U73.8, U74.1, U74.8, U75.1, U75.8, U76.1, U76.8, U8.1, U8.8, U9.1, U9.8; no longer C10.1, C11.1, C12.1, C9.1, IC2.3, U$1.VCC, U$10.VCC, U$11.VCC, U$12.VCC, U$13.VCC, U$14.VCC, U$15.VCC, U$16.VCC, U$17.VCC, U$18.VCC, U$19.VCC, U$2.VCC, U$20.VCC, U$21.VCC, U$22.VCC, U$23.VCC, U$24.VCC, U$25.VCC, U$26.VCC, U$27.VCC, U$28.VCC, U$29.VCC, U$3.VCC, U$30.VCC, U$31.VCC, U$32.VCC, U$33.VCC, U$34.VCC, U$35.VCC, U$36.VCC, U$37.VCC, U$38.VCC, U$39.VCC, U$4.VCC, U$40.VCC, U$41.VCC, U$42.VCC, U$43.VCC, U$44.VCC, U$45.VCC, U$46.VCC, U$47.VCC, U$48.VCC, U$49.VCC, U$5.VCC, U$50.VCC, U$51.VCC, U$52.VCC, U$53.VCC, U$54.VCC, U$55.VCC, U$56.VCC, U$57.VCC, U$58.VCC, U$59.VCC, U$6.VCC, U$60.VCC, U$61.VCC, U$62.VCC, U$63.VCC, U$64.VCC, U$65.VCC, U$66.VCC, U$67.VCC, U$68.VCC, U$69.VCC, U$7.VCC, U$70.VCC, U$71.VCC, U$72.VCC, U$73.VCC, U$8.VCC, U$9.VCC
- net GND: now also C20.2, C21.-, U10.6, U10.7, U11.6, U11.7, U12.6, U12.7, U13.6, U13.7, U14.6, U14.7, U15.6, U15.7, U16.6, U16.7, U17.6, U17.7, U18.6, U18.7, U19.6, U19.7, U2.6, U2.7, U20.6, U20.7, U21.6, U21.7, U22.6, U22.7, U23.6, U23.7, U24.6, U24.7, U25.6, U25.7, U26.6, U26.7, U27.6, U27.7, U28.6, U28.7, U29.6, U29.7, U3.2, U30.6, U30.7, U31.6, U31.7, U32.6, U32.7, U33.6, U33.7, U34.6, U34.7, U35.6, U35.7, U36.6, U36.7, U37.6, U37.7, U38.6, U38.7, U39.6, U39.7, U40.6, U40.7, U41.6, U41.7, U42.6, U42.7, U43.6, U43.7, U44.6, U44.7, U45.6, U45.7, U46.6, U46.7, U47.6, U47.7, U48.6, U48.7, U49.6, U49.7, U5.6, U5.7, U50.6, U50.7, U51.6, U51.7, U52.6, U52.7, U53.6, U53.7, U54.6, U54.7, U55.6, U55.7, U56.6, U56.7, U57.6, U57.7, U58.6, U58.7, U59.6, U59.7, U6.6, U6.7, U60.6, U60.7, U61.6, U61.7, U62.6, U62.7, U63.6, U63.7, U64.6, U64.7, U65.6, U65.7, U66.6, U66.7, U67.6, U67.7, U68.6, U68.7, U69.6, U69.7, U7.6, U7.7, U70.6, U70.7, U71.6, U71.7, U72.6, U72.7, U73.6, U73.7, U74.6, U74.7, U75.6, U75.7, U76.6, U76.7, U8.6, U8.7, U9.6, U9.7; no longer C10.2, C11.2, C12.2, C9.2, IC2.1, JP2.4, U$1.GND, U$10.GND, U$11.GND, U$12.GND, U$13.GND, U$14.GND, U$15.GND, U$16.GND, U$17.GND, U$18.GND, U$19.GND, U$2.GND, U$20.GND, U$21.GND, U$22.GND, U$23.GND, U$24.GND, U$25.GND, U$26.GND, U$27.GND, U$28.GND, U$29.GND, U$3.GND, U$30.GND, U$31.GND, U$32.GND, U$33.GND, U$34.GND, U$35.GND, U$36.GND, U$37.GND, U$38.GND, U$39.GND, U$4.GND, U$40.GND, U$41.GND, U$42.GND, U$43.GND, U$44.GND, U$45.GND, U$46.GND, U$47.GND, U$48.GND, U$49.GND, U$5.GND, U$50.GND, U$51.GND, U$52.GND, U$53.GND, U$54.GND, U$55.GND, U$56.GND, U$57.GND, U$58.GND, U$59.GND, U$6.GND, U$60.GND, U$61.GND, U$62.GND, U$63.GND, U$64.GND, U$65.GND, U$66.GND, U$67.GND, U$68.GND, U$69.GND, U$7.GND, U$70.GND, U$71.GND, U$72.GND, U$73.GND, U$8.GND, U$9.GND
- net N$10: now also U2.3, U5.4; no longer R3.1, U$19.CLKI
- net N$100: now also U42.3, U44.4; no longer U$40.SDO, U$41.SDI
- net N$101: now also U45.2, U46.5; no longer U$40.CLKO, U$41.CLKI
- net N$102: now also U45.3, U46.4; no longer U$41.SDO, U$42.SDI
- net N$103: now also U46.2, U47.5; no longer U$41.CLKO, U$42.CLKI
- net N$104: now also U46.3, U47.4; no longer U$42.SDO, U$43.SDI
- net N$105: now also U47.2, U48.5; no longer U$42.CLKO, U$43.CLKI
- net N$106: now also U47.3, U48.4; no longer U$43.SDO, U$44.SDI
- net N$107: now also U48.2, U49.5; no longer U$43.CLKO, U$44.CLKI
- net N$108: now also U48.3, U49.4; no longer U$44.SDO, U$45.SDI
- net N$109: now also U49.2, U50.5; no longer U$44.CLKO, U$45.CLKI
- net N$11: now also U6.2, U7.5; no longer U$11.SDO, U$12.SDI
- net N$110: now also U49.3, U50.4; no longer U$45.SDO, U$46.SDI
- net N$111: now also U50.2, U51.5; no longer U$45.CLKO, U$46.CLKI
- net N$113: now also U50.3, U51.4; no longer U$46.SDO, U$47.SDI
- net N$114: now also U51.2, U52.5; no longer U$46.CLKO, U$47.CLKI
- net N$115: now also U51.3, U52.4; no longer U$47.SDO, U$48.SDI
- net N$116: now also U52.2, U53.5; no longer U$47.CLKO, U$48.CLKI
- net N$117: now also U52.3, U53.4; no longer U$48.SDO, U$49.SDI
- net N$118: now also U53.2, U54.5; no longer U$48.CLKO, U$49.CLKI
- net N$119: now also U53.3, U54.4; no longer U$49.SDO, U$50.SDI
- net N$120: now also U54.2, U56.5; no longer U$49.CLKO, U$50.CLKI
- net N$121: now also U54.3, U56.4; no longer U$50.SDO, U$51.SDI
- net N$122: now also U55.5, U56.2; no longer U$50.CLKO, U$51.CLKI
- net N$123: now also U55.4, U56.3; no longer U$51.SDO, U$52.SDI
- net N$124: now also U57.2, U58.5; no longer U$51.CLKO, U$52.CLKI
- net N$125: now also U57.3, U58.4; no longer U$52.SDO, U$53.SDI
- net N$126: now also U55.2, U57.5; no longer U$52.CLKO, U$53.CLKI
- net N$127: now also U55.3, U57.4; no longer U$53.SDO, U$54.SDI
- net N$128: now also U58.2, U59.5; no longer U$53.CLKO, U$54.CLKI
- net N$131: now also U58.3, U59.4; no longer U$55.SDO, U$56.SDI
- net N$132: now also U59.2, U60.5; no longer U$55.CLKO, U$56.CLKI
- net N$133: now also U59.3, U60.4; no longer U$56.SDO, U$57.SDI
- net N$134: now also U60.2, U61.5; no longer U$56.CLKO, U$57.CLKI
- net N$135: now also U60.3, U61.4; no longer U$57.SDO, U$58.SDI
- net N$136: now also U61.2, U62.5; no longer U$57.CLKO, U$58.CLKI
- net N$137: now also U61.3, U62.4; no longer U$58.SDO, U$59.SDI
- net N$138: now also U62.2, U63.5; no longer U$58.CLKO, U$59.CLKI
- net N$139: now also U62.3, U63.4; no longer U$59.SDO, U$60.SDI
- net N$140: now also U63.2, U64.5; no longer U$59.CLKO, U$60.CLKI
- net N$141: now also U63.3, U64.4; no longer U$60.SDO, U$61.SDI
- net N$142: now also U64.2, U65.5; no longer U$60.CLKO, U$61.CLKI
- net N$143: now also U64.3, U65.4; no longer U$61.SDO, U$62.SDI
- net N$144: now also U65.2, U66.5; no longer U$61.CLKO, U$62.CLKI
- net N$145: now also U65.3, U66.4; no longer U$62.SDO, U$63.SDI
- net N$146: now also U66.2, U67.5; no longer U$62.CLKO, U$63.CLKI
- net N$147: now also U66.3, U67.4; no longer U$63.SDO, U$64.SDI
- net N$148: now also U67.2, U69.5; no longer U$63.CLKO, U$64.CLKI
- net N$149: now also U67.3, U69.4; no longer U$64.SDO, U$65.SDI
- net N$150: now also U68.5, U69.2; no longer U$64.CLKO, U$65.CLKI
- net N$151: now also U68.4, U69.3; no longer U$65.SDO, U$66.SDI
- net N$152: now also U70.2, U71.5; no longer U$65.CLKO, U$66.CLKI
- net N$153: now also U70.3, U71.4; no longer U$66.SDO, U$67.SDI
- net N$154: now also U68.2, U70.5; no longer U$66.CLKO, U$67.CLKI
- net N$155: now also U68.3, U70.4; no longer U$67.SDO, U$68.SDI
- net N$156: now also U71.2, U72.5; no longer U$67.CLKO, U$68.CLKI
- net N$157: now also U71.3, U72.4; no longer U$68.SDO, U$69.SDI
- net N$158: now also U72.2, U73.5; no longer U$68.CLKO, U$69.CLKI
- net N$159: now also U72.3, U73.4; no longer U$69.SDO, U$70.SDI
- net N$16: now also U6.3, U7.4; no longer R4.2, U$37.CLKI
- net N$160: now also U73.2, U74.5; no longer U$69.CLKO, U$70.CLKI
- net N$161: now also U73.3, U74.4; no longer U$70.SDO, U$71.SDI
- net N$162: now also U74.2, U75.5; no longer U$70.CLKO, U$71.CLKI
- net N$163: now also U74.3, U75.4; no longer U$71.SDO, U$72.SDI
- net N$164: now also U75.2, U76.5; no longer U$71.CLKO, U$72.CLKI
- net N$165: now also U75.3, U76.4; no longer U$72.SDO, U$73.SDI
- net N$17: now also U7.2, U8.5; no longer U$1.SDO, U$3.SDI
- net N$18: now also U7.3, U8.4; no longer R5.2, U$2.CLKI
- net N$20: now also U8.2, U9.5; no longer U$1.CLKO, U$3.CLKI
- net N$24: now also U8.3, U9.4; no longer U$11.CLKO, U$12.CLKI
- net N$25: now also U10.5, U9.2; no longer U$12.SDO, U$13.SDI
- net N$27: now also U10.4, U9.3; no longer U$12.CLKO, U$13.CLKI
- net N$28: now also U10.2, U11.5; no longer U$13.SDO, U$14.SDI
- net N$29: now also U10.3, U11.4; no longer U$3.SDO, U$4.SDI
- net N$30: now also U11.2, U12.5; no longer U$3.CLKO, U$4.CLKI
- net N$31: now also U11.3, U12.4; no longer U$13.CLKO, U$14.CLKI
- net N$32: now also U12.2, U13.5; no longer U$14.SDO, U$15.SDI
- net N$33: now also U12.3, U13.4; no longer U$14.CLKO, U$15.CLKI
- net N$34: now also U13.2, U14.5; no longer U$4.SDO, U$5.SDI
- net N$35: now also U13.3, U14.4; no longer U$4.CLKO, U$5.CLKI
- net N$36: now also U14.2, U15.5; no longer U$15.SDO, U$16.SDI
- net N$37: now also U14.3, U15.4; no longer U$15.CLKO, U$16.CLKI
- net N$38: now also U15.2, U17.5; no longer U$16.SDO, U$17.SDI
- net N$39: now also U15.3, U17.4; no longer U$16.CLKO, U$17.CLKI
- net N$40: now also U16.5, U17.2; no longer U$5.SDO, U$6.SDI
- net N$41: now also U16.4, U17.3; no longer U$5.CLKO, U$6.CLKI
- net N$42: now also U18.2, U19.5; no longer U$17.SDO, U$18.SDI
- net N$43: now also U18.3, U19.4; no longer U$17.CLKO, U$18.CLKI
- net N$44: now also U16.2, U18.5; no longer R6.1, U$55.CLKI
- net N$46: now also U16.3, U18.4; no longer U$6.SDO, U$7.SDI
- net N$47: now also U19.2, U20.5; no longer R7.2, U$2.SDI
- net N$48: now also U19.3, U20.4; no longer U$19.SDO, U$20.SDI
- net N$49: now also U20.2, U21.5; no longer U$19.CLKO, U$20.CLKI
- net N$5: no longer JP2.2
- net N$51: now also U20.3, U21.4; no longer U$20.SDO, U$21.SDI
- net N$52: now also U21.2, U22.5; no longer U$20.CLKO, U$21.CLKI
- net N$53: now also U21.3, U22.4; no longer U$21.SDO, U$22.SDI
- net N$54: now also U22.2, U23.5; no longer U$6.CLKO, U$7.CLKI
- net N$55: now also U22.3, U23.4; no longer U$21.CLKO, U$22.CLKI
- net N$56: now also U23.2, U24.5; no longer U$22.SDO, U$23.SDI
- net N$57: now also U23.3, U24.4; no longer U$22.CLKO, U$23.CLKI
- net N$58: now also U24.2, U25.5; no longer U$23.SDO, U$24.SDI
- net N$59: now also U24.3, U25.4; no longer U$23.CLKO, U$24.CLKI
- net N$60: now also U25.2, U26.5; no longer U$7.SDO, U$8.SDI
- net N$61: now also U25.3, U26.4; no longer U$24.SDO, U$25.SDI
- net N$62: now also U26.2, U27.5; no longer U$7.CLKO, U$8.CLKI
- net N$63: now also U26.3, U27.4; no longer U$24.CLKO, U$25.CLKI
- net N$64: now also U27.2, U28.5; no longer U$25.SDO, U$26.SDI
- net N$65: now also U27.3, U28.4; no longer U$25.CLKO, U$26.CLKI
- net N$66: now also U28.2, U30.5; no longer U$8.SDO, U$9.SDI
- net N$67: now also U28.3, U30.4; no longer U$8.CLKO, U$9.CLKI
- net N$68: now also U29.5, U30.2; no longer U$26.SDO, U$27.SDI
- net N$69: now also U29.4, U30.3; no longer U$26.CLKO, U$27.CLKI
- net N$7: now also U5.2, U6.5; no longer U$10.SDO, U$11.SDI
- net N$70: now also U31.2, U32.5; no longer U$10.SDI, U$9.SDO
- net N$71: now also U31.3, U32.4; no longer U$10.CLKI, U$9.CLKO
- net N$72: now also U29.2, U31.5; no longer U$27.SDO, U$28.SDI
- net N$73: now also U29.3, U31.4; no longer U$27.CLKO, U$28.CLKI
- net N$74: now also U32.2, U33.5; no longer R8.2, U$37.SDI
- net N$75: now also U32.3, U33.4; no longer U$28.SDO, U$29.SDI
- net N$76: now also U33.2, U34.5; no longer U$28.CLKO, U$29.CLKI
- net N$77: now also U33.3, U34.4; no longer U$29.SDO, U$30.SDI
- net N$78: now also U34.2, U35.5; no longer U$29.CLKO, U$30.CLKI
- net N$79: now also U34.3, U35.4; no longer U$30.SDO, U$31.SDI
- net N$8: now also U5.3, U6.4; no longer U$10.CLKO, U$11.CLKI
- net N$80: now also U35.2, U36.5; no longer U$30.CLKO, U$31.CLKI
- net N$81: now also U35.3, U36.4; no longer U$31.SDO, U$32.SDI
- net N$82: now also U36.2, U37.5; no longer U$31.CLKO, U$32.CLKI
- net N$83: now also U36.3, U37.4; no longer U$32.SDO, U$33.SDI
- net N$84: now also U37.2, U38.5; no longer U$32.CLKO, U$33.CLKI
- net N$85: now also U37.3, U38.4; no longer U$33.SDO, U$34.SDI
- net N$86: now also U38.2, U39.5; no longer U$33.CLKO, U$34.CLKI
- net N$87: now also U38.3, U39.4; no longer U$34.SDO, U$35.SDI
- net N$88: now also U39.2, U40.5; no longer U$34.CLKO, U$35.CLKI
- net N$89: now also U39.3, U40.4; no longer U$35.SDO, U$36.SDI
- net N$9: now also U2.2, U5.5; no longer U$1.CLKI, U$2.CLKO
- net N$90: now also U40.2, U41.5; no longer U$35.CLKO, U$36.CLKI
- net N$91: now also U40.3, U41.4; no longer R9.1, U$19.SDI
- net N$93: now also U41.2, U43.5; no longer U$37.SDO, U$38.SDI
- net N$94: now also U41.3, U43.4; no longer U$37.CLKO, U$38.CLKI
- net N$95: now also U42.5, U43.2; no longer R10.1, U$55.SDI
- net N$96: now also U42.4, U43.3; no longer U$38.SDO, U$39.SDI
- net N$97: now also U44.2, U45.5; no longer U$38.CLKO, U$39.CLKI
- net N$98: now also U44.3, U45.4; no longer U$39.SDO, U$40.SDI
- net N$99: now also U42.2, U44.5; no longer U$39.CLKO, U$40.CLKI
Routing:
- net GND: track 849.5 -> 582.3 mm
- net +5V: track 267.2 -> 391.9 mm, vias 2 -> 4
- net +15V: track 147.2 -> 33.8 mm, vias 2 -> 0
- net N$18: track 35.0 -> 1.10 mm, vias 1 -> 0
- net +3V3: track 113.1 -> 93.6 mm
- net N$5: track 29.0 -> 21.6 mm
- net N$3: track 0.00 -> 3.06 mm
- net N$10: track 0.00 -> 1.10 mm
- net N$47: track 0.00 -> 1.10 mm
- net N$44: track 0.00 -> 1.10 mm
- net N$95: track 0.00 -> 1.10 mm
- net N$91: track 0.00 -> 1.10 mm
- net N$74: track 0.00 -> 1.10 mm
- net N$9: track 1.10 -> 0.00 mm
- net N$6: track 1.10 -> 0.00 mm
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- added copper zone on layer 16, net +5V

Commit message: a
Parts:
- removed C21: (no value), rcl:B/3528-21W
- removed R14: 4.7uH, rcl:R0805
- added C1, C9: (no value), resistor:C0805
- added C10, C11: 0.1uF, rcl:C0603
- added C24, C3: 10uF, rcl:C1206
- added FB1: 30Ω/1.8A, SparkFun-Coils:0603
- added L2: 4.7uH, rcl:L2825P
- added R16: 20k, rcl:R0603
- added U4: EMB1061, EMB1061:EMB1061
- C2, C4, C5, C6, C7, C8: value (none) -> 0.1uF; device resistor:C0805 -> rcl:C0603
- C20: value (none) -> 1uF
- R1: device resistor:R0805 -> resistor:R0603
- moved R9 34.9 mm to (-67.5, 7.30), turned to 180 degrees
- moved R3 28.3 mm to (-67.5, 8.70), turned to 180 degrees
- moved R2 17.8 mm to (-54.4, 3.00)
- moved C4 16.2 mm to (-38.2, -2.45), turned to 90 degrees
- moved C7 15.3 mm to (-53.2, -1.65)
- moved R13 10.5 mm to (44.2, -4.00), turned to 0 degrees
- moved R15 7.20 mm to (-31.0, -0.10), turned to 180 degrees
- moved R11 6.80 mm to (45.0, -2.00), turned to 270 degrees
- moved R12 6.63 mm to (49.0, -3.30), turned to 0 degrees
- moved C8 3.62 mm to (-53.2, 1.25), turned to 270 degrees
- moved C16 3.13 mm to (49.2, -0.40), turned to 270 degrees
- moved R1 1.55 mm to (-55.0, -5.80), flipped to the bottom
- moved U$74 1.49 mm to (47.2, 0.00), turned to 270 degrees
- moved C17 1.30 mm to (42.4, 1.60), turned to 90 degrees
- moved R5 0.50 mm to (-54.5, 6.20)
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Connections:
- removed net N$15 (its old number): R3.2, U1.29
- new net CKI_1: U2.5
- new net N$166: R9.2, U4.P$10
- new net N$169: R3.2, U4.P$11
- new net N$6: R16.1, U$74.5
- new net N$62: C20.1, FB1.1, U3.5
- new net SDI_1: U2.4
- net +15V: now also C1.1, R16.2; no longer U$74.5
- net +3V3: now also C10.1, C11.1, FB1.2, U4.P$8; no longer C20.1, U3.5
- net +5V: now also C24.1, C3.1, C9.1, L2.1; no longer C21.+, R14.2
- net GND: now also C1.2, C10.2, C11.2, C24.2, C3.2, C9.2, U4.P$22, U4.P$9; no longer C21.-
- net N$129: now also L2.2; no longer R14.1
- net N$92: no longer R9.2
Routing:
- net GND: track 582.3 -> 562.9 mm, vias 3 -> 25
- net N$12: track 44.8 -> 25.6 mm, vias 0 -> 1
- net N$5: track 21.6 -> 3.15 mm
- net +5V: track 391.9 -> 375.7 mm, vias 4 -> 15
- net +3V3: track 93.6 -> 108.8 mm
- net N$6: track 0.00 -> 12.8 mm, vias 0 -> 2
- net +15V: track 33.8 -> 22.4 mm
- net N$62: track 0.00 -> 7.53 mm
- net N$129: track 12.5 -> 6.12 mm
- net N$168: track 3.21 -> 6.14 mm
- net N$19: track 2.77 -> 0.00 mm
- net N$14: track 14.1 -> 16.3 mm
- net N$13: track 28.2 -> 30.2 mm, vias 0 -> 1
- net N$167: track 2.54 -> 1.26 mm
- net N$9: track 0.00 -> 1.10 mm
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- added copper zone on layer 1, net +15V
- added copper zone on layer 1, net +3V3
- added copper zone on layer 1, net +5V
- added copper zone on layer 15, net +5V
- added copper zone on layer 2, net GND

Commit message: sdf
Parts:
- removed R10, R7, R8: (no value), resistor:R0603
- added C12, C13, C14: 0.1uF, rcl:C0603
- added JP2: (no value), pinhead:1X03
- C1: value (none) -> 0.1uF; device resistor:C0805 -> rcl:C0603
- moved R4 35.9 mm to (-74.6, -8.70), turned to 180 degrees
- moved R6 21.8 mm to (-52.0, 7.80), turned to 180 degrees
- moved R2 16.3 mm to (-38.5, 6.60)
- moved R9 14.3 mm to (-53.9, 3.00), turned to 90 degrees
- moved R3 9.53 mm to (-71.4, 0.00), turned to 270 degrees
- moved R5 2.52 mm to (-52.0, 5.90)
- moved C7 1.34 mm to (-53.8, -2.85)
- moved C6 1.30 mm to (-51.4, -6.90)
- moved C8 1.25 mm to (-53.8, 0.15)
- moved C10 0.20 mm to (-38.1, -4.90)
- moved C11 0.20 mm to (-71.5, -5.90)
- moved C16 0.20 mm to (49.0, -0.40)
- moved C20 0.20 mm to (-34.1, -3.00)
- moved D3 0.20 mm to (37.5, 5.30)
- moved D5 0.20 mm to (37.5, -5.30)
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Connections:
- net N$166 renamed BLE_TX
- net N$169 renamed BLE_RX
- removed net N$112: R10.2, U1.5
- removed net N$45 (its old number): R6.2, U1.4
- new net N$19: R3.1, U1.50
- net +3V3: now also R4.1
- net +5V: now also C12.1, C13.1, C14.1, JP2.1
- net CKI_1: now also R5.2
- net GND: now also C12.2, C13.2, C14.2, JP2.2
- net N$21: now also R6.1, U1.48; no longer R4.1, U1.44
- net N$4: now also R9.1, U1.51; no longer R7.1, U1.48
- net N$5: now also R4.2, U4.P$3; no longer R2.2, U1.50
- net N$50: now also JP2.3, R2.2, U1.30; no longer R8.1, U1.45
- net SDI_1: now also R6.2
Routing:
- net N$50: track 0.00 -> 144.2 mm, vias 0 -> 1
- net SDI_1: track 0.00 -> 50.2 mm, vias 0 -> 1
- net CKI_1: track 0.00 -> 46.2 mm, vias 0 -> 1
- net N$19: track 0.00 -> 22.7 mm
- net BLE_TX: track 0.00 -> 22.6 mm
- net +3V3: track 108.8 -> 87.9 mm, vias 0 -> 13
- net GND: track 562.9 -> 577.8 mm, vias 25 -> 33
- net N$5: track 3.15 -> 12.4 mm
- net N$21: track 0.00 -> 2.99 mm
- net +5V: track 375.7 -> 378.3 mm
- net N$4: track 0.00 -> 2.42 mm
- net BLE_RX: track 0.00 -> 2.37 mm
- net N$45: track 0.00 -> 2.35 mm
- net +15V: track 22.4 -> 23.0 mm
- added copper zone on layer 15, net +3V3
