File: POVRotorV2/POVRotor.sch (EAGLE design)
At the start: 108 parts, among them U1 PIC32MZ2048EFH064-I/PT

Commit message: a
Parts:
- added R15: 41k, rcl:R-US_R0603
Connections:
- new net N$3: R15.1, U$74.EN
- net +15V: now also R15.2; no longer U$74.EN
Changed lines of the file:
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@@
 <?xml version="1.0" encoding="utf-8"?>
 <!DOCTYPE eagle SYSTEM "eagle.dtd">
-<eagle version="9.3.1">
+<eagle version="9.4.2">
 <drawing>
 <settings>
@@
 <part name="SUPPLY17" library="supply2" library_urn="urn:adsk.eagle:library:372" deviceset="GND" device=""/>
 <part name="SUPPLY18" library="supply2" library_urn="urn:adsk.eagle:library:372" deviceset="GND" device=""/>
+<part name="R15" library="rcl" library_urn="urn:adsk.eagle:library:334" deviceset="R-US_" device="R0603" package3d_urn="urn:adsk.eagle:package:23555/3" value="41k"/>
 </parts>
 <sheets>
@@
 <attribute name="VALUE" x="48.895" y="116.205" size="1.778" layer="96"/>
 </instance>
+<instance part="R15" gate="G$1" x="22.86" y="142.24" smashed="yes" rot="R180">
+<attribute name="NAME" x="15.494" y="142.4686" size="1.778" layer="95"/>
+<attribute name="VALUE" x="25.908" y="142.494" size="1.778" layer="96"/>
+</instance>
 </instances>
 <busses>
@@
 <wire x1="12.7" y1="132.08" x2="5.08" y2="132.08" width="0.1524" layer="91"/>
 <wire x1="5.08" y1="132.08" x2="5.08" y2="142.24" width="0.1524" layer="91"/>
-<pinref part="U$74" gate="G$1" pin="EN"/>
 <wire x1="5.08" y1="142.24" x2="5.08" y2="149.86" width="0.1524" layer="91"/>
-<wire x1="33.02" y1="134.62" x2="35.56" y2="134.62" width="0.1524" layer="91"/>
-<wire x1="35.56" y1="134.62" x2="35.56" y2="142.24" width="0.1524" layer="91"/>
-<wire x1="35.56" y1="142.24" x2="5.08" y2="142.24" width="0.1524" layer="91"/>
 <junction x="5.08" y="142.24"/>
 <wire x1="-2.54" y1="137.16" x2="-2.54" y2="142.24" width="0.1524" layer="91"/>
@@
 <pinref part="C17" gate="G$1" pin="+"/>
 <pinref part="SUPPLY16" gate="+15V" pin="+15V"/>
+<pinref part="R15" gate="G$1" pin="2"/>
+<wire x1="17.78" y1="142.24" x2="5.08" y2="142.24" width="0.1524" layer="91"/>
 </segment>
 </net>
@@
 </segment>
 </net>
+<net name="N$3" class="0">
+<segment>
+<wire x1="35.56" y1="134.62" x2="35.56" y2="142.24" width="0.1524" layer="91"/>
+<pinref part="U$74" gate="G$1" pin="EN"/>
+<wire x1="33.02" y1="134.62" x2="35.56" y2="134.62" width="0.1524" layer="91"/>
+<pinref part="R15" gate="G$1" pin="1"/>
+<wire x1="27.94" y1="142.24" x2="35.56" y2="142.24" width="0.1524" layer="91"/>
+</segment>
+</net>
