File: POVRotorV2/POVRotor.sch (EAGLE design)
At the start: 102 parts, among them IC1 LM2576S, U1 PIC32MZ2048EFH064-I/PT

Commit message: a
Parts:
- removed C1, C3: (no value), resistor:CPOL-USE2,5-6E
- removed D1: (no value), telefunken:BYS10
- removed IC1: LM2576S, lm2576:LM2576S
- removed L2: (no value), resistor:L-USL4532P
- added C16: 0.1uF, rcl:C-EUC0603
- added C17: (no value), rcl:CPOL-USC/6032-28R
- added R10, R7, R8, R9: (no value), resistor:R-US_R0603
- added R11: 75k, rcl:R-US_R0603
- added R12: 41k, rcl:R-US_R0603
- added R13: 7.6k, rcl:R-US_R0603
- added R14: 4.7uH, rcl:R-EU_R0805
- added U$74: AP65211A, SOT95P280X140-6N:AP65211A
Connections:
- removed net N$3: D1.K, IC1.OUT, L2.1
- new net N$112: R10.2, U1.AN13/C1INC/RPG7/SDA4/PMA4/RG7
- new net N$129: C16.1, R14.1, U$74.SW
- new net N$130: C16.2, U$74.BST
- new net N$167: R11.1, U$74.FB
- new net N$168: R11.2, R12.1, R13.2
- new net N$4: R7.1, U1.SOSCO/RPC14/T1CK/RC14
- new net N$47: R7.2, U$2.SDI
- new net N$50: R8.1, U1.AERXCLK/AEREFCLK/ECRS/RPD11/PMCS1/PMA14/RD11
- new net N$74: R8.2, U$37.SDI
- new net N$91: R9.1, U$19.SDI
- new net N$92: R9.2, U1.TMS/CVREFOUT/AN5/RPB10/PMA13/RB10
- new net N$95: R10.1, U$55.SDI
- net +15V: now also C17.+, U$74.EN, U$74.IN; no longer C3.+, IC1.VIN
- net +5V: now also R12.2, R14.2; no longer C1.+, IC1.FB, L2.2
- net GND: now also C17.-, R13.1, U$74.GND; no longer C1.-, C3.-, D1.A, IC1.GND, IC1.OFF

Commit message: s
Parts:
- removed C10, C11, C12, C9: (no value), resistor:C-USC0805
- removed IC2: (no value), lm2576:LM1117
- removed JP2: (no value), pinhead:PINHD-1X4
- removed U$1, U$10, U$11, U$12, U$13, U$14, U$15, U$16, U$17, U$18, U$19, U$2, U$20, U$21, U$22, U$23, U$24, U$25, U$26, U$27, U$28, U$29, U$3, U$30, U$31, U$32, U$33, U$34, U$35, U$36, U$37, U$38, U$39, U$4, U$40, U$41, U$42, U$43, U$44, U$45, U$46, U$47, U$48, U$49, U$5, U$50, U$51, U$52, U$53, U$54, U$55, U$56, U$57, U$58, U$59, U$6, U$60, U$61, U$62, U$63, U$64, U$65, U$66, U$67, U$68, U$69, U$7, U$70, U$71, U$72, U$73, U$8, U$9: 2020LED, APA2020:2020LED
- added C20: (no value), rcl:C-USC0805
- added C21: (no value), rcl:CPOL-USB/3528-21W
- added R15: 75k, rcl:R-US_R0603
- added U10, U11, U12, U13, U14, U15, U16, U17, U18, U19, U2, U20, U21, U22, U23, U24, U25, U26, U27, U28, U29, U30, U31, U32, U33, U34, U35, U36, U37, U38, U39, U40, U41, U42, U43, U44, U45, U46, U47, U48, U49, U5, U50, U51, U52, U53, U54, U55, U56, U57, U58, U59, U6, U60, U61, U62, U63, U64, U65, U66, U67, U68, U69, U7, U70, U71, U72, U73, U74, U75, U76, U8, U9: 3341, APA102:3341
- added U3: TLV75533PDBVR, TLV75533PDBVR:TLV75533PDBVR
Connections:
- removed net N$166: U$72.CLKO, U$73.CLKI
- removed net N$6: U$1.SDI, U$2.SDO
- new net N$3: R15.2, U3.EN
- net +3V3: now also C20.1, U3.OUT; no longer IC2.OUT, JP2.1
- net +5V: now also C21.+, R15.1, U10.VDD, U11.VDD, U12.VDD, U13.VDD, U14.VDD, U15.VDD, U16.VDD, U17.VDD, U18.VDD, U19.VDD, U2.VDD, U20.VDD, U21.VDD, U22.VDD, U23.VDD, U24.VDD, U25.VDD, U26.VDD, U27.VDD, U28.VDD, U29.VDD, U3.IN, U30.VDD, U31.VDD, U32.VDD, U33.VDD, U34.VDD, U35.VDD, U36.VDD, U37.VDD, U38.VDD, U39.VDD, U40.VDD, U41.VDD, U42.VDD, U43.VDD, U44.VDD, U45.VDD, U46.VDD, U47.VDD, U48.VDD, U49.VDD, U5.VDD, U50.VDD, U51.VDD, U52.VDD, U53.VDD, U54.VDD, U55.VDD, U56.VDD, U57.VDD, U58.VDD, U59.VDD, U6.VDD, U60.VDD, U61.VDD, U62.VDD, U63.VDD, U64.VDD, U65.VDD, U66.VDD, U67.VDD, U68.VDD, U69.VDD, U7.VDD, U70.VDD, U71.VDD, U72.VDD, U73.VDD, U74.VDD, U75.VDD, U76.VDD, U8.VDD, U9.VDD; no longer C10.1, C11.1, C12.1, C9.1, IC2.IN, U$1.VCC, U$10.VCC, U$11.VCC, U$12.VCC, U$13.VCC, U$14.VCC, U$15.VCC, U$16.VCC, U$17.VCC, U$18.VCC, U$19.VCC, U$2.VCC, U$20.VCC, U$21.VCC, U$22.VCC, U$23.VCC, U$24.VCC, U$25.VCC, U$26.VCC, U$27.VCC, U$28.VCC, U$29.VCC, U$3.VCC, U$30.VCC, U$31.VCC, U$32.VCC, U$33.VCC, U$34.VCC, U$35.VCC, U$36.VCC, U$37.VCC, U$38.VCC, U$39.VCC, U$4.VCC, U$40.VCC, U$41.VCC, U$42.VCC, U$43.VCC, U$44.VCC, U$45.VCC, U$46.VCC, U$47.VCC, U$48.VCC, U$49.VCC, U$5.VCC, U$50.VCC, U$51.VCC, U$52.VCC, U$53.VCC, U$54.VCC, U$55.VCC, U$56.VCC, U$57.VCC, U$58.VCC, U$59.VCC, U$6.VCC, U$60.VCC, U$61.VCC, U$62.VCC, U$63.VCC, U$64.VCC, U$65.VCC, U$66.VCC, U$67.VCC, U$68.VCC, U$69.VCC, U$7.VCC, U$70.VCC, U$71.VCC, U$72.VCC, U$73.VCC, U$8.VCC, U$9.VCC
- net GND: now also C20.2, C21.-, U10.GND, U11.GND, U12.GND, U13.GND, U14.GND, U15.GND, U16.GND, U17.GND, U18.GND, U19.GND, U2.GND, U20.GND, U21.GND, U22.GND, U23.GND, U24.GND, U25.GND, U26.GND, U27.GND, U28.GND, U29.GND, U3.GND, U30.GND, U31.GND, U32.GND, U33.GND, U34.GND, U35.GND, U36.GND, U37.GND, U38.GND, U39.GND, U40.GND, U41.GND, U42.GND, U43.GND, U44.GND, U45.GND, U46.GND, U47.GND, U48.GND, U49.GND, U5.GND, U50.GND, U51.GND, U52.GND, U53.GND, U54.GND, U55.GND, U56.GND, U57.GND, U58.GND, U59.GND, U6.GND, U60.GND, U61.GND, U62.GND, U63.GND, U64.GND, U65.GND, U66.GND, U67.GND, U68.GND, U69.GND, U7.GND, U70.GND, U71.GND, U72.GND, U73.GND, U74.GND, U75.GND, U76.GND, U8.GND, U9.GND; no longer C10.2, C11.2, C12.2, C9.2, IC2.GND, JP2.4, U$1.GND, U$10.GND, U$11.GND, U$12.GND, U$13.GND, U$14.GND, U$15.GND, U$16.GND, U$17.GND, U$18.GND, U$19.GND, U$2.GND, U$20.GND, U$21.GND, U$22.GND, U$23.GND, U$24.GND, U$25.GND, U$26.GND, U$27.GND, U$28.GND, U$29.GND, U$3.GND, U$30.GND, U$31.GND, U$32.GND, U$33.GND, U$34.GND, U$35.GND, U$36.GND, U$37.GND, U$38.GND, U$39.GND, U$4.GND, U$40.GND, U$41.GND, U$42.GND, U$43.GND, U$44.GND, U$45.GND, U$46.GND, U$47.GND, U$48.GND, U$49.GND, U$5.GND, U$50.GND, U$51.GND, U$52.GND, U$53.GND, U$54.GND, U$55.GND, U$56.GND, U$57.GND, U$58.GND, U$59.GND, U$6.GND, U$60.GND, U$61.GND, U$62.GND, U$63.GND, U$64.GND, U$65.GND, U$66.GND, U$67.GND, U$68.GND, U$69.GND, U$7.GND, U$70.GND, U$71.GND, U$72.GND, U$73.GND, U$8.GND, U$9.GND
- net N$10: now also U2.SDO, U5.SDI; no longer R3.1, U$19.CLKI
- net N$100: now also U42.SDO, U44.SDI; no longer U$40.SDO, U$41.SDI
- net N$101: now also U45.CKO, U46.CKI; no longer U$40.CLKO, U$41.CLKI
- net N$102: now also U45.SDO, U46.SDI; no longer U$41.SDO, U$42.SDI
- net N$103: now also U46.CKO, U47.CKI; no longer U$41.CLKO, U$42.CLKI
- net N$104: now also U46.SDO, U47.SDI; no longer U$42.SDO, U$43.SDI
- net N$105: now also U47.CKO, U48.CKI; no longer U$42.CLKO, U$43.CLKI
- net N$106: now also U47.SDO, U48.SDI; no longer U$43.SDO, U$44.SDI
- net N$107: now also U48.CKO, U49.CKI; no longer U$43.CLKO, U$44.CLKI
- net N$108: now also U48.SDO, U49.SDI; no longer U$44.SDO, U$45.SDI
- net N$109: now also U49.CKO, U50.CKI; no longer U$44.CLKO, U$45.CLKI
- net N$11: now also U6.CKO, U7.CKI; no longer U$11.SDO, U$12.SDI
- net N$110: now also U49.SDO, U50.SDI; no longer U$45.SDO, U$46.SDI
- net N$111: now also U50.CKO, U51.CKI; no longer U$45.CLKO, U$46.CLKI
- net N$113: now also U50.SDO, U51.SDI; no longer U$46.SDO, U$47.SDI
- net N$114: now also U51.CKO, U52.CKI; no longer U$46.CLKO, U$47.CLKI
- net N$115: now also U51.SDO, U52.SDI; no longer U$47.SDO, U$48.SDI
- net N$116: now also U52.CKO, U53.CKI; no longer U$47.CLKO, U$48.CLKI
- net N$117: now also U52.SDO, U53.SDI; no longer U$48.SDO, U$49.SDI
- net N$118: now also U53.CKO, U54.CKI; no longer U$48.CLKO, U$49.CLKI
- net N$119: now also U53.SDO, U54.SDI; no longer U$49.SDO, U$50.SDI
- net N$120: now also U54.CKO, U56.CKI; no longer U$49.CLKO, U$50.CLKI
- net N$121: now also U54.SDO, U56.SDI; no longer U$50.SDO, U$51.SDI
- net N$122: now also U55.CKI, U56.CKO; no longer U$50.CLKO, U$51.CLKI
- net N$123: now also U55.SDI, U56.SDO; no longer U$51.SDO, U$52.SDI
- net N$124: now also U57.CKO, U58.CKI; no longer U$51.CLKO, U$52.CLKI
- net N$125: now also U57.SDO, U58.SDI; no longer U$52.SDO, U$53.SDI
- net N$126: now also U55.CKO, U57.CKI; no longer U$52.CLKO, U$53.CLKI
- net N$127: now also U55.SDO, U57.SDI; no longer U$53.SDO, U$54.SDI
- net N$128: now also U58.CKO, U59.CKI; no longer U$53.CLKO, U$54.CLKI
- net N$131: now also U58.SDO, U59.SDI; no longer U$55.SDO, U$56.SDI
- net N$132: now also U59.CKO, U60.CKI; no longer U$55.CLKO, U$56.CLKI
- net N$133: now also U59.SDO, U60.SDI; no longer U$56.SDO, U$57.SDI
- net N$134: now also U60.CKO, U61.CKI; no longer U$56.CLKO, U$57.CLKI
- net N$135: now also U60.SDO, U61.SDI; no longer U$57.SDO, U$58.SDI
- net N$136: now also U61.CKO, U62.CKI; no longer U$57.CLKO, U$58.CLKI
- net N$137: now also U61.SDO, U62.SDI; no longer U$58.SDO, U$59.SDI
- net N$138: now also U62.CKO, U63.CKI; no longer U$58.CLKO, U$59.CLKI
- net N$139: now also U62.SDO, U63.SDI; no longer U$59.SDO, U$60.SDI
- net N$140: now also U63.CKO, U64.CKI; no longer U$59.CLKO, U$60.CLKI
- net N$141: now also U63.SDO, U64.SDI; no longer U$60.SDO, U$61.SDI
- net N$142: now also U64.CKO, U65.CKI; no longer U$60.CLKO, U$61.CLKI
- net N$143: now also U64.SDO, U65.SDI; no longer U$61.SDO, U$62.SDI
- net N$144: now also U65.CKO, U66.CKI; no longer U$61.CLKO, U$62.CLKI
- net N$145: now also U65.SDO, U66.SDI; no longer U$62.SDO, U$63.SDI
- net N$146: now also U66.CKO, U67.CKI; no longer U$62.CLKO, U$63.CLKI
- net N$147: now also U66.SDO, U67.SDI; no longer U$63.SDO, U$64.SDI
- net N$148: now also U67.CKO, U69.CKI; no longer U$63.CLKO, U$64.CLKI
- net N$149: now also U67.SDO, U69.SDI; no longer U$64.SDO, U$65.SDI
- net N$150: now also U68.CKI, U69.CKO; no longer U$64.CLKO, U$65.CLKI
- net N$151: now also U68.SDI, U69.SDO; no longer U$65.SDO, U$66.SDI
- net N$152: now also U70.CKO, U71.CKI; no longer U$65.CLKO, U$66.CLKI
- net N$153: now also U70.SDO, U71.SDI; no longer U$66.SDO, U$67.SDI
- net N$154: now also U68.CKO, U70.CKI; no longer U$66.CLKO, U$67.CLKI
- net N$155: now also U68.SDO, U70.SDI; no longer U$67.SDO, U$68.SDI
- net N$156: now also U71.CKO, U72.CKI; no longer U$67.CLKO, U$68.CLKI
- net N$157: now also U71.SDO, U72.SDI; no longer U$68.SDO, U$69.SDI
- net N$158: now also U72.CKO, U73.CKI; no longer U$68.CLKO, U$69.CLKI
- net N$159: now also U72.SDO, U73.SDI; no longer U$69.SDO, U$70.SDI
- net N$16: now also U6.SDO, U7.SDI; no longer R4.2, U$37.CLKI
- net N$160: now also U73.CKO, U74.CKI; no longer U$69.CLKO, U$70.CLKI
- net N$161: now also U73.SDO, U74.SDI; no longer U$70.SDO, U$71.SDI
- net N$162: now also U74.CKO, U75.CKI; no longer U$70.CLKO, U$71.CLKI
- net N$163: now also U74.SDO, U75.SDI; no longer U$71.SDO, U$72.SDI
- net N$164: now also U75.CKO, U76.CKI; no longer U$71.CLKO, U$72.CLKI
- net N$165: now also U75.SDO, U76.SDI; no longer U$72.SDO, U$73.SDI
- net N$17: now also U7.CKO, U8.CKI; no longer U$1.SDO, U$3.SDI
- net N$18: now also U7.SDO, U8.SDI; no longer R5.2, U$2.CLKI
- net N$20: now also U8.CKO, U9.CKI; no longer U$1.CLKO, U$3.CLKI
- net N$24: now also U8.SDO, U9.SDI; no longer U$11.CLKO, U$12.CLKI
- net N$25: now also U10.CKI, U9.CKO; no longer U$12.SDO, U$13.SDI
- net N$27: now also U10.SDI, U9.SDO; no longer U$12.CLKO, U$13.CLKI
- net N$28: now also U10.CKO, U11.CKI; no longer U$13.SDO, U$14.SDI
- net N$29: now also U10.SDO, U11.SDI; no longer U$3.SDO, U$4.SDI
- net N$30: now also U11.CKO, U12.CKI; no longer U$3.CLKO, U$4.CLKI
- net N$31: now also U11.SDO, U12.SDI; no longer U$13.CLKO, U$14.CLKI
- net N$32: now also U12.CKO, U13.CKI; no longer U$14.SDO, U$15.SDI
- net N$33: now also U12.SDO, U13.SDI; no longer U$14.CLKO, U$15.CLKI
- net N$34: now also U13.CKO, U14.CKI; no longer U$4.SDO, U$5.SDI
- net N$35: now also U13.SDO, U14.SDI; no longer U$4.CLKO, U$5.CLKI
- net N$36: now also U14.CKO, U15.CKI; no longer U$15.SDO, U$16.SDI
- net N$37: now also U14.SDO, U15.SDI; no longer U$15.CLKO, U$16.CLKI
- net N$38: now also U15.CKO, U17.CKI; no longer U$16.SDO, U$17.SDI
- net N$39: now also U15.SDO, U17.SDI; no longer U$16.CLKO, U$17.CLKI
- net N$40: now also U16.CKI, U17.CKO; no longer U$5.SDO, U$6.SDI
- net N$41: now also U16.SDI, U17.SDO; no longer U$5.CLKO, U$6.CLKI
- net N$42: now also U18.CKO, U19.CKI; no longer U$17.SDO, U$18.SDI
- net N$43: now also U18.SDO, U19.SDI; no longer U$17.CLKO, U$18.CLKI
- net N$44: now also U16.CKO, U18.CKI; no longer R6.1, U$55.CLKI
- net N$46: now also U16.SDO, U18.SDI; no longer U$6.SDO, U$7.SDI
- net N$47: now also U19.CKO, U20.CKI; no longer R7.2, U$2.SDI
- net N$48: now also U19.SDO, U20.SDI; no longer U$19.SDO, U$20.SDI
- net N$49: now also U20.CKO, U21.CKI; no longer U$19.CLKO, U$20.CLKI
- net N$5: no longer JP2.2
- net N$51: now also U20.SDO, U21.SDI; no longer U$20.SDO, U$21.SDI
- net N$52: now also U21.CKO, U22.CKI; no longer U$20.CLKO, U$21.CLKI
- net N$53: now also U21.SDO, U22.SDI; no longer U$21.SDO, U$22.SDI
- net N$54: now also U22.CKO, U23.CKI; no longer U$6.CLKO, U$7.CLKI
- net N$55: now also U22.SDO, U23.SDI; no longer U$21.CLKO, U$22.CLKI
- net N$56: now also U23.CKO, U24.CKI; no longer U$22.SDO, U$23.SDI
- net N$57: now also U23.SDO, U24.SDI; no longer U$22.CLKO, U$23.CLKI
- net N$58: now also U24.CKO, U25.CKI; no longer U$23.SDO, U$24.SDI
- net N$59: now also U24.SDO, U25.SDI; no longer U$23.CLKO, U$24.CLKI
- net N$60: now also U25.CKO, U26.CKI; no longer U$7.SDO, U$8.SDI
- net N$61: now also U25.SDO, U26.SDI; no longer U$24.SDO, U$25.SDI
- net N$62: now also U26.CKO, U27.CKI; no longer U$7.CLKO, U$8.CLKI
- net N$63: now also U26.SDO, U27.SDI; no longer U$24.CLKO, U$25.CLKI
- net N$64: now also U27.CKO, U28.CKI; no longer U$25.SDO, U$26.SDI
- net N$65: now also U27.SDO, U28.SDI; no longer U$25.CLKO, U$26.CLKI
- net N$66: now also U28.CKO, U30.CKI; no longer U$8.SDO, U$9.SDI
- net N$67: now also U28.SDO, U30.SDI; no longer U$8.CLKO, U$9.CLKI
- net N$68: now also U29.CKI, U30.CKO; no longer U$26.SDO, U$27.SDI
- net N$69: now also U29.SDI, U30.SDO; no longer U$26.CLKO, U$27.CLKI
- net N$7: now also U5.CKO, U6.CKI; no longer U$10.SDO, U$11.SDI
- net N$70: now also U31.CKO, U32.CKI; no longer U$10.SDI, U$9.SDO
- net N$71: now also U31.SDO, U32.SDI; no longer U$10.CLKI, U$9.CLKO
- net N$72: now also U29.CKO, U31.CKI; no longer U$27.SDO, U$28.SDI
- net N$73: now also U29.SDO, U31.SDI; no longer U$27.CLKO, U$28.CLKI
- net N$74: now also U32.CKO, U33.CKI; no longer R8.2, U$37.SDI
- net N$75: now also U32.SDO, U33.SDI; no longer U$28.SDO, U$29.SDI
- net N$76: now also U33.CKO, U34.CKI; no longer U$28.CLKO, U$29.CLKI
- net N$77: now also U33.SDO, U34.SDI; no longer U$29.SDO, U$30.SDI
- net N$78: now also U34.CKO, U35.CKI; no longer U$29.CLKO, U$30.CLKI
- net N$79: now also U34.SDO, U35.SDI; no longer U$30.SDO, U$31.SDI
- net N$8: now also U5.SDO, U6.SDI; no longer U$10.CLKO, U$11.CLKI
- net N$80: now also U35.CKO, U36.CKI; no longer U$30.CLKO, U$31.CLKI
- net N$81: now also U35.SDO, U36.SDI; no longer U$31.SDO, U$32.SDI
- net N$82: now also U36.CKO, U37.CKI; no longer U$31.CLKO, U$32.CLKI
- net N$83: now also U36.SDO, U37.SDI; no longer U$32.SDO, U$33.SDI
- net N$84: now also U37.CKO, U38.CKI; no longer U$32.CLKO, U$33.CLKI
- net N$85: now also U37.SDO, U38.SDI; no longer U$33.SDO, U$34.SDI
- net N$86: now also U38.CKO, U39.CKI; no longer U$33.CLKO, U$34.CLKI
- net N$87: now also U38.SDO, U39.SDI; no longer U$34.SDO, U$35.SDI
- net N$88: now also U39.CKO, U40.CKI; no longer U$34.CLKO, U$35.CLKI
- net N$89: now also U39.SDO, U40.SDI; no longer U$35.SDO, U$36.SDI
- net N$9: now also U2.CKO, U5.CKI; no longer U$1.CLKI, U$2.CLKO
- net N$90: now also U40.CKO, U41.CKI; no longer U$35.CLKO, U$36.CLKI
- net N$91: now also U40.SDO, U41.SDI; no longer R9.1, U$19.SDI
- net N$93: now also U41.CKO, U43.CKI; no longer U$37.SDO, U$38.SDI
- net N$94: now also U41.SDO, U43.SDI; no longer U$37.CLKO, U$38.CLKI
- net N$95: now also U42.CKI, U43.CKO; no longer R10.1, U$55.SDI
- net N$96: now also U42.SDI, U43.SDO; no longer U$38.SDO, U$39.SDI
- net N$97: now also U44.CKO, U45.CKI; no longer U$38.CLKO, U$39.CLKI
- net N$98: now also U44.SDO, U45.SDI; no longer U$39.SDO, U$40.SDI
- net N$99: now also U42.CKO, U44.CKI; no longer U$39.CLKO, U$40.CLKI

Commit message: a
Parts:
- removed C21: (no value), rcl:CPOL-USB/3528-21W
- removed R14: 4.7uH, rcl:R-EU_R0805
- added C1, C9: (no value), resistor:C-USC0805
- added C10, C11: 0.1uF, rcl:C-EUC0603
- added C24, C3: 10uF, rcl:C-EUC1206
- added FB1: 30Ω/1.8A, SparkFun-Coils:FERRITE_BEAD-0603
- added L2: 4.7uH, rcl:L-EUL2825P
- added R16: 20k, rcl:R-US_R0603
- added U4: EMB1061, EMB1061:EMB1061
- C2, C4, C5, C6, C7, C8: value (none) -> 0.1uF; device resistor:C-USC0805 -> rcl:C-EUC0603
- C20: value (none) -> 1uF
- R1: device resistor:R-US_R0805 -> resistor:R-US_R0603
Connections:
- removed net N$15 (its old number): R3.2, U1.AN9/RPB14/SCK3/PMA1/RB14
- new net CKI_1: U2.CKI
- new net N$166: R9.2, U4.UART_TXD
- new net N$169: R3.2, U4.UART_RXD
- new net N$6: R16.1, U$74.EN
- new net N$62: C20.1, FB1.1, U3.OUT
- new net SDI_1: U2.SDI
- net +15V: now also C1.1, R16.2; no longer U$74.EN
- net +3V3: now also C10.1, C11.1, FB1.2, U4.VCC; no longer C20.1, U3.OUT
- net +5V: now also C24.1, C3.1, C9.1, L2.1; no longer C21.+, R14.2
- net GND: now also C1.2, C10.2, C11.2, C24.2, C3.2, C9.2, U4.GND; no longer C21.-
- net N$129: now also L2.2; no longer R14.1
- net N$92: no longer R9.2
Other:
- moved on the sheet: C17, C2, C4, C5, C6, C7, C8, R3, R9
