File: New folder/Quad-4layer.brd (EAGLE design)
At the start: 58 x 67 mm, 105 parts, among them U1 CAT24C02, U2 TLV75533PDBVR, U3 SAM-M8Q, U6 TLV75533PDBVR, U7 TLV75533PDBVR, U8 TLV75533PDBVR

Commit message: sdf
Parts:
- removed C24, C36: 0.1uF, rcl:C0603
- moved C21 4.40 mm to (22.4, 26.6)
- moved R31 1.17 mm to (10.1, 16.7), turned to 90 degrees
Connections:
- net +5V: no longer C24.1, C36.1
- net GND: no longer C24.2, C36.2
Routing:
- net +5V: track 41.6 -> 43.7 mm
Changed lines of the file:
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@@
 <layers>
 <layer number="1" name="Top" color="4" fill="1" visible="yes" active="yes"/>
-<layer number="2" name="GND" color="16" fill="1" visible="no" active="yes"/>
+<layer number="2" name="GND" color="16" fill="1" visible="yes" active="yes"/>
 <layer number="3" name="Route3" color="17" fill="1" visible="no" active="no"/>
 <layer number="4" name="Route4" color="18" fill="1" visible="no" active="no"/>
@@
 <layer number="13" name="Route13" color="21" fill="1" visible="no" active="no"/>
 <layer number="14" name="Route14" color="22" fill="1" visible="no" active="no"/>
-<layer number="15" name="VDD" color="23" fill="1" visible="no" active="yes"/>
+<layer number="15" name="VDD" color="23" fill="1" visible="yes" active="yes"/>
 <layer number="16" name="Bottom" color="1" fill="1" visible="yes" active="yes"/>
 <layer number="17" name="Pads" color="2" fill="1" visible="yes" active="yes"/>
@@
 <layer number="23" name="tOrigins" color="52" fill="1" visible="yes" active="yes"/>
 <layer number="24" name="bOrigins" color="52" fill="1" visible="yes" active="yes"/>
-<layer number="25" name="tNames" color="7" fill="1" visible="yes" active="yes"/>
-<layer number="26" name="bNames" color="7" fill="1" visible="yes" active="yes"/>
+<layer number="25" name="tNames" color="7" fill="1" visible="no" active="yes"/>
+<layer number="26" name="bNames" color="7" fill="1" visible="no" active="yes"/>
 <layer number="27" name="tValues" color="7" fill="1" visible="no" active="yes"/>
 <layer number="28" name="bValues" color="7" fill="1" visible="no" active="yes"/>
@@
 <attribute name="VALUE" x="25.765" y="27.695" size="1.27" layer="27"/>
 </element>
-<element name="R31" library="rcl" library_urn="urn:adsk.eagle:library:334" package="R0603" package3d_urn="urn:adsk.eagle:package:23555/3" value="10k" x="9.1" y="16.1" smashed="yes" rot="R180">
-<attribute name="NAME" x="8.465" y="17.035" size="0.6096" layer="25"/>
-<attribute name="SPICEPREFIX" value="R" x="9.1" y="16.1" size="1.778" layer="27" rot="R180" display="off"/>
-<attribute name="VALUE" x="9.735" y="18.005" size="1.27" layer="27" rot="R180"/>
+<element name="R31" library="rcl" library_urn="urn:adsk.eagle:library:334" package="R0603" package3d_urn="urn:adsk.eagle:package:23555/3" value="10k" x="10.1" y="16.7" smashed="yes" rot="R90">
+<attribute name="NAME" x="9.465" y="15.965" size="0.6096" layer="25" rot="R90"/>
+<attribute name="SPICEPREFIX" value="R" x="10.1" y="16.7" size="1.778" layer="27" rot="R90" display="off"/>
+<attribute name="VALUE" x="12.005" y="16.065" size="1.27" layer="27" rot="R90"/>
 </element>
 <element name="CN1" library="adafruit" library_urn="urn:adsk.eagle:library:420" package="JST-PH-2-THM-RA" package3d_urn="urn:adsk.eagle:package:6240694/1" value="" x="4.2" y="25.3" smashed="yes">
@@
 <attribute name="VALUE" x="26.03" y="-1.16" size="1.27" layer="28" rot="MR180"/>
 </element>
-<element name="C21" library="rcl" library_urn="urn:adsk.eagle:library:334" package="C1206" package3d_urn="urn:adsk.eagle:package:23618/2" value="10uF" x="18" y="26.4" smashed="yes" rot="R270">
-<attribute name="NAME" x="17.33" y="23.47" size="0.6096" layer="25"/>
-<attribute name="POPULARITY" value="54" x="18" y="26.4" size="1.778" layer="27" rot="R270" display="off"/>
-<attribute name="SPICEPREFIX" value="C" x="18" y="26.4" size="1.778" layer="27" rot="R270" display="off"/>
-<attribute name="VALUE" x="15.46" y="27.67" size="1.27" layer="27" rot="R270"/>
+<element name="C21" library="rcl" library_urn="urn:adsk.eagle:library:334" package="C1206" package3d_urn="urn:adsk.eagle:package:23618/2" value="10uF" x="22.4" y="26.6" smashed="yes" rot="R270">
+<attribute name="NAME" x="21.73" y="23.67" size="0.6096" layer="25"/>
+<attribute name="POPULARITY" value="54" x="22.4" y="26.6" size="1.778" layer="27" rot="R270" display="off"/>
+<attribute name="SPICEPREFIX" value="C" x="22.4" y="26.6" size="1.778" layer="27" rot="R270" display="off"/>
+<attribute name="VALUE" x="19.86" y="27.87" size="1.27" layer="27" rot="R270"/>
 </element>
 <element name="C26" library="rcl" library_urn="urn:adsk.eagle:library:334" package="C0603" package3d_urn="urn:adsk.eagle:package:23616/2" value="0.1uF" x="15.5" y="-22.1" smashed="yes">
@@
 <attribute name="POPULARITY" value="79" x="50.65" y="12.1" size="1.778" layer="27" rot="R270" display="off"/>
 <attribute name="VALUE" x="47.475" y="19.72" size="1.27" layer="27" rot="R270"/>
-</element>
-<element name="C24" library="rcl" library_urn="urn:adsk.eagle:library:334" package="C0603" package3d_urn="urn:adsk.eagle:package:23616/2" value="0.1uF" x="22.6" y="26.5" smashed="yes" rot="R270">
-<attribute name="NAME" x="23.235" y="27.135" size="1.27" layer="25" rot="R270"/>
-<attribute name="POPULARITY" value="73" x="22.6" y="26.5" size="1.778" layer="27" rot="R270" display="off"/>
-<attribute name="SPICEPREFIX" value="C" x="22.6" y="26.5" size="1.778" layer="27" rot="R270" display="off"/>
-<attribute name="VALUE" x="20.695" y="27.135" size="1.27" layer="27" rot="R270"/>
-</element>
-<element name="C36" library="rcl" library_urn="urn:adsk.eagle:library:334" package="C0603" package3d_urn="urn:adsk.eagle:package:23616/2" value="0.1uF" x="13.3" y="18" smashed="yes" rot="R180">
-<attribute name="NAME" x="14.865" y="17.535" size="0.6096" layer="25"/>
-<attribute name="POPULARITY" value="73" x="13.3" y="18" size="1.778" layer="27" rot="R180" display="off"/>
-<attribute name="SPICEPREFIX" value="C" x="13.3" y="18" size="1.778" layer="27" rot="R180" display="off"/>
-<attribute name="VALUE" x="13.935" y="19.905" size="1.27" layer="27" rot="R180"/>
 </element>
 </elements>
@@
 <wire x1="12.38" y1="11.27" x2="7.7" y2="11.27" width="0.4064" layer="1"/>
 <contactref element="JP7" pad="3"/>
-<contactref element="C24" pad="2"/>
-<contactref element="C36" pad="2"/>
-<wire x1="12.45" y1="16.8" x2="12.45" y2="18" width="0" layer="19" extent="1-1"/>
 </signal>
 <signal name="SCL">
@@
 <contactref element="R31" pad="2"/>
 <contactref element="C30" pad="1"/>
-<via x="15.4" y="17.2" extent="1-16" drill="0.35"/>
-<via x="15.4" y="18.1" extent="1-16" drill="0.35"/>
-<via x="15.4" y="16.3" extent="1-16" drill="0.35"/>
-<wire x1="14.15" y1="16.8" x2="14.1" y2="16.85" width="0.4064" layer="1"/>
+<via x="13.1" y="18" extent="1-16" drill="0.35"/>
+<via x="13.7" y="18" extent="1-16" drill="0.35"/>
+<via x="12.2" y="18" extent="1-16" drill="0.35"/>
+<wire x1="14.15" y1="16.8" x2="13.7" y2="17.25" width="0.4064" layer="1"/>
+<wire x1="13.7" y1="17.25" x2="13.7" y2="18" width="0.4064" layer="1"/>
+<wire x1="13.7" y1="18" x2="13.1" y2="18" width="0.4064" layer="1"/>
+<wire x1="13.1" y1="18" x2="12.2" y2="18" width="0.4064" layer="1"/>
 <wire x1="13.55" y1="15.455" x2="13.55" y2="15.95" width="0.4064" layer="1"/>
 <wire x1="14.15" y1="16.55" x2="14.15" y2="16.8" width="0.4064" layer="1"/>
 <wire x1="13.55" y1="15.95" x2="14.15" y2="16.55" width="0.4064" layer="1"/>
+<wire x1="10.1" y1="17.55" x2="10.55" y2="18" width="0.254" layer="1"/>
+<wire x1="10.55" y1="18" x2="12.2" y2="18" width="0.254" layer="1"/>
 <contactref element="C21" pad="1"/>
 <wire x1="27.25" y1="29.6" x2="27.35" y2="29.6" width="0.4064" layer="1"/>
@@
 <wire x1="27.25" y1="30.25" x2="26.7" y2="30.8" width="0.4064" layer="1"/>
 <contactref element="JP6" pad="4"/>
-<contactref element="C24" pad="1"/>
-<contactref element="C36" pad="1"/>
-<wire x1="14.15" y1="18" x2="14.15" y2="16.8" width="0.4064" layer="1"/>
-<wire x1="14.15" y1="18" x2="14.25" y2="18.1" width="0.4064" layer="1"/>
-<wire x1="14.25" y1="18.1" x2="15.4" y2="18.1" width="0.4064" layer="1"/>
-<wire x1="15.4" y1="18.1" x2="15.4" y2="17.2" width="0.4064" layer="1"/>
-<wire x1="15.4" y1="17.2" x2="15.4" y2="16.6" width="0.4064" layer="1"/>
-<wire x1="15.4" y1="16.6" x2="15.4" y2="16.3" width="0.4064" layer="1"/>
-<wire x1="14.15" y1="16.8" x2="14.35" y2="16.6" width="0.4064" layer="1"/>
-<wire x1="14.35" y1="16.6" x2="15.4" y2="16.6" width="0.4064" layer="1"/>
-<polygon width="0.254" layer="1" isolate="0.254" thermals="no">
-<vertex x="13.4" y="18.4"/>
-<vertex x="15.7" y="18.4"/>
-<vertex x="15.7" y="16"/>
-<vertex x="14.7" y="15"/>
-<vertex x="13.4" y="15"/>
-</polygon>
-<wire x1="7.7" y1="13.81" x2="7.7" y2="15.55" width="0.254" layer="1"/>
-<wire x1="7.7" y1="15.55" x2="8.25" y2="16.1" width="0.254" layer="1"/>
+<wire x1="7.7" y1="13.81" x2="7.7" y2="15.9" width="0.4064" layer="1"/>
+<wire x1="9.35" y1="17.55" x2="10.1" y2="17.55" width="0.4064" layer="1"/>
+<wire x1="7.7" y1="15.9" x2="9.35" y2="17.55" width="0.4064" layer="1"/>
 </signal>
 <signal name="ESC_1">
@@
 <contactref element="U6" pad="3"/>
 <contactref element="R31" pad="1"/>
-<wire x1="9.95" y1="16.1" x2="10.35" y2="15.7" width="0.254" layer="1"/>
+<wire x1="10.1" y1="15.85" x2="10.25" y2="15.7" width="0.254" layer="1"/>
 <wire x1="11.405" y1="15.7" x2="11.65" y2="15.455" width="0.254" layer="1"/>
-<wire x1="10.35" y1="15.7" x2="11.405" y2="15.7" width="0.254" layer="1"/>
+<wire x1="10.25" y1="15.7" x2="11.405" y2="15.7" width="0.254" layer="1"/>
 </signal>
 <signal name="N$33">
